Commit message: fix: file path in xacro

File: dsr_description2/urdf/a0509.blue.urdf (robot description, URDF)
Before this commit: robot a0509, 8 links, 7 joints
Links:
- link base_link: geometry visual mesh filename=$(find dsr_description2)/meshes/a0509_blue/A0509_0_0.dae scale=0.001 0.001 0.001
- link link_1: geometry visual mesh filename=$(find dsr_description2)/meshes/a0509_blue/A0509_1_0.dae scale=0.001 0.001 0.001; visual mesh filename=$(find dsr_description2)/meshes/a0509_blue/A0509_1_1.dae scale=0.001 0.001 0.001
- link link_2: geometry visual mesh filename=$(find dsr_description2)/meshes/a0509_blue/A0509_2_0.dae scale=0.001 0.001 0.001; visual mesh filename=$(find dsr_description2)/meshes/a0509_blue/A0509_2_1.dae scale=0.001 0.001 0.001
- link link_3: geometry visual mesh filename=$(find dsr_description2)/meshes/a0509_blue/A0509_3_0.dae scale=0.001 0.001 0.001; visual mesh filename=$(find dsr_description2)/meshes/a0509_blue/A0509_3_1.dae scale=0.001 0.001 0.001
- link link_4: geometry visual mesh filename=$(find dsr_description2)/meshes/a0509_blue/A0509_4_0.dae scale=0.001 0.001 0.001; visual mesh filename=$(find dsr_description2)/meshes/a0509_blue/A0509_4_1.dae scale=0.001 0.001 0.001
- link link_5: geometry visual mesh filename=$(find dsr_description2)/meshes/a0509_blue/A0509_5_0.dae scale=0.001 0.001 0.001; visual mesh filename=$(find dsr_description2)/meshes/a0509_blue/A0509_5_1.dae scale=0.001 0.001 0.001
- link link_6: geometry visual mesh filename=$(find dsr_description2)/meshes/a0509_blue/A0509_6_0.dae scale=0.001 0.001 0.001

File: dsr_description2/urdf/a0509.urdf (robot description, URDF)
Before this commit: robot a0509, 9 links, 8 joints
Links:
- link base_link: geometry collision mesh filename=$(find dsr_description2)/meshes/a0509_collision/A0509_0_0.d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 scale=0.001 0.001 0.001; visual mesh filename=$(find dsr_description2)/meshes/a0509_white/A0509_0_0.dae scale=0.001 0.001 0.001
- link link_1: geometry collision mesh filename=$(find dsr_description2)/meshes/a0509_collision/A0509_1_0.d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 scale=0.001 0.001 0.001; collision mesh filename=$(find dsr_description2)/meshes/a0509_collision/A0509_1_1.d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 scale=0.001 0.001 0.001
- link link_2: geometry collision mesh filename=$(find dsr_description2)/meshes/a0509_collision/A0509_2_0.d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 scale=0.001 0.001 0.001; collision mesh filename=$(find dsr_description2)/meshes/a0509_collision/A0509_2_1.d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 scale=0.001 0.001 0.001
- link link_3: geometry collision mesh filename=$(find dsr_description2)/meshes/a0509_collision/A0509_3_0.d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 scale=0.001 0.001 0.001; collision mesh filename=$(find dsr_description2)/meshes/a0509_collision/A0509_3_1.d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 scale=0.001 0.001 0.001
- link link_4: geometry collision mesh filename=$(find dsr_description2)/meshes/a0509_collision/A0509_4_0.d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 scale=0.001 0.001 0.001; collision mesh filename=$(find dsr_description2)/meshes/a0509_collision/A0509_4_1.d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 scale=0.001 0.001 0.001
- link link_5: geometry collision mesh filename=$(find dsr_description2)/meshes/a0509_collision/A0509_5_0.d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 scale=0.001 0.001 0.001; collision mesh filename=$(find dsr_description2)/meshes/a0509_collision/A0509_5_1.d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 scale=0.001 0.001 0.001
- link link_6: geometry collision mesh filename=$(find dsr_description2)/meshes/a0509_collision/A0509_6_0.d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 scale=0.001 0.001 0.001; visual mesh filename=$(find dsr_description2)/meshes/a0509_white/A0509_6_0.dae scale=0.001 0.001 0.001

File: dsr_description2/urdf/a0509.white.urdf (robot description, URDF)
Before this commit: robot a0509, 8 links, 7 joints
Links:
- link base_link: geometry visual mesh filename=$(find dsr_description2)/meshes/a0509_white/A0509_0_0.dae scale=0.001 0.001 0.001
- link link_1: geometry visual mesh filename=$(find dsr_description2)/meshes/a0509_white/A0509_1_0.dae scale=0.001 0.001 0.001; visual mesh filename=$(find dsr_description2)/meshes/a0509_white/A0509_1_1.dae scale=0.001 0.001 0.001
- link link_2: geometry visual mesh filename=$(find dsr_description2)/meshes/a0509_white/A0509_2_0.dae scale=0.001 0.001 0.001; visual mesh filename=$(find dsr_description2)/meshes/a0509_white/A0509_2_1.dae scale=0.001 0.001 0.001
- link link_3: geometry visual mesh filename=$(find dsr_description2)/meshes/a0509_white/A0509_3_0.dae scale=0.001 0.001 0.001; visual mesh filename=$(find dsr_description2)/meshes/a0509_white/A0509_3_1.dae scale=0.001 0.001 0.001
- link link_4: geometry visual mesh filename=$(find dsr_description2)/meshes/a0509_white/A0509_4_0.dae scale=0.001 0.001 0.001; visual mesh filename=$(find dsr_description2)/meshes/a0509_white/A0509_4_1.dae scale=0.001 0.001 0.001
- link link_5: geometry visual mesh filename=$(find dsr_description2)/meshes/a0509_white/A0509_5_0.dae scale=0.001 0.001 0.001; visual mesh filename=$(find dsr_description2)/meshes/a0509_white/A0509_5_1.dae scale=0.001 0.001 0.001
- link link_6: geometry visual mesh filename=$(find dsr_description2)/meshes/a0509_white/A0509_6_0.dae scale=0.001 0.001 0.001

File: dsr_description2/urdf/a0912.blue.urdf (robot description, URDF)
Before this commit: robot a0912, 8 links, 7 joints
Links:
- link base_link: geometry visual mesh filename=$(find dsr_description2)/meshes/a0912_blue/A0912_0_0.dae scale=0.001 0.001 0.001
- link link_1: geometry visual mesh filename=$(find dsr_description2)/meshes/a0912_blue/A0912_1_0.dae scale=0.001 0.001 0.001; visual mesh filename=$(find dsr_description2)/meshes/a0912_blue/A0912_1_1.dae scale=0.001 0.001 0.001
- link link_2: geometry visual mesh filename=$(find dsr_description2)/meshes/a0912_blue/A0912_2_0.dae scale=0.001 0.001 0.001; visual mesh filename=$(find dsr_description2)/meshes/a0912_blue/A0912_2_1.dae scale=0.001 0.001 0.001
- link link_3: geometry visual mesh filename=$(find dsr_description2)/meshes/a0912_blue/A0912_3_0.dae scale=0.001 0.001 0.001; visual mesh filename=$(find dsr_description2)/meshes/a0912_blue/A0912_3_1.dae scale=0.001 0.001 0.001
- link link_4: geometry visual mesh filename=$(find dsr_description2)/meshes/a0912_blue/A0912_4_0.dae scale=0.001 0.001 0.001; visual mesh filename=$(find dsr_description2)/meshes/a0912_blue/A0912_4_1.dae scale=0.001 0.001 0.001
- link link_5: geometry visual mesh filename=$(find dsr_description2)/meshes/a0912_blue/A0912_5_0.dae scale=0.001 0.001 0.001; visual mesh filename=$(find dsr_description2)/meshes/a0912_blue/A0912_5_1.dae scale=0.001 0.001 0.001
- link link_6: geometry visual mesh filename=$(find dsr_description2)/meshes/a0912_blue/A0912_6_0.dae scale=0.001 0.001 0.001

File: dsr_description2/urdf/a0912.urdf (robot description, URDF)
Before this commit: robot a0912, 9 links, 8 joints
Links:
- link base_link: geometry collision mesh filename=$(find dsr_description2)/meshes/a0912_collision/A0912_0_0.d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 scale=0.001 0.001 0.001; visual mesh filename=$(find dsr_description2)/meshes/a0912_white/A0912_0_0.dae scale=0.001 0.001 0.001
- link link_1: geometry collision mesh filename=$(find dsr_description2)/meshes/a0912_collision/A0912_1_0.d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 scale=0.001 0.001 0.001; collision mesh filename=$(find dsr_description2)/meshes/a0912_collision/A0912_1_1.d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 scale=0.001 0.001 0.001
- link link_2: geometry collision mesh filename=$(find dsr_description2)/meshes/a0912_collision/A0912_2_0.d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 scale=0.001 0.001 0.001; collision mesh filename=$(find dsr_description2)/meshes/a0912_collision/A0912_2_1.d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 scale=0.001 0.001 0.001
- link link_3: geometry collision mesh filename=$(find dsr_description2)/meshes/a0912_collision/A0912_3_0.d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 scale=0.001 0.001 0.001; collision mesh filename=$(find dsr_description2)/meshes/a0912_collision/A0912_3_1.d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 scale=0.001 0.001 0.001
- link link_4: geometry collision mesh filename=$(find dsr_description2)/meshes/a0912_collision/A0912_4_0.d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 scale=0.001 0.001 0.001; collision mesh filename=$(find dsr_description2)/meshes/a0912_collision/A0912_4_1.d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 scale=0.001 0.001 0.001
- link link_5: geometry collision mesh filename=$(find dsr_description2)/meshes/a0912_collision/A0912_5_0.d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 scale=0.001 0.001 0.001; collision mesh filename=$(find dsr_description2)/meshes/a0912_collision/A0912_5_1.d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 scale=0.001 0.001 0.001
- link link_6: geometry collision mesh filename=$(find dsr_description2)/meshes/a0912_collision/A0912_6_0.d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 scale=0.001 0.001 0.001; visual mesh filename=$(find dsr_description2)/meshes/a0912_white/A0912_6_0.dae scale=0.001 0.001 0.001

File: dsr_description2/urdf/a0912.white.urdf (robot description, URDF)
Before this commit: robot a0912, 8 links, 7 joints
Links:
- link base_link: geometry visual mesh filename=$(find dsr_description2)/meshes/a0912_white/A0912_0_0.dae scale=0.001 0.001 0.001
- link link_1: geometry visual mesh filename=$(find dsr_description2)/meshes/a0912_white/A0912_1_0.dae scale=0.001 0.001 0.001; visual mesh filename=$(find dsr_description2)/meshes/a0912_white/A0912_1_1.dae scale=0.001 0.001 0.001
- link link_2: geometry visual mesh filename=$(find dsr_description2)/meshes/a0912_white/A0912_2_0.dae scale=0.001 0.001 0.001; visual mesh filename=$(find dsr_description2)/meshes/a0912_white/A0912_2_1.dae scale=0.001 0.001 0.001
- link link_3: geometry visual mesh filename=$(find dsr_description2)/meshes/a0912_white/A0912_3_0.dae scale=0.001 0.001 0.001; visual mesh filename=$(find dsr_description2)/meshes/a0912_white/A0912_3_1.dae scale=0.001 0.001 0.001
- link link_4: geometry visual mesh filename=$(find dsr_description2)/meshes/a0912_white/A0912_4_0.dae scale=0.001 0.001 0.001; visual mesh filename=$(find dsr_description2)/meshes/a0912_white/A0912_4_1.dae scale=0.001 0.001 0.001
- link link_5: geometry visual mesh filename=$(find dsr_description2)/meshes/a0912_white/A0912_5_0.dae scale=0.001 0.001 0.001; visual mesh filename=$(find dsr_description2)/meshes/a0912_white/A0912_5_1.dae scale=0.001 0.001 0.001
- link link_6: geometry visual mesh filename=$(find dsr_description2)/meshes/a0912_white/A0912_6_0.dae scale=0.001 0.001 0.001

File: dsr_description2/urdf/e0509.urdf (robot description, URDF)
Before this commit: robot e0509, 9 links, 8 joints
Links:
- link base_link: geometry collision mesh filename=$(find dsr_description2)/meshes/e0509_collision/E0509_0_0.d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 scale=0.001 0.001 0.001; visual mesh filename=$(find dsr_description2)/meshes/e0509_white/E0509_0_0.dae scale=0.001 0.001 0.001
- link link_1: geometry collision mesh filename=$(find dsr_description2)/meshes/e0509_collision/E0509_1_1.d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 scale=0.001 0.001 0.001; collision mesh filename=$(find dsr_description2)/meshes/e0509_collision/E0509_1_2.d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 scale=0.001 0.001 0.001
- link link_2: geometry collision mesh filename=$(find dsr_description2)/meshes/e0509_collision/E0509_2_1.d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 scale=0.001 0.001 0.001; collision mesh filename=$(find dsr_description2)/meshes/e0509_collision/E0509_2_2.d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 scale=0.001 0.001 0.001
- link link_3: geometry collision mesh filename=$(find dsr_description2)/meshes/e0509_collision/E0509_3_1.d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 scale=0.001 0.001 0.001; collision mesh filename=$(find dsr_description2)/meshes/e0509_collision/E0509_3_2.d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 scale=0.001 0.001 0.001
- link link_4: geometry collision mesh filename=$(find dsr_description2)/meshes/e0509_collision/E0509_4_1.d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 scale=0.001 0.001 0.001; collision mesh filename=$(find dsr_description2)/meshes/e0509_collision/E0509_4_2.d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 scale=0.001 0.001 0.001
- link link_5: geometry collision mesh filename=$(find dsr_description2)/meshes/e0509_collision/E0509_5_1.d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 scale=0.001 0.001 0.001; collision mesh filename=$(find dsr_description2)/meshes/e0509_collision/E0509_5_2.d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 scale=0.001 0.001 0.001
- link link_6: geometry collision mesh filename=$(find dsr_description2)/meshes/e0509_collision/E0509_6_1.d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 scale=0.001 0.001 0.001; visual mesh filename=$(find dsr_description2)/meshes/e0509_white/E0509_6_1.dae scale=0.001 0.001 0.001

File: dsr_description2/urdf/h2017.blue.urdf (robot description, URDF)
Before this commit: robot h2017, 8 links, 7 joints
Links:
- link base_link: geometry visual mesh filename=$(find dsr_description2)/meshes/h2017_blue/H2017_0_0.dae scale=0.001 0.001 0.001
- link link_1: geometry visual mesh filename=$(find dsr_description2)/meshes/h2017_blue/H2017_1_0.dae scale=0.001 0.001 0.001
- link link_2: geometry visual mesh filename=$(find dsr_description2)/meshes/h2017_blue/H2017_2_0.dae scale=0.001 0.001 0.001; visual mesh filename=$(find dsr_description2)/meshes/h2017_blue/H2017_2_1.dae scale=0.001 0.001 0.001
- link link_3: geometry visual mesh filename=$(find dsr_description2)/meshes/h2017_blue/H2017_3_0.dae scale=0.001 0.001 0.001
- link link_4: geometry visual mesh filename=$(find dsr_description2)/meshes/h2017_blue/H2017_4_0.dae scale=0.001 0.001 0.001; visual mesh filename=$(find dsr_description2)/meshes/h2017_blue/H2017_4_1.dae scale=0.001 0.001 0.001
- link link_5: geometry visual mesh filename=$(find dsr_description2)/meshes/h2017_blue/H2017_5_0.dae scale=0.001 0.001 0.001
- link link_6: geometry visual mesh filename=$(find dsr_description2)/meshes/h2017_blue/H2017_6_0.dae scale=0.001 0.001 0.001

File: dsr_description2/urdf/h2515.blue.urdf (robot description, URDF)
Before this commit: robot h2515, 8 links, 7 joints
Links:
- link base_link: geometry visual mesh filename=$(find dsr_description2)/meshes/h2515_blue/H2515_0_0.dae scale=0.001 0.001 0.001
- link link_1: geometry visual mesh filename=$(find dsr_description2)/meshes/h2515_blue/H2515_1_0.dae scale=0.001 0.001 0.001
- link link_2: geometry visual mesh filename=$(find dsr_description2)/meshes/h2515_blue/H2515_2_0.dae scale=0.001 0.001 0.001; visual mesh filename=$(find dsr_description2)/meshes/h2515_blue/H2515_2_1.dae scale=0.001 0.001 0.001
- link link_3: geometry visual mesh filename=$(find dsr_description2)/meshes/h2515_blue/H2515_3_0.dae scale=0.001 0.001 0.001
- link link_4: geometry visual mesh filename=$(find dsr_description2)/meshes/h2515_blue/H2515_4_0.dae scale=0.001 0.001 0.001; visual mesh filename=$(find dsr_description2)/meshes/h2515_blue/H2515_4_1.dae scale=0.001 0.001 0.001
- link link_5: geometry visual mesh filename=$(find dsr_description2)/meshes/h2515_blue/H2515_5_0.dae scale=0.001 0.001 0.001
- link link_6: geometry visual mesh filename=$(find dsr_description2)/meshes/h2515_blue/H2515_6_0.dae scale=0.001 0.001 0.001

File: dsr_description2/urdf/h2515.urdf (robot description, URDF)
Before this commit: robot h2515, 9 links, 8 joints
Links:
- link base_link: geometry collision mesh filename=$(find dsr_description2)/meshes/h2515_collision/H2515_0_0.d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 scale=0.001 0.001 0.001; visual mesh filename=$(find dsr_description2)/meshes/h2515_blue/H2515_0_0.dae scale=0.001 0.001 0.001
- link link_1: geometry collision mesh filename=$(find dsr_description2)/meshes/h2515_collision/H2515_1_0.d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 scale=0.001 0.001 0.001; visual mesh filename=$(find dsr_description2)/meshes/h2515_white/H2515_1_0.dae scale=0.001 0.001 0.001
- link link_2: geometry collision mesh filename=$(find dsr_description2)/meshes/h2515_collision/H2515_2_0.d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 scale=0.001 0.001 0.001; collision mesh filename=$(find dsr_description2)/meshes/h2515_collision/H2515_2_1.d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 scale=0.001 0.001 0.001
- link link_3: geometry collision mesh filename=$(find dsr_description2)/meshes/h2515_collision/H2515_3_0.d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 scale=0.001 0.001 0.001; visual mesh filename=$(find dsr_description2)/meshes/h2515_white/H2515_3_0.dae scale=0.001 0.001 0.001
- link link_4: geometry collision mesh filename=$(find dsr_description2)/meshes/h2515_collision/H2515_4_0.d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 scale=0.001 0.001 0.001; collision mesh filename=$(find dsr_description2)/meshes/h2515_collision/H2515_4_1.d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 scale=0.001 0.001 0.001
- link link_5: geometry collision mesh filename=$(find dsr_description2)/meshes/h2515_collision/H2515_5_0.d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 scale=0.001 0.001 0.001; visual mesh filename=$(find dsr_description2)/meshes/h2515_white/H2515_5_0.dae scale=0.001 0.001 0.001
- link link_6: geometry collision mesh filename=$(find dsr_description2)/meshes/h2515_collision/H2515_6_0.d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 scale=0.001 0.001 0.001; visual mesh filename=$(find dsr_description2)/meshes/h2515_white/H2515_6_0.dae scale=0.001 0.001 0.001

File: dsr_description2/urdf/h2515.white.urdf (robot description, URDF)
Before this commit: robot h2515, 8 links, 7 joints
Links:
- link base_link: geometry visual mesh filename=$(find dsr_description2)/meshes/h2515_white/H2515_0_0.dae scale=0.001 0.001 0.001
- link link_1: geometry visual mesh filename=$(find dsr_description2)/meshes/h2515_white/H2515_1_0.dae scale=0.001 0.001 0.001
- link link_2: geometry visual mesh filename=$(find dsr_description2)/meshes/h2515_white/H2515_2_0.dae scale=0.001 0.001 0.001; visual mesh filename=$(find dsr_description2)/meshes/h2515_white/H2515_2_1.dae scale=0.001 0.001 0.001
- link link_3: geometry visual mesh filename=$(find dsr_description2)/meshes/h2515_white/H2515_3_0.dae scale=0.001 0.001 0.001
- link link_4: geometry visual mesh filename=$(find dsr_description2)/meshes/h2515_white/H2515_4_0.dae scale=0.001 0.001 0.001; visual mesh filename=$(find dsr_description2)/meshes/h2515_white/H2515_4_1.dae scale=0.001 0.001 0.001
- link link_5: geometry visual mesh filename=$(find dsr_description2)/meshes/h2515_white/H2515_5_0.dae scale=0.001 0.001 0.001
- link link_6: geometry visual mesh filename=$(find dsr_description2)/meshes/h2515_white/H2515_6_0.dae scale=0.001 0.001 0.001

File: dsr_description2/urdf/m0609.blue.urdf (robot description, URDF)
Before this commit: robot m0609, 8 links, 7 joints
Links:
- link base_link: geometry visual mesh filename=$(find dsr_description2)/meshes/m0609_blue/MF0609_0_0.dae scale=0.001 0.001 0.001
- link link_1: geometry visual mesh filename=$(find dsr_description2)/meshes/m0609_blue/MF0609_1_0.dae scale=0.001 0.001 0.001
- link link_2: geometry visual mesh filename=$(find dsr_description2)/meshes/m0609_blue/MF0609_2_0.dae scale=0.001 0.001 0.001; visual mesh filename=$(find dsr_description2)/meshes/m0609_blue/MF0609_2_1.dae scale=0.001 0.001 0.001
- link link_3: geometry visual mesh filename=$(find dsr_description2)/meshes/m0609_blue/MF0609_3_0.dae scale=0.001 0.001 0.001
- link link_4: geometry visual mesh filename=$(find dsr_description2)/meshes/m0609_blue/MF0609_4_0.dae scale=0.001 0.001 0.001; visual mesh filename=$(find dsr_description2)/meshes/m0609_blue/MF0609_4_1.dae scale=0.001 0.001 0.001
- link link_5: geometry visual mesh filename=$(find dsr_description2)/meshes/m0609_blue/MF0609_5_0.dae scale=0.001 0.001 0.001
- link link_6: geometry visual mesh filename=$(find dsr_description2)/meshes/m0609_blue/MF0609_6_0.dae scale=0.001 0.001 0.001

File: dsr_description2/urdf/m0609.urdf (robot description, URDF)
Before this commit: robot m0609, 9 links, 8 joints
Links:
- link base_link: geometry collision mesh filename=$(find dsr_description2)/meshes/m0609_collision/MF0609_0_0.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 scale=0.001 0.001 0.001; visual mesh filename=$(find dsr_description2)/meshes/m0609_white/MF0609_0_0.dae scale=0.001 0.001 0.001
- link link_1: geometry collision mesh filename=$(find dsr_description2)/meshes/m0609_collision/MF0609_1_0.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 scale=0.001 0.001 0.001; visual mesh filename=$(find dsr_description2)/meshes/m0609_white/MF0609_1_0.dae scale=0.001 0.001 0.001
- link link_2: geometry collision mesh filename=$(find dsr_description2)/meshes/m0609_collision/MF0609_2_0.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 scale=0.001 0.001 0.001; collision mesh filename=$(find dsr_description2)/meshes/m0609_collision/MF0609_2_1.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 scale=0.001 0.001 0.001
- link link_3: geometry collision mesh filename=$(find dsr_description2)/meshes/m0609_collision/MF0609_3_0.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 scale=0.001 0.001 0.001; visual mesh filename=$(find dsr_description2)/meshes/m0609_white/MF0609_3_0.dae scale=0.001 0.001 0.001
- link link_4: geometry collision mesh filename=$(find dsr_description2)/meshes/m0609_collision/MF0609_4_0.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 scale=0.001 0.001 0.001; collision mesh filename=$(find dsr_description2)/meshes/m0609_collision/MF0609_4_1.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 scale=0.001 0.001 0.001
- link link_5: geometry collision mesh filename=$(find dsr_description2)/meshes/m0609_collision/MF0609_5_0.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 scale=0.001 0.001 0.001; visual mesh filename=$(find dsr_description2)/meshes/m0609_white/MF0609_5_0.dae scale=0.001 0.001 0.001
- link link_6: geometry collision mesh filename=$(find dsr_description2)/meshes/m0609_collision/MF0609_6_0.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 scale=0.001 0.001 0.001; visual mesh filename=$(find dsr_description2)/meshes/m0609_white/MF0609_6_0.dae scale=0.001 0.001 0.001

File: dsr_description2/urdf/m0609.white.urdf (robot description, URDF)
Before this commit: robot m0609, 8 links, 7 joints
Links:
- link base_link: geometry visual mesh filename=$(find dsr_description2)/meshes/m0609_white/MF0609_0_0.dae scale=0.001 0.001 0.001
- link link_1: geometry visual mesh filename=$(find dsr_description2)/meshes/m0609_white/MF0609_1_0.dae scale=0.001 0.001 0.001
- link link_2: geometry visual mesh filename=$(find dsr_description2)/meshes/m0609_white/MF0609_2_0.dae scale=0.001 0.001 0.001; visual mesh filename=$(find dsr_description2)/meshes/m0609_white/MF0609_2_1.dae scale=0.001 0.001 0.001
- link link_3: geometry visual mesh filename=$(find dsr_description2)/meshes/m0609_white/MF0609_3_0.dae scale=0.001 0.001 0.001
- link link_4: geometry visual mesh filename=$(find dsr_description2)/meshes/m0609_white/MF0609_4_0.dae scale=0.001 0.001 0.001; visual mesh filename=$(find dsr_description2)/meshes/m0609_white/MF0609_4_1.dae scale=0.001 0.001 0.001
- link link_5: geometry visual mesh filename=$(find dsr_description2)/meshes/m0609_white/MF0609_5_0.dae scale=0.001 0.001 0.001
- link link_6: geometry visual mesh filename=$(find dsr_description2)/meshes/m0609_white/MF0609_6_0.dae scale=0.001 0.001 0.001

File: dsr_description2/urdf/m0617.blue.urdf (robot description, URDF)
Before this commit: robot m0617, 8 links, 7 joints
Links:
- link base_link: geometry visual mesh filename=$(find dsr_description2)/meshes/m0617_blue/MF0617_0_0.dae scale=0.001 0.001 0.001
- link link_1: geometry visual mesh filename=$(find dsr_description2)/meshes/m0617_blue/MF0617_1_0.dae scale=0.001 0.001 0.001
- link link_2: geometry visual mesh filename=$(find dsr_description2)/meshes/m0617_blue/MF0617_2_0.dae scale=0.001 0.001 0.001; visual mesh filename=$(find dsr_description2)/meshes/m0617_blue/MF0617_2_1.dae scale=0.001 0.001 0.001
- link link_3: geometry visual mesh filename=$(find dsr_description2)/meshes/m0617_blue/MF0617_3_0.dae scale=0.001 0.001 0.001
- link link_4: geometry visual mesh filename=$(find dsr_description2)/meshes/m0617_blue/MF0617_4_0.dae scale=0.001 0.001 0.001; visual mesh filename=$(find dsr_description2)/meshes/m0617_blue/MF0617_4_1.dae scale=0.001 0.001 0.001
- link link_5: geometry visual mesh filename=$(find dsr_description2)/meshes/m0617_blue/MF0617_5_0.dae scale=0.001 0.001 0.001
- link link_6: geometry visual mesh filename=$(find dsr_description2)/meshes/m0617_blue/MF0617_6_0.dae scale=0.001 0.001 0.001
