Commit message: fix: file path in xacro

File: dsr_description2/urdf/m0617.urdf (robot description, URDF)
Before this commit: robot m0617, 9 links, 8 joints
Links:
- link base_link: geometry collision mesh filename=$(find dsr_description2)/meshes/m0617_collision/MF0617_0_0.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 scale=0.001 0.001 0.001; visual mesh filename=$(find dsr_description2)/meshes/m0617_white/MF0617_0_0.dae scale=0.001 0.001 0.001
- link link_1: geometry collision mesh filename=$(find dsr_description2)/meshes/m0617_collision/MF0617_1_0.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 scale=0.001 0.001 0.001; visual mesh filename=$(find dsr_description2)/meshes/m0617_white/MF0617_1_0.dae scale=0.001 0.001 0.001
- link link_2: geometry collision mesh filename=$(find dsr_description2)/meshes/m0617_collision/MF0617_2_0.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 scale=0.001 0.001 0.001; collision mesh filename=$(find dsr_description2)/meshes/m0617_collision/MF0617_2_1.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 scale=0.001 0.001 0.001
- link link_3: geometry collision mesh filename=$(find dsr_description2)/meshes/m0617_collision/MF0617_3_0.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 scale=0.001 0.001 0.001; visual mesh filename=$(find dsr_description2)/meshes/m0617_white/MF0617_3_0.dae scale=0.001 0.001 0.001
- link link_4: geometry collision mesh filename=$(find dsr_description2)/meshes/m0617_collision/MF0617_4_0.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 scale=0.001 0.001 0.001; collision mesh filename=$(find dsr_description2)/meshes/m0617_collision/MF0617_4_1.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 scale=0.001 0.001 0.001
- link link_5: geometry collision mesh filename=$(find dsr_description2)/meshes/m0617_collision/MF0617_5_0.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 scale=0.001 0.001 0.001; visual mesh filename=$(find dsr_description2)/meshes/m0617_white/MF0617_5_0.dae scale=0.001 0.001 0.001
- link link_6: geometry collision mesh filename=$(find dsr_description2)/meshes/m0617_collision/MF0617_6_0.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 scale=0.001 0.001 0.001; visual mesh filename=$(find dsr_description2)/meshes/m0617_white/MF0617_6_0.dae scale=0.001 0.001 0.001

File: dsr_description2/urdf/m0617.white.urdf (robot description, URDF)
Before this commit: robot m0617, 8 links, 7 joints
Links:
- link base_link: geometry visual mesh filename=$(find dsr_description2)/meshes/m0617_white/MF0617_0_0.dae scale=0.001 0.001 0.001
- link link_1: geometry visual mesh filename=$(find dsr_description2)/meshes/m0617_white/MF0617_1_0.dae scale=0.001 0.001 0.001
- link link_2: geometry visual mesh filename=$(find dsr_description2)/meshes/m0617_white/MF0617_2_0.dae scale=0.001 0.001 0.001; visual mesh filename=$(find dsr_description2)/meshes/m0617_white/MF0617_2_1.dae scale=0.001 0.001 0.001
- link link_3: geometry visual mesh filename=$(find dsr_description2)/meshes/m0617_white/MF0617_3_0.dae scale=0.001 0.001 0.001
- link link_4: geometry visual mesh filename=$(find dsr_description2)/meshes/m0617_white/MF0617_4_0.dae scale=0.001 0.001 0.001; visual mesh filename=$(find dsr_description2)/meshes/m0617_white/MF0617_4_1.dae scale=0.001 0.001 0.001
- link link_5: geometry visual mesh filename=$(find dsr_description2)/meshes/m0617_white/MF0617_5_0.dae scale=0.001 0.001 0.001
- link link_6: geometry visual mesh filename=$(find dsr_description2)/meshes/m0617_white/MF0617_6_0.dae scale=0.001 0.001 0.001

File: dsr_description2/urdf/m1013.blue.urdf (robot description, URDF)
Before this commit: robot m1013, 8 links, 7 joints
Links:
- link base_link: geometry visual mesh filename=$(find dsr_description2)/meshes/m1013_blue/MF1013_0_0.dae scale=0.001 0.001 0.001
- link link_1: geometry visual mesh filename=$(find dsr_description2)/meshes/m1013_blue/MF1013_1_0.dae scale=0.001 0.001 0.001
- link link_2: geometry visual mesh filename=$(find dsr_description2)/meshes/m1013_blue/MF1013_2_0.dae scale=0.001 0.001 0.001; visual mesh filename=$(find dsr_description2)/meshes/m1013_blue/MF1013_2_1.dae scale=0.001 0.001 0.001
- link link_3: geometry visual mesh filename=$(find dsr_description2)/meshes/m1013_blue/MF1013_3_0.dae scale=0.001 0.001 0.001
- link link_4: geometry visual mesh filename=$(find dsr_description2)/meshes/m1013_blue/MF1013_4_0.dae scale=0.001 0.001 0.001; visual mesh filename=$(find dsr_description2)/meshes/m1013_blue/MF1013_4_1.dae scale=0.001 0.001 0.001
- link link_5: geometry visual mesh filename=$(find dsr_description2)/meshes/m1013_blue/MF1013_5_0.dae scale=0.001 0.001 0.001
- link link_6: geometry visual mesh filename=$(find dsr_description2)/meshes/m1013_blue/MF1013_6_0.dae scale=0.001 0.001 0.001

File: dsr_description2/urdf/m1013.urdf (robot description, URDF)
Before this commit: robot m1013, 9 links, 8 joints
Links:
- link base_link: geometry collision mesh filename=$(find dsr_description2)/meshes/m1013_collision/MF1013_0_0.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 scale=0.001 0.001 0.001; visual mesh filename=$(find dsr_description2)/meshes/m1013_white/MF1013_0_0.dae scale=0.001 0.001 0.001
- link link_1: geometry collision mesh filename=$(find dsr_description2)/meshes/m1013_collision/MF1013_1_0.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 scale=0.001 0.001 0.001; visual mesh filename=$(find dsr_description2)/meshes/m1013_white/MF1013_1_0.dae scale=0.001 0.001 0.001
- link link_2: geometry collision mesh filename=$(find dsr_description2)/meshes/m1013_collision/MF1013_2_0.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 scale=0.001 0.001 0.001; collision mesh filename=$(find dsr_description2)/meshes/m1013_collision/MF1013_2_1.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 scale=0.001 0.001 0.001
- link link_3: geometry collision mesh filename=$(find dsr_description2)/meshes/m1013_collision/MF1013_3_0.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 scale=0.001 0.001 0.001; visual mesh filename=$(find dsr_description2)/meshes/m1013_white/MF1013_3_0.dae scale=0.001 0.001 0.001
- link link_4: geometry collision mesh filename=$(find dsr_description2)/meshes/m1013_collision/MF1013_4_0.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 scale=0.001 0.001 0.001; collision mesh filename=$(find dsr_description2)/meshes/m1013_collision/MF1013_4_1.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 scale=0.001 0.001 0.001
- link link_5: geometry collision mesh filename=$(find dsr_description2)/meshes/m1013_collision/MF1013_5_0.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 scale=0.001 0.001 0.001; visual mesh filename=$(find dsr_description2)/meshes/m1013_white/MF1013_5_0.dae scale=0.001 0.001 0.001
- link link_6: geometry collision mesh filename=$(find dsr_description2)/meshes/m1013_collision/MF1013_6_0.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 scale=0.001 0.001 0.001; visual mesh filename=$(find dsr_description2)/meshes/m1013_white/MF1013_6_0.dae scale=0.001 0.001 0.001

File: dsr_description2/urdf/m1013.white.urdf (robot description, URDF)
Before this commit: robot m1013, 8 links, 7 joints
Links:
- link base_link: geometry visual mesh filename=$(find dsr_description2)/meshes/m1013_white/MF1013_0_0.dae scale=0.001 0.001 0.001
- link link_1: geometry visual mesh filename=$(find dsr_description2)/meshes/m1013_white/MF1013_1_0.dae scale=0.001 0.001 0.001
- link link_2: geometry visual mesh filename=$(find dsr_description2)/meshes/m1013_white/MF1013_2_0.dae scale=0.001 0.001 0.001; visual mesh filename=$(find dsr_description2)/meshes/m1013_white/MF1013_2_1.dae scale=0.001 0.001 0.001
- link link_3: geometry visual mesh filename=$(find dsr_description2)/meshes/m1013_white/MF1013_3_0.dae scale=0.001 0.001 0.001
- link link_4: geometry visual mesh filename=$(find dsr_description2)/meshes/m1013_white/MF1013_4_0.dae scale=0.001 0.001 0.001; visual mesh filename=$(find dsr_description2)/meshes/m1013_white/MF1013_4_1.dae scale=0.001 0.001 0.001
- link link_5: geometry visual mesh filename=$(find dsr_description2)/meshes/m1013_white/MF1013_5_0.dae scale=0.001 0.001 0.001
- link link_6: geometry visual mesh filename=$(find dsr_description2)/meshes/m1013_white/MF1013_6_0.dae scale=0.001 0.001 0.001
