Commit message: Update moveit_config_file for P3020

File: dsr_description2/urdf/p3020.urdf (robot description, URDF)
Before this commit: robot P3020, 23 links, 22 joints
Links:
- removed link FLANGE
- removed link L1
- removed link L1-1
- removed link L1-2
- removed link L1-3
- removed link L1-4
- removed link L2
- removed link L2-1
- removed link L2-2
- removed link L2-3
- removed link L2-4
- removed link L2-5
- removed link L2-6
- removed link L2-7
- removed link L3
- removed link L3-1
- removed link L3-2
- removed link L3-3
- removed link L5
- removed link L5-1
- removed link L5-2
- removed link L6
- removed link base
- added link base_link; collision mesh filename=package://dsr_description2/meshes/p3020/1.STL scale=0.001 0.001 0.001; visual mesh filename=package://dsr_description2/meshes/p3020/1.STL scale=0.001 0.001 0.001
- added link link_1; collision mesh filename=package://dsr_description2/meshes/p3020/2-1.STL scale=0.001 0.001 0.001; collision mesh filename=package://dsr_description2/meshes/p3020/2-2.STL scale=0.001 0.001 0.001
- added link link_2; collision mesh filename=package://dsr_description2/meshes/p3020/3-1.STL scale=0.001 0.001 0.001; collision mesh filename=package://dsr_description2/meshes/p3020/3-2.STL scale=0.001 0.001 0.001
- added link link_3; collision mesh filename=package://dsr_description2/meshes/p3020/4-1.STL scale=0.001 0.001 0.001; collision mesh filename=package://dsr_description2/meshes/p3020/4-2.STL scale=0.001 0.001 0.001
- added link link_4
- added link link_5; collision mesh filename=package://dsr_description2/meshes/p3020/6-1.STL scale=0.001 0.001 0.001; collision mesh filename=package://dsr_description2/meshes/p3020/6-2.STL scale=0.001 0.001 0.001
- added link link_6; collision mesh filename=package://dsr_description2/meshes/p3020/7.STL scale=0.001 0.001 0.001; visual mesh filename=package://dsr_description2/meshes/p3020/7.STL scale=0.001 0.001 0.001
Joints:
- removed joint J1
- removed joint J1-1
- removed joint J1-2
- removed joint J1-3
- removed joint J1-4
- removed joint J2
- removed joint J2-1
- removed joint J2-2
- removed joint J2-3
- removed joint J2-4
- removed joint J2-5
- removed joint J2-6
- removed joint J2-7
- removed joint J3
- removed joint J3-1
- removed joint J3-2
- removed joint J3-3
- removed joint J5
- removed joint J5-1
- removed joint J5-2
- removed joint J6
- removed joint JF
- added joint joint_1: type revolute, parent base_link, child link_1, origin xyz=0 0 0.3943, axis 0 0 1, limit lower=-6.2832 upper=6.2832 effort=50 velocity=3.927
- added joint joint_2: type revolute, parent link_1, child link_2, origin xyz=0 0 0, axis 0 1 0, limit lower=-6.2832 upper=6.2832 effort=50 velocity=3.927
- added joint joint_3: type revolute, parent link_2, child link_3, origin xyz=0 0 1.01, axis 0 1 0, limit lower=-6.2832 upper=6.2832 effort=50 velocity=3.927
- added joint joint_4: type fixed, parent link_3, child link_4, origin xyz=0 0 0
- added joint joint_5: type revolute, parent link_4, child link_5, origin xyz=0 0.20785 0.89, axis 0 1 0, limit lower=-6.2832 upper=6.2832 effort=50 velocity=3.927
- added joint joint_6: type revolute, parent link_5, child link_6, origin xyz=0 0 0.13, axis 0 0 1, limit lower=-6.2832 upper=6.2832 effort=50 velocity=3.927

File: dsr_moveit2/p3020_moveit_config/config/dsr.ros2_control.xacro (robot description, xacro)
@@ -34,5 +34,5 @@
                 </state_interface>
             </joint>
-            <joint name="joint_4">
+            <!-- <joint name="joint_4">
                 <command_interface name="position"/>
                 <state_interface name="position">
@@ -42,5 +42,5 @@
                     <param name="initial_value">0.0</param>
                 </state_interface>
-            </joint>
+            </joint> -->
             <joint name="joint_5">
                 <command_interface name="position"/>
