Commit message: Revised URDF files

File: dsr_description2/urdf/m0609.urdf (robot description, URDF)
Before this commit: robot m0609, 8 links, 7 joints
Joints:
- joint joint_1: origin xyz=0 0 0.1 rpy=0 0 0 -> xyz=0 0 0.1345 rpy=0 0 0

File: dsr_description2/urdf/m0609_isaac_sim.urdf (robot description, URDF)
Before this commit: robot m0609, 9 links, 8 joints
Joints:
- joint joint_1: origin xyz=0 0 0.1 rpy=0 0 0 -> xyz=0 0 0.1345 rpy=0 0 0
