Commit message: update P3020 Model description

File: dsr_description2/xacro/macro.p3020.white.xacro (robot description, xacro)
@@ -28,4 +28,7 @@
                     <mesh filename="package://dsr_description2/meshes/p3020/2-1.STL" scale="0.001 0.001 0.001" />
                 </geometry>
+                <material name="P3020_0">
+                    <color rgba="0.8 0.8 0.8 1" />
+                </material>
             </visual>
             <visual>
@@ -33,4 +36,7 @@
                     <mesh filename="package://dsr_description2/meshes/p3020/2-2.STL" scale="0.001 0.001 0.001" />
                 </geometry>
+                <material name="P3020_0">
+                    <color rgba="0.8 0.8 0.8 1" />
+                </material>
             </visual>
             <visual>
@@ -38,4 +44,7 @@
                     <mesh filename="package://dsr_description2/meshes/p3020/2-3.STL" scale="0.001 0.001 0.001" />
                 </geometry>
+                <material name="P3020_0">
+                    <color rgba="0.8 0.8 0.8 1" />
+                </material>
             </visual>
             <visual>
@@ -43,4 +52,7 @@
                     <mesh filename="package://dsr_description2/meshes/p3020/2-4.STL" scale="0.001 0.001 0.001" />
                 </geometry>
+                <material name="P3020_0">
+                    <color rgba="0.8 0.8 0.8 1" />
+                </material>
             </visual>
             <visual>
@@ -48,4 +60,7 @@
                     <mesh filename="package://dsr_description2/meshes/p3020/2-5.STL" scale="0.001 0.001 0.001" />
                 </geometry>
+                <material name="P3020_0">
+                    <color rgba="0.8 0.8 0.8 1" />
+                </material>
             </visual>
         </link>
@@ -56,4 +71,7 @@
                     <mesh filename="package://dsr_description2/meshes/p3020/3-1.STL" scale="0.001 0.001 0.001" />
                 </geometry>
+                <material name="P3020_0">
+                    <color rgba="0.8 0.8 0.8 1" />
+                </material>
             </visual>
             <visual>
@@ -61,4 +79,7 @@
                     <mesh filename="package://dsr_description2/meshes/p3020/3-2.STL" scale="0.001 0.001 0.001" />
                 </geometry>
+                <material name="P3020_0">
+                    <color rgba="0.8 0.8 0.8 1" />
+                </material>
             </visual>
             <visual>
@@ -71,4 +92,39 @@
                     <mesh filename="package://dsr_description2/meshes/p3020/3-4.STL" scale="0.001 0.001 0.001" />
                 </geometry>
+                <material name="P3020_0">
+                    <color rgba="0.8 0.8 0.8 1" />
+                </material>
+            </visual>
+            <visual>
+                <geometry>
+                    <mesh filename="package://dsr_description2/meshes/p3020/3-5.STL" scale="0.001 0.001 0.001" />
+                </geometry>
+                <material name="P3020_0">
+                    <color rgba="0.8 0.8 0.8 1" />
+                </material>
+            </visual>
+            <visual>
+                <geometry>
+                    <mesh filename="package://dsr_description2/meshes/p3020/3-6.STL" scale="0.001 0.001 0.001" />
+                </geometry>
+                <material name="P3020_0">
+                    <color rgba="0.8 0.8 0.8 1" />
+                </material>
+            </visual>
+            <visual>
+                <geometry>
+                    <mesh filename="package://dsr_description2/meshes/p3020/3-7.STL" scale="0.001 0.001 0.001" />
+                </geometry>
+                <material name="P3020_0">
+                    <color rgba="0.8 0.8 0.8 1" />
+                </material>
+            </visual>
+            <visual>
+                <geometry>
+                    <mesh filename="package://dsr_description2/meshes/p3020/3-8.STL" scale="0.001 0.001 0.001" />
+                </geometry>
+                <material name="P3020_0">
+                    <color rgba="0.8 0.8 0.8 1" />
+                </material>
             </visual>
         </link>
@@ -79,4 +135,7 @@
                     <mesh filename="package://dsr_description2/meshes/p3020/4-1.STL" scale="0.001 0.001 0.001" />
                 </geometry>
+                <material name="P3020_0">
+                    <color rgba="0.8 0.8 0.8 1" />
+                </material>
             </visual>
             <visual>
@@ -84,13 +143,27 @@
                     <mesh filename="package://dsr_description2/meshes/p3020/4-2.STL" scale="0.001 0.001 0.001" />
                 </geometry>
+                <material name="P3020_0">
+                    <color rgba="0.8 0.8 0.8 1" />
+                </material>
+            </visual>
+            <visual>
+                <geometry>
+                    <mesh filename="package://dsr_description2/meshes/p3020/4-3.STL" scale="0.001 0.001 0.001" />
+                </geometry>
+                <material name="P3020_0">
+                    <color rgba="0.8 0.8 0.8 1" />
+                </material>
+            </visual>
+            <visual>
+                <geometry>
+                    <mesh filename="package://dsr_description2/meshes/p3020/4-4.STL" scale="0.001 0.001 0.001" />
+                </geometry>
+                <material name="P3020_0">
+                    <color rgba="0.8 0.8 0.8 1" />
+                </material>
             </visual>
         </link>
         <!-- link_4 (Dummy Link for joint_4) -->
         <link name="link_4">
-            <visual>
-                <geometry>
-                    <box size="1 1 1"/>  <!-- Small placeholder box -->
-                </geometry>
-            </visual>
         </link>
         <!-- link_5 -->
@@ -100,4 +173,7 @@
                     <mesh filename="package://dsr_description2/meshes/p3020/6-1.STL" scale="0.001 0.001 0.001" />
                 </geometry>
+                <material name="P3020_0">
+                    <color rgba="0.8 0.8 0.8 1" />
+                </material>
             </visual>
             <visual>
@@ -105,4 +181,15 @@
                     <mesh filename="package://dsr_description2/meshes/p3020/6-2.STL" scale="0.001 0.001 0.001" />
                 </geometry>
+                <material name="P3020_0">
+                    <color rgba="0.8 0.8 0.8 1" />
+                </material>
+            </visual>
+            <visual>
+                <geometry>
+                    <mesh filename="package://dsr_description2/meshes/p3020/6-3.STL" scale="0.001 0.001 0.001" />
+                </geometry>
+                <material name="P3020_0">
+                    <color rgba="0.8 0.8 0.8 1" />
+                </material>
             </visual>
         </link>
@@ -113,4 +200,7 @@
                     <mesh filename="package://dsr_description2/meshes/p3020/7.STL" scale="0.001 0.001 0.001" />
                 </geometry>
+                <material name="P3020_0">
+                    <color rgba="0.8 0.8 0.8 1" />
+                </material>
             </visual>
         </link>
@@ -123,5 +213,5 @@
         </joint>
         <joint name="joint_2" type="continuous">
-            <origin xyz="0 0 3.943"/>
+            <origin xyz="0 0 0"/>
             <parent link="link_1"/>
             <child link="link_2"/>
@@ -129,5 +219,5 @@
         </joint>
         <joint name="joint_3" type="continuous">
-            <origin xyz="0 0 10.1"/>
+            <origin xyz="0 0 0"/>
             <parent link="link_2"/>
             <child link="link_3"/>
@@ -141,5 +231,5 @@
         </joint>
         <joint name="joint_5" type="continuous">
-            <origin xyz="0 0 8.9"/>
+            <origin xyz="0 0 0"/>
             <parent link="link_4"/>
             <child link="link_5"/>
@@ -147,5 +237,5 @@
         </joint>
         <joint name="joint_6" type="continuous">
-            <origin xyz="0 2.0785 0"/>
+            <origin xyz="0 0 0"/>
             <parent link="link_5"/>
             <child link="link_6"/>
