Commit message: d

File: dsr_description2/xacro/m1013.urdf.xacro (robot description, xacro)
@@ -11,4 +11,5 @@
   <xacro:arg name="mode" default=""/>
   <xacro:arg name="model" default=""/>
+  <xacro:arg name="update_rate" default=""/>
   <xacro:property name="cr" value="$(arg color)"/>
   <xacro:property name="gr" value="$(arg gripper)"/>
@@ -20,4 +21,5 @@
   <xacro:property name="mode" value="$(arg mode)"/>
   <xacro:property name="model" value="$(arg model)"/>
+  <xacro:property name="update_rate" value="$(arg update_rate)"/>
   <xacro:if value="${cr == 'white'}">
      <xacro:include filename="$(find dsr_description2)/xacro/macro.m1013.white.xacro" />
@@ -53,4 +55,5 @@
         mode="${mode}"
         model="${model}"
+        update_rate="${update_rate}"
       />
     </xacro:unless>
