Commit message: Add moveit_config_file for P3020

File: dsr_description2/ros2_control/p3020.ros2_control.xacro (robot description, xacro)
@@ -71,10 +71,10 @@
       <joint name="joint_4">
         <command_interface name="position">
-          <param name="min">{-2*pi}</param>
-          <param name="max">{2*pi}</param>
+          <param name="min">0.0</param>
+          <param name="max">0.0</param>
         </command_interface>
         <command_interface name="velocity">
-          <param name="min">-3.2</param>
-          <param name="max">3.2</param>
+          <param name="min">0.0</param>
+          <param name="max">0.0</param>
         </command_interface>
         <state_interface name="position">

File: dsr_description2/xacro/macro.p3020.white.xacro (robot description, xacro)
@@ -206,5 +206,5 @@
         </link>
         <!-- Joints -->
-        <joint name="joint_1" type="continuous">
+        <joint name="joint_1" type="revolute">
             <origin xyz="0 0 0"/>
             <parent link="base_link"/>
@@ -212,5 +212,5 @@
             <axis xyz="0 0 1"/>
         </joint>
-        <joint name="joint_2" type="continuous">
+        <joint name="joint_2" type="revolute">
             <origin xyz="0 0 0"/>
             <parent link="link_1"/>
@@ -218,5 +218,5 @@
             <axis xyz="0 1 0"/>
         </joint>
-        <joint name="joint_3" type="continuous">
+        <joint name="joint_3" type="revolute">
             <origin xyz="0 0 0"/>
             <parent link="link_2"/>
@@ -230,5 +230,5 @@
             <child link="link_4"/>
         </joint>
-        <joint name="joint_5" type="continuous">
+        <joint name="joint_5" type="revolute">
             <origin xyz="0 0 0"/>
             <parent link="link_4"/>
@@ -236,5 +236,5 @@
             <axis xyz="0 1 0"/>
         </joint>
-        <joint name="joint_6" type="continuous">
+        <joint name="joint_6" type="revolute">
             <origin xyz="0 0 0"/>
             <parent link="link_5"/>
