Commit message: Add readme file

File: dsr_description2/ros2_control/m0609.mj_ros2_control.xacro (robot description, xacro)
@@ -5,6 +5,6 @@
     <xacro:include filename="$(find dsr_description2)/config/macro.materials.xacro" />
     <xacro:property name="default_position_kp" value="2000" />
-    <xacro:property name="default_position_ki" value="1" />
-    <xacro:property name="default_position_kd" value="1" />
+    <xacro:property name="default_position_ki" value="10" />
+    <xacro:property name="default_position_kd" value="10" />
     <xacro:property name="default_position_i_max" value="1000" />
     <xacro:macro name="joint_pid_params" params="kp:=${default_position_kp} ki:=${default_position_ki} kd:=${default_position_kd} i_max:=${default_position_i_max}">

File: dsr_description2/ros2_control/m1013.mj_ros2_control.xacro (robot description, xacro)
@@ -4,7 +4,7 @@
     <xacro:include filename="$(find dsr_description2)/config/macro.transmission.xacro" />
     <xacro:include filename="$(find dsr_description2)/config/macro.materials.xacro" />
-    <xacro:property name="default_position_kp" value="3000" />
+    <xacro:property name="default_position_kp" value="2000" />
     <xacro:property name="default_position_ki" value="10" />
-    <xacro:property name="default_position_kd" value="20" />
+    <xacro:property name="default_position_kd" value="10" />
     <xacro:property name="default_position_i_max" value="1000" />
     <xacro:macro name="joint_pid_params" params="kp:=${default_position_kp} ki:=${default_position_ki} kd:=${default_position_kd} i_max:=${default_position_i_max}">
