Commit message: Add red dot and scene for checking.

File: dsr_description2/ros2_control/m1013.mj_ros2_control.xacro (robot description, xacro)
@@ -4,6 +4,6 @@
     <xacro:include filename="$(find dsr_description2)/config/macro.transmission.xacro" />
     <xacro:include filename="$(find dsr_description2)/config/macro.materials.xacro" />
-    <xacro:property name="default_position_kp" value="2000" />
-    <xacro:property name="default_position_ki" value="1" />
+    <xacro:property name="default_position_kp" value="1000" />
+    <xacro:property name="default_position_ki" value="10" />
     <xacro:property name="default_position_kd" value="20" />
     <xacro:property name="default_position_i_max" value="1000" />
@@ -15,5 +15,4 @@
         <command_interface name="position_pid"/>
     </xacro:macro>
-    <!-- 수정 필요 -->
     <xacro:macro name="m1013_mj_ros2_control" params="
     name:=m1013

Commit message: Erase useless file, small change in XML files for test.

File: dsr_description2/ros2_control/m1013.mj_ros2_control.xacro (robot description, xacro)
@@ -4,5 +4,5 @@
     <xacro:include filename="$(find dsr_description2)/config/macro.transmission.xacro" />
     <xacro:include filename="$(find dsr_description2)/config/macro.materials.xacro" />
-    <xacro:property name="default_position_kp" value="1000" />
+    <xacro:property name="default_position_kp" value="2000" />
     <xacro:property name="default_position_ki" value="10" />
     <xacro:property name="default_position_kd" value="20" />

Commit message: Remove test code for gripper launch

File: dsr_description2/ros2_control/m1013.mj_ros2_control.xacro (robot description, xacro)
@@ -4,5 +4,5 @@
     <xacro:include filename="$(find dsr_description2)/config/macro.transmission.xacro" />
     <xacro:include filename="$(find dsr_description2)/config/macro.materials.xacro" />
-    <xacro:property name="default_position_kp" value="2000" />
+    <xacro:property name="default_position_kp" value="3000" />
     <xacro:property name="default_position_ki" value="10" />
     <xacro:property name="default_position_kd" value="20" />

Commit message: Now everything can be set in the main launch. Merge default and gripper launch file, new modul 'build_scene' added. Fix slope demo STL. + extra change

File: dsr_description2/ros2_control/m1013.mj_ros2_control.xacro (robot description, xacro)
@@ -4,5 +4,5 @@
     <xacro:include filename="$(find dsr_description2)/config/macro.transmission.xacro" />
     <xacro:include filename="$(find dsr_description2)/config/macro.materials.xacro" />
-    <xacro:property name="default_position_kp" value="2000" />
+    <xacro:property name="default_position_kp" value="2500" />
     <xacro:property name="default_position_ki" value="10" />
     <xacro:property name="default_position_kd" value="10" />
