Commit message: Now support also H2017 blue, remove test example + extra tuning.

File: dsr_description2/ros2_control/h2017.mj_ros2_control.xacro (robot description, xacro)
@@ -1,10 +1,10 @@
 <?xml version="1.0" ?>
-<robot name="m0609" xmlns:xacro="http://ros.org/wiki/xacro">
+<robot name="h2017" xmlns:xacro="http://ros.org/wiki/xacro">
     <xacro:include filename="$(find dsr_description2)/config/macro.gazebo.xacro" />
     <xacro:include filename="$(find dsr_description2)/config/macro.transmission.xacro" />
     <xacro:include filename="$(find dsr_description2)/config/macro.materials.xacro" />
-    <xacro:property name="default_position_kp" value="2000" />
+    <xacro:property name="default_position_kp" value="5000" />
     <xacro:property name="default_position_ki" value="10" />
-    <xacro:property name="default_position_kd" value="10" />
+    <xacro:property name="default_position_kd" value="0.01" />
     <xacro:property name="default_position_i_max" value="1000" />
     <xacro:macro name="joint_pid_params" params="kp:=${default_position_kp} ki:=${default_position_ki} kd:=${default_position_kd} i_max:=${default_position_i_max}">
@@ -15,6 +15,6 @@
         <command_interface name="position_pid"/>
     </xacro:macro>
-    <xacro:macro name="m0609_mj_ros2_control" params="
-    name:=m0609
+    <xacro:macro name="h2017_mj_ros2_control" params="
+    name:=h2017
     namespace
     rate:=100
@@ -24,5 +24,5 @@
     port:=12345
     mode:=real
-    model:=m0609
+    model:=h2017
     gripper:=none
     mobile:=none
