Commit message: Tuned H2525, A0509, A0912

File: dsr_description2/ros2_control/a0912.mj_ros2_control.xacro (robot description, xacro)
@@ -4,5 +4,5 @@
     <xacro:include filename="$(find dsr_description2)/config/macro.transmission.xacro" />
     <xacro:include filename="$(find dsr_description2)/config/macro.materials.xacro" />
-    <xacro:property name="default_position_kp" value="2500" />
+    <xacro:property name="default_position_kp" value="3000" />
     <xacro:property name="default_position_ki" value="10" />
     <xacro:property name="default_position_kd" value="10" />

File: dsr_description2/ros2_control/h2515.mj_ros2_control.xacro (robot description, xacro)
@@ -4,7 +4,7 @@
     <xacro:include filename="$(find dsr_description2)/config/macro.transmission.xacro" />
     <xacro:include filename="$(find dsr_description2)/config/macro.materials.xacro" />
-    <xacro:property name="default_position_kp" value="2500" />
+    <xacro:property name="default_position_kp" value="4500" />
     <xacro:property name="default_position_ki" value="10" />
-    <xacro:property name="default_position_kd" value="10" />
+    <xacro:property name="default_position_kd" value="0.1" />
     <xacro:property name="default_position_i_max" value="1000" />
     <xacro:macro name="joint_pid_params" params="kp:=${default_position_kp} ki:=${default_position_ki} kd:=${default_position_kd} i_max:=${default_position_i_max}">
