Commit message: Refactor: Update p3020/a0509 configs and hardware interface
- Modified files related to p3020 and a0509 robot models

- Updated dsr_hw_interface2.cpp and dsr_controller2.cpp

- Planned to document xacro/URDF configuration changes in upcoming commits

File: dsr_description2/ros2_control/a0509.ros2_control.xacro (robot description, xacro)
@@ -13,4 +13,9 @@
   mobile:=none
   ">
+    <!--modified-->
+    <!-- Precompute pi-based values using xacro to avoid runtime parsing errors in ros2_control -->
+    <xacro:property name="double_pi" value="${2.0 * pi}"/>
+    <xacro:property name="neg_double_pi" value="${-2.0 * pi}"/>
+    <xacro:property name="neg_pi" value="${-1.0 * pi}"/>
     <ros2_control name="${name}" type="system">
       <hardware>
@@ -29,6 +34,6 @@
       <joint name="joint_1">
         <command_interface name="position">
-          <param name="min">{-2*pi}</param>
-          <param name="max">{2*pi}</param>
+          <param name="min">${neg_double_pi}</param>
+          <param name="max">${double_pi}</param>
         </command_interface>
         <command_interface name="velocity">
@@ -43,6 +48,6 @@
       <joint name="joint_2">
         <command_interface name="position">
-          <param name="min">{-2*pi}</param>
-          <param name="max">{2*pi}</param>
+          <param name="min">${neg_double_pi}</param>
+          <param name="max">${double_pi}</param>
         </command_interface>
         <command_interface name="velocity">
@@ -57,6 +62,6 @@
       <joint name="joint_3">
         <command_interface name="position">
-          <param name="min">{-pi}</param>
-          <param name="max">{pi}</param>
+          <param name="min">${neg_pi}</param>
+          <param name="max">${pi}</param>
         </command_interface>
         <command_interface name="velocity">
@@ -71,6 +76,6 @@
       <joint name="joint_4">
         <command_interface name="position">
-          <param name="min">{-2*pi}</param>
-          <param name="max">{2*pi}</param>
+          <param name="min">${neg_double_pi}</param>
+          <param name="max">${double_pi}</param>
         </command_interface>
         <command_interface name="velocity">
@@ -85,6 +90,6 @@
       <joint name="joint_5">
         <command_interface name="position">
-          <param name="min">{-2*pi}</param>
-          <param name="max">{2*pi}</param>
+          <param name="min">${neg_double_pi}</param>
+          <param name="max">${double_pi}</param>
         </command_interface>
         <command_interface name="velocity">
@@ -99,6 +104,6 @@
       <joint name="joint_6">
         <command_interface name="position">
-          <param name="min">{-2*pi}</param>
-          <param name="max">{2*pi}</param>
+          <param name="min">${neg_double_pi}</param>
+          <param name="max">${double_pi}</param>
         </command_interface>
         <command_interface name="velocity">

File: dsr_description2/ros2_control/p3020.ros2_control.xacro (robot description, xacro)
@@ -13,4 +13,9 @@
   mobile:=none
   ">
+    <!--modified-->
+    <!-- Precompute pi-based values using xacro to avoid runtime parsing errors in ros2_control -->
+    <xacro:property name="double_pi" value="${2.0 * pi}"/>
+    <xacro:property name="neg_double_pi" value="${-2.0 * pi}"/>
+    <xacro:property name="neg_pi" value="${-1.0 * pi}"/>
     <ros2_control name="${name}" type="system">
       <hardware>
@@ -29,6 +34,6 @@
       <joint name="joint_1">
         <command_interface name="position">
-          <param name="min">{-2*pi}</param>
-          <param name="max">{2*pi}</param>
+          <param name="min">${neg_double_pi}</param>
+          <param name="max">${double_pi}</param>
         </command_interface>
         <command_interface name="velocity">
@@ -43,6 +48,6 @@
       <joint name="joint_2">
         <command_interface name="position">
-          <param name="min">{-2*pi}</param>
-          <param name="max">{2*pi}</param>
+          <param name="min">${neg_double_pi}</param>
+          <param name="max">${double_pi}</param>
         </command_interface>
         <command_interface name="velocity">
@@ -57,6 +62,6 @@
       <joint name="joint_3">
         <command_interface name="position">
-          <param name="min">{-pi}</param>
-          <param name="max">{pi}</param>
+          <param name="min">${neg_pi}</param>
+          <param name="max">${pi}</param>
         </command_interface>
         <command_interface name="velocity">
@@ -69,12 +74,13 @@
         <state_interface name="velocity"/>
       </joint>
+<!--
       <joint name="joint_4">
         <command_interface name="position">
-          <param name="min">0.0</param>
-          <param name="max">0.0</param>
+          <param name="min">${neg_double_pi}</param>
+          <param name="max">${double_pi}</param>
         </command_interface>
         <command_interface name="velocity">
-          <param name="min">0.0</param>
-          <param name="max">0.0</param>
+          <param name="min">-3.2</param>
+          <param name="max">3.2</param>
         </command_interface>
         <state_interface name="position">
@@ -83,8 +89,9 @@
         <state_interface name="velocity"/>
       </joint>
+-->
       <joint name="joint_5">
         <command_interface name="position">
-          <param name="min">{-2*pi}</param>
-          <param name="max">{2*pi}</param>
+          <param name="min">${neg_double_pi}</param>
+          <param name="max">${double_pi}</param>
         </command_interface>
         <command_interface name="velocity">
@@ -99,6 +106,6 @@
       <joint name="joint_6">
         <command_interface name="position">
-          <param name="min">{-2*pi}</param>
-          <param name="max">{2*pi}</param>
+          <param name="min">${neg_double_pi}</param>
+          <param name="max">${double_pi}</param>
         </command_interface>
         <command_interface name="velocity">

File: dsr_description2/xacro/macro.p3020.blue.xacro (robot description, xacro)
@@ -284,5 +284,5 @@
             <origin rpy="1.5708           0           0" xyz="0       -0.89           -0.1731"/>
             <axis xyz="0 0 1"/>
-            <!-- <limit effort="163" lower="0" upper="0" velocity="0"/> -->
+            <limit effort="163" lower="0" upper="0" velocity="0"/>
         </joint>
        <joint name="joint_5" type="revolute">

File: dsr_description2/xacro/macro.p3020.white.xacro (robot description, xacro)
@@ -275,5 +275,5 @@
             <origin rpy="1.5708           0           0" xyz="0       -0.89           -0.1731"/>
             <axis xyz="0 0 1"/>
-            <!-- <limit effort="163" lower="0" upper="0" velocity="0"/> -->
+            <limit effort="163" lower="0" upper="0" velocity="0"/>
         </joint>
        <joint name="joint_5" type="revolute">

Commit message: Refactoring codes

File: dsr_description2/ros2_control/a0509.ros2_control.xacro (robot description, xacro)
@@ -13,6 +13,4 @@
   mobile:=none
   ">
-    <!--modified-->
-    <!-- Precompute pi-based values using xacro to avoid runtime parsing errors in ros2_control -->
     <xacro:property name="double_pi" value="${2.0 * pi}"/>
     <xacro:property name="neg_double_pi" value="${-2.0 * pi}"/>

File: dsr_description2/ros2_control/h2515.ros2_control.xacro (robot description, xacro)
@@ -69,5 +69,5 @@
         <state_interface name="position">
           <param name="initial_value">0.0</param>
-        </state_interface> <!-- FIXED: missing closing tag -->
+        </state_interface>
         <state_interface name="velocity"/>
       </joint>

File: dsr_description2/ros2_control/m1013.ros2_control.xacro (robot description, xacro)
@@ -13,6 +13,4 @@
     mobile:=none
   ">
-    <!--gijungnam-->
-    <!-- Precompute pi-based values using xacro to avoid runtime parsing errors in ros2_control -->
     <xacro:property name="double_pi" value="${2.0 * pi}"/>
     <xacro:property name="neg_double_pi" value="${-2.0 * pi}"/>

File: dsr_description2/ros2_control/p3020.ros2_control.xacro (robot description, xacro)
@@ -13,6 +13,4 @@
   mobile:=none
   ">
-    <!--modified-->
-    <!-- Precompute pi-based values using xacro to avoid runtime parsing errors in ros2_control -->
     <xacro:property name="double_pi" value="${2.0 * pi}"/>
     <xacro:property name="neg_double_pi" value="${-2.0 * pi}"/>

File: dsr_description2/xacro/macro.p3020.blue.xacro (robot description, xacro)
@@ -284,5 +284,5 @@
             <origin rpy="1.5708           0           0" xyz="0       -0.89           -0.1731"/>
             <axis xyz="0 0 1"/>
-            <limit effort="163" lower="0" upper="0" velocity="0"/>
+            <!--<limit effort="163" lower="0" upper="0" velocity="0"/>-->
         </joint>
        <joint name="joint_5" type="revolute">

File: dsr_description2/xacro/macro.p3020.white.xacro (robot description, xacro)
@@ -275,5 +275,5 @@
             <origin rpy="1.5708           0           0" xyz="0       -0.89           -0.1731"/>
             <axis xyz="0 0 1"/>
-            <limit effort="163" lower="0" upper="0" velocity="0"/>
+            <!--<limit effort="163" lower="0" upper="0" velocity="0"/>-->
         </joint>
        <joint name="joint_5" type="revolute">
