Commit message: Update: gripper moveit

File: dsr_description2/ros2_control/robotiq.ros2_control.xacro (robot description, xacro)
@@ -5,4 +5,7 @@
   <xacro:arg name="mock_sensor_commands" default="true"/>
   <xacro:arg name="com_port" default="/dev/ttyUSB0"/>
+  <!-- 조인트/시스템 이름을 파라미터화 (프리픽스 대응) -->
+  <xacro:arg name="joint_name"  default="robotiq_85_left_knuckle_joint"/>
+  <xacro:arg name="system_name" default="robotiq_gripper_system"/>
   <xacro:arg name="pos_min" default="0.0"/>
   <xacro:arg name="pos_max" default="0.8"/>
@@ -15,4 +18,6 @@
       mode:=${mode}
       com_port:=${com_port}
+      joint_name:=${joint_name}
+      system_name:=${system_name}
       pos_min:=${pos_min}
       pos_max:=${pos_max}
@@ -23,7 +28,9 @@
       max_force:=${max_force}
       mock_sensor_commands:=${mock_sensor_commands}">
+    <!-- REAL: 실제 하드웨어 드라이버 -->
     <xacro:if value="${mode == 'real'}">
-      <ros2_control name="robotiq_gripper_system" type="system">
+      <ros2_control name="${system_name}" type="system">
         <hardware>
+          <!-- 실제 사용 드라이버 플러그인명 확인/수정 필요 -->
           <plugin>robotiq_driver/RobotiqGripperHardwareInterface</plugin>
           <param name="COM_port">${com_port}</param>
@@ -33,5 +40,5 @@
           <param name="gripper_max_force">${max_force}</param>
         </hardware>
-        <joint name="robotiq_85_left_knuckle_joint">
+        <joint name="${joint_name}">
           <command_interface name="position">
             <param name="min">${pos_min}</param>
@@ -45,6 +52,7 @@
       </ros2_control>
     </xacro:if>
+    <!-- VIRTUAL: 모의 하드웨어 -->
     <xacro:unless value="${mode == 'real'}">
-      <ros2_control name="robotiq_gripper_system" type="system">
+      <ros2_control name="${system_name}" type="system">
         <hardware>
           <plugin>mock_components/GenericSystem</plugin>
@@ -52,5 +60,5 @@
           <param name="state_following_offset">0.0</param>
         </hardware>
-        <joint name="robotiq_85_left_knuckle_joint">
+        <joint name="${joint_name}">
           <command_interface name="position">
             <param name="min">${pos_min}</param>

File: dsr_description2/xacro/m1013.urdf.xacro (robot description, xacro)
@@ -2,12 +2,18 @@
 <robot xmlns:xacro="http://www.ros.org/wiki/xacro" name="m1013">
   <xacro:arg name="mode" default="virtual"/>
+  <xacro:arg name="color" default="white"/>
+  <xacro:arg name="namespace" default=""/>
+  <!-- gripper 제어 인자 -->
+  <xacro:arg name="gripper" default="none"/>            <!-- none | robotique -->
+  <xacro:arg name="gripper_prefix" default=""/>         <!-- 멀티로봇 시 dsr01_ 등 -->
+  <xacro:arg name="gripper_parent_link" default="link_6"/>  <!-- 말단 프레임 기본값 -->
   <xacro:arg name="gripper_com_port" default="/dev/ttyUSB0"/>
-  <xacro:arg name="color"   default="white"/>
-  <xacro:arg name="gripper" default="none"/>
-  <xacro:arg name="namespace" default=""/>
+  <!-- Gazebo 분기 -->
   <xacro:arg name="use_gazebo" default="false"/>
   <xacro:property name="cr" value="$(arg color)"/>
-  <xacro:property name="gr" value="$(arg gripper)"/>
   <xacro:property name="gz" value="$(arg use_gazebo)"/>
+  <!-- 표현식에서 사용할 gripper 프로퍼티 (중요) -->
+  <xacro:property name="gripper" value="$(arg gripper)"/>
+  <!-- 본체 색상 -->
   <xacro:if value="${cr == 'white'}">
     <xacro:include filename="$(find dsr_description2)/xacro/macro.m1013.white.xacro"/>
@@ -17,5 +23,5 @@
   </xacro:if>
   <xacro:m1013 namespace="$(arg namespace)"/>
-  <!-- 월드 고정 -->
+  <!-- world 고정 -->
   <link name="world"/>
   <joint name="world_fixed" type="fixed">
@@ -24,4 +30,5 @@
     <child  link="base_link"/>
   </joint>
+  <!-- ros2_control (본체) -->
   <xacro:if value="${gz == 'true'}">
     <xacro:include filename="$(find dsr_description2)/ros2_control/m1013.gz_ros2_control.xacro"/>
@@ -32,223 +39,24 @@
     <xacro:m1013_ros2_control name="m1013"/>
   </xacro:unless>
-  <xacro:if value="${gr != 'none'}">
-    <link name="robotiq_85_base_link">
-    <visual>
-        <geometry>
-        <mesh filename="package://dsr_description2/meshes/gripper/robotiq/2f85/visual/robotiq_base.dae"/>
-        </geometry>
-    </visual>
-    <collision>
-        <geometry>
-        <mesh filename="package://dsr_description2/meshes/gripper/robotiq/2f85/collision/robotiq_base.stl"/>
-        </geometry>
-    </collision>
-    <inertial>
-        <origin xyz="0.0 2.274e-05 0.03232288" rpy="0 0 0"/>
-        <mass value="6.6320197e-01"/>
-        <inertia ixx="5.1617816e-04" iyy="5.8802208e-04" izz="3.9462776e-04" ixy="2.936e-8" ixz="0.0" iyz="-3.2296e-7"/>
-    </inertial>
-    </link>
-    <link name="robotiq_85_left_knuckle_link">
-    <visual>
-        <geometry>
-        <mesh filename="package://dsr_description2/meshes/gripper/robotiq/2f85/visual/left_knuckle.dae"/>
-        </geometry>
-    </visual>
-    <collision>
-        <geometry>
-        <mesh filename="package://dsr_description2/meshes/gripper/robotiq/2f85/collision/left_knuckle.stl"/>
-        </geometry>
-    </collision>
-    <inertial>
-        <origin xyz="0.01213197 0.0002 -0.00058647" rpy="0 0 0"/>
-        <mass value="1.384773208e-02"/>
-        <inertia ixx="3.5232e-7" iyy="2.31944e-6" izz="2.23136e-6" ixy="0.0" ixz="1.1744e-7" iyz="0"/>
-    </inertial>
-    </link>
-    <link name="robotiq_85_right_knuckle_link">
-    <visual>
-        <geometry>
-        <mesh filename="package://dsr_description2/meshes/gripper/robotiq/2f85/visual/right_knuckle.dae"/>
-        </geometry>
-    </visual>
-    <collision>
-        <geometry>
-        <mesh filename="package://dsr_description2/meshes/gripper/robotiq/2f85/collision/right_knuckle.stl"/>
-        </geometry>
-    </collision>
-    <inertial>
-        <origin xyz="-0.01213197 0.0002 -0.00058647" rpy="0 0 0"/>
-        <mass value="1.384773208e-02"/>
-        <inertia ixx="3.5232e-7" iyy="2.31944e-6" izz="2.23136e-6" ixy="0.0" ixz="-1.1744e-7" iyz="0.0"/>
-    </inertial>
-    </link>
-    <link name="robotiq_85_left_finger_link">
-    <visual>
-        <geometry>
-        <mesh filename="package://dsr_description2/meshes/gripper/robotiq/2f85/visual/left_finger.dae"/>
-        </geometry>
-    </visual>
-    <collision>
-        <geometry>
-        <mesh filename="package://dsr_description2/meshes/gripper/robotiq/2f85/collision/left_finger.stl"/>
-        </geometry>
-    </collision>
-    <inertial>
-        <origin xyz="0.00346899 -0.00079447 0.01867121" rpy="0 0 0"/>
-        <mass value="4.260376752e-02"/>
-        <inertia ixx="1.385792000000000e-05" iyy="1.183208e-05" izz="5.19672e-06" ixy="0.0" ixz="-2.17264e-06" iyz="0.0"/>
-    </inertial>
-    </link>
-    <link name="robotiq_85_right_finger_link">
-    <visual>
-        <geometry>
-        <mesh filename="package://dsr_description2/meshes/gripper/robotiq/2f85/visual/right_finger.dae"/>
-        </geometry>
-    </visual>
-    <collision>
-        <geometry>
-        <mesh filename="package://dsr_description2/meshes/gripper/robotiq/2f85/collision/right_finger.stl"/>
-        </geometry>
-    </collision>
-    <inertial>
-        <origin xyz="-0.00346899 -5.53e-06 0.01867121" rpy="0 0 0"/>
-        <mass value="4.260376752000000e-02"/>
-        <inertia ixx="1.385792e-05" iyy="1.183208e-05" izz="5.19672e-06" ixy="0.0" ixz="2.17264e-06" iyz="0.0"/>
-    </inertial>
-    </link>
-    <link name="robotiq_85_left_inner_knuckle_link">
-    <visual>
-        <geometry>
-        <mesh filename="package://dsr_description2/meshes/gripper/robotiq/2f85/visual/left_inner_knuckle.dae"/>
-        </geometry>
-    </visual>
-    <collision>
-        <geometry>
-        <mesh filename="package://dsr_description2/meshes/gripper/robotiq/2f85/collision/left_inner_knuckle.stl"/>
-        </geometry>
-    </collision>
-    <inertial>
-        <origin xyz="0.01897699 0.00015001 0.02247101" rpy="0 0 0"/>
-        <mass value="2.969376448e-02"/>
-        <inertia ixx="9.57136e-06" iyy="8.69056e-06" izz="8.19144e-06" ixy="0.0" ixz="-3.93424e-06" iyz="0.0"/>
-    </inertial>
-    </link>
-    <link name="robotiq_85_right_inner_knuckle_link">
-    <visual>
-        <geometry>
-        <mesh filename="package://dsr_description2/meshes/gripper/robotiq/2f85/visual/right_inner_knuckle.dae"/>
-        </geometry>
-    </visual>
-    <collision>
-        <geometry>
-        <mesh filename="package://dsr_description2/meshes/gripper/robotiq/2f85/collision/right_inner_knuckle.stl"/>
-        </geometry>
-    </collision>
-    <inertial>
-        <origin xyz="-0.01926824 5.001e-05 0.02222178" rpy="0 0 0"/>
-        <mass value="2.969376448e-02"/>
-        <inertia ixx="9.42456e-06" iyy="8.69056e-06" izz="8.33824e-06" ixy="0.0" ixz="3.9636e-06" iyz="0.0"/>
-    </inertial>
-    </link>
-    <link name="robotiq_85_left_finger_tip_link">
-    <visual>
-        <geometry>
-        <mesh filename="package://dsr_description2/meshes/gripper/robotiq/2f85/visual/left_finger_tip.dae"/>
-        </geometry>
-    </visual>
-    <collision>
-        <geometry>
-        <mesh filename="package://dsr_description2/meshes/gripper/robotiq/2f85/collision/left_finger_tip.stl"/>
-        </geometry>
-    </collision>
-    <inertial>
-        <origin xyz="-0.01456706 -0.0008 0.01649701" rpy="0 0 0"/>
-        <mass value="4.268588744e-02"/>
-        <inertia ixx="1.048152e-05" iyy="1.197888e-05" izz="4.22784e-06" ixy="0.0" ixz="3.5232e-6" iyz="0.0"/>
-    </inertial>
-    </link>
-    <link name="robotiq_85_right_finger_tip_link">
-    <visual>
-        <geometry>
-        <mesh filename="package://dsr_description2/meshes/gripper/robotiq/2f85/visual/right_finger_tip.dae"/>
-        </geometry>
-    </visual>
-    <collision>
-        <geometry>
-        <mesh filename="package://dsr_description2/meshes/gripper/robotiq/2f85/collision/right_finger_tip.stl"/>
-        </geometry>
-    </collision>
-    <inertial>
-        <origin xyz="0.01456706 5e-05 0.01649701" rpy="0 0 0"/>
-        <mass value="4.268588744e-02"/>
-        <inertia ixx="1.048152e-05" iyy="1.197888e-05" izz="4.22784e-06" ixy="0.0" ixz="-3.5232e-06" iyz="0.0"/>
-    </inertial>
-    </link>
-    <!-- ===== Robotiq 2F-85 조인트들 ===== -->
-    <joint name="robotiq_85_base_joint" type="fixed">
-    <parent link="link_6"/>
-    <child  link="robotiq_85_base_link"/>
-    <origin xyz="0 0 0.0" rpy="0 0 0"/>
-    </joint>
-    <joint name="robotiq_85_left_knuckle_joint" type="revolute">
-    <parent link="robotiq_85_base_link"/>
-    <child  link="robotiq_85_left_knuckle_link"/>
-    <axis xyz="0 -1 0"/>
-    <origin xyz="0.03060114 0.0 0.05490452" rpy="0 0 0"/>
-    <limit lower="0.0" upper="0.8" velocity="0.5" effort="50"/>
-    </joint>
-    <joint name="robotiq_85_right_knuckle_joint" type="revolute">
-    <parent link="robotiq_85_base_link"/>
-    <child  link="robotiq_85_right_knuckle_link"/>
-    <axis xyz="0 -1 0"/>
-    <origin xyz="-0.03060114 0.0 0.05490452" rpy="0 0 0"/>
-    <limit lower="-0.8" upper="0.0" velocity="0.5" effort="50"/>
-    <mimic joint="robotiq_85_left_knuckle_joint" multiplier="-1"/>
-    </joint>
-    <joint name="robotiq_85_left_finger_joint" type="fixed">
-    <parent link="robotiq_85_left_knuckle_link"/>
-    <child  link="robotiq_85_left_finger_link"/>
-    <origin xyz="0.03152616 0.0 -0.00376347" rpy="0 0 0"/>
-    </joint>
-    <joint name="robotiq_85_right_finger_joint" type="fixed">
-    <parent link="robotiq_85_right_knuckle_link"/>
-    <child  link="robotiq_85_right_finger_link"/>
-    <origin xyz="-0.03152616 0.0 -0.00376347" rpy="0 0 0"/>
-    </joint>
-    <joint name="robotiq_85_left_inner_knuckle_joint" type="continuous">
-    <parent link="robotiq_85_base_link"/>
-    <child  link="robotiq_85_left_inner_knuckle_link"/>
-    <axis xyz="0 -1 0"/>
-    <origin xyz="0.0127 0.0 0.06142" rpy="0 0 0"/>
-    <mimic joint="robotiq_85_left_knuckle_joint"/>
-    </joint>
-    <joint name="robotiq_85_right_inner_knuckle_joint" type="continuous">
-    <parent link="robotiq_85_base_link"/>
-    <child  link="robotiq_85_right_inner_knuckle_link"/>
-    <axis xyz="0 -1 0"/>
-    <origin xyz="-0.0127 0.0 0.06142" rpy="0 0 0"/>
-    <mimic joint="robotiq_85_left_knuckle_joint" multiplier="-1"/>
-    </joint>
-    <joint name="robotiq_85_left_finger_tip_joint" type="continuous">
-    <parent link="robotiq_85_left_finger_link"/>
-    <child  link="robotiq_85_left_finger_tip_link"/>
-    <axis xyz="0 -1 0"/>
-    <origin xyz="0.00563134 0.0 0.04718515" rpy="0 0 0"/>
-    <mimic joint="robotiq_85_left_knuckle_joint" multiplier="-1"/>
-    </joint>
-    <joint name="robotiq_85_right_finger_tip_joint" type="continuous">
-    <parent link="robotiq_85_right_finger_link"/>
-    <child  link="robotiq_85_right_finger_tip_link"/>
-    <axis xyz="0 -1 0"/>
-    <origin xyz="-0.00563134 0.0 0.04718515" rpy="0 0 0"/>
-    <mimic joint="robotiq_85_left_knuckle_joint"/>
-    </joint>
-    <!-- ros2_control system for Robotiq gripper -->
+  <!-- === Gripper (조건부) === -->
+  <xacro:if value="${gripper == 'robotique'}">
+    <!-- 2F-85 기구부 -->
+    <xacro:include filename="$(find dsr_description2)/xacro/robotiq_85.xacro"/>
+    <xacro:robotiq_85 parent="$(arg gripper_parent_link)" prefix="$(arg gripper_prefix)"/>
+    <!-- ros2_control system for Robotiq -->
     <xacro:include filename="$(find dsr_description2)/ros2_control/robotiq.ros2_control.xacro"/>
     <xacro:robotiq_gripper_system
-    mode="$(arg mode)"
-    com_port="$(arg gripper_com_port)"
-    pos_min="0.0" pos_max="0.8" init_pos="0.0"/>
+        mode="$(arg mode)"
+        com_port="$(arg gripper_com_port)"
+        joint_name="$(arg gripper_prefix)robotiq_85_left_knuckle_joint"
+        system_name="$(arg gripper_prefix)robotiq_gripper_system"
+        pos_min="0.0"
+        pos_max="0.8"
+        init_pos="0.0"
+        speed_mult="1.0"
+        force_mult="0.5"
+        max_speed="0.150"
+        max_force="235.0"
+        mock_sensor_commands="true" />
   </xacro:if>
 </robot>
