Commit message: Try to control 2f85 gripper, changing from bringup rviz2

File: dsr_description2/ros2_control/m1013.ros2_control.xacro (robot description, xacro)
@@ -46,5 +46,6 @@
           <param name="min">${neg_double_pi}</param>
           <param name="max">${double_pi}</param>
-        </command_interface>
+        </command_interface
+        >
         <command_interface name="velocity">
           <param name="min">-3.15</param>

File: dsr_description2/xacro/m1013.urdf.xacro (robot description, xacro)
@@ -15,4 +15,217 @@
   </xacro:if>
   <xacro:m1013 namespace="$(arg namespace)"/>
+  <!-- Robotiq 2F-85 Gripper -->
+  <link name="robotiq_85_base_link">
+      <visual>
+          <geometry>
+              <mesh filename="package://dsr_description2/meshes/gripper/robotiq/2f85/visual/robotiq_base.dae" />
+          </geometry>
+      </visual>
+      <collision>
+          <geometry>
+              <mesh filename="package://dsr_description2/meshes/gripper/robotiq/2f85/collision/robotiq_base.stl" />
+          </geometry>
+      </collision>
+      <inertial>
+          <origin xyz="0.0 2.274e-05 0.03232288" rpy="0 0 0" />
+          <mass value="6.6320197e-01" />
+          <inertia ixx="5.1617816e-04" iyy="5.8802208e-04" izz="3.9462776e-04" ixy="2.936e-8" ixz="0.0" iyz="-3.2296e-7" />
+      </inertial>
+  </link>
+  <link name="robotiq_85_left_knuckle_link">
+      <visual>
+          <geometry>
+              <mesh filename="package://dsr_description2/meshes/gripper/robotiq/2f85/visual/left_knuckle.dae" />
+          </geometry>
+      </visual>
+      <collision>
+          <geometry>
+              <mesh filename="package://dsr_description2/meshes/gripper/robotiq/2f85/collision/left_knuckle.stl" />
+          </geometry>
+      </collision>
+      <inertial>
+          <origin xyz="0.01213197 0.0002 -0.00058647" rpy="0 0 0" />
+          <mass value="1.384773208e-02" />
+          <inertia ixx="3.5232e-7" iyy="2.31944e-6" izz="2.23136e-6" ixy="0.0" ixz="1.1744e-7" iyz="0" />
+      </inertial>
+  </link>
+  <link name="robotiq_85_right_knuckle_link">
+      <visual>
+          <geometry>
+              <mesh filename="package://dsr_description2/meshes/gripper/robotiq/2f85/visual/right_knuckle.dae" />
+          </geometry>
+      </visual>
+      <collision>
+          <geometry>
+              <mesh filename="package://dsr_description2/meshes/gripper/robotiq/2f85/collision/right_knuckle.stl" />
+          </geometry>
+      </collision>
+      <inertial>
+          <origin xyz="-0.01213197 0.0002 -0.00058647" rpy="0 0 0" />
+          <mass value="1.384773208e-02" />
+          <inertia ixx="3.5232e-7" iyy="2.31944e-6" izz="2.23136e-6" ixy="0.0" ixz="-1.1744e-7" iyz="0.0" />
+      </inertial>
+  </link>
+  <link name="robotiq_85_left_finger_link">
+      <visual>
+          <geometry>
+              <mesh filename="package://dsr_description2/meshes/gripper/robotiq/2f85/visual/left_finger.dae" />
+          </geometry>
+      </visual>
+      <collision>
+          <geometry>
+              <mesh filename="package://dsr_description2/meshes/gripper/robotiq/2f85/collision/left_finger.stl" />
+          </geometry>
+      </collision>
+      <inertial>
+          <origin xyz="0.00346899 -0.00079447 0.01867121" rpy="0 0 0" />
+          <mass value="4.260376752e-02" />
+          <inertia ixx="1.385792000000000e-05" iyy="1.183208e-05" izz="5.19672e-06" ixy="0.0" ixz="-2.17264e-06" iyz="0.0" />
+      </inertial>
+  </link>
+  <link name="robotiq_85_right_finger_link">
+      <visual>
+          <geometry>
+              <mesh filename="package://dsr_description2/meshes/gripper/robotiq/2f85/visual/right_finger.dae" />
+          </geometry>
+      </visual>
+      <collision>
+          <geometry>
+              <mesh filename="package://dsr_description2/meshes/gripper/robotiq/2f85/collision/right_finger.stl" />
+          </geometry>
+      </collision>
+      <inertial>
+          <origin xyz="-0.00346899 -5.53e-06 0.01867121" rpy="0 0 0" />
+          <mass value="4.260376752000000e-02" />
+          <inertia ixx="1.385792e-05" iyy="1.183208e-05" izz="5.19672e-06" ixy="0.0" ixz="2.17264e-06" iyz="0.0" />
+      </inertial>
+  </link>
+  <link name="robotiq_85_left_inner_knuckle_link">
+      <visual>
+          <geometry>
+              <mesh filename="package://dsr_description2/meshes/gripper/robotiq/2f85/visual/left_inner_knuckle.dae" />
+          </geometry>
+      </visual>
+      <collision>
+          <geometry>
+              <mesh filename="package://dsr_description2/meshes/gripper/robotiq/2f85/collision/left_inner_knuckle.stl" />
+          </geometry>
+      </collision>
+      <inertial>
+          <origin xyz="0.01897699 0.00015001 0.02247101" rpy="0 0 0" />
+          <mass value="2.969376448e-02" />
+          <inertia ixx="9.57136e-06" iyy="8.69056e-06" izz="8.19144e-06" ixy="0.0" ixz="-3.93424e-06" iyz="0.0" />
+      </inertial>
+  </link>
+  <link name="robotiq_85_right_inner_knuckle_link">
+      <visual>
+          <geometry>
+              <mesh filename="package://dsr_description2/meshes/gripper/robotiq/2f85/visual/right_inner_knuckle.dae" />
+          </geometry>
+      </visual>
+      <collision>
+          <geometry>
+              <mesh filename="package://dsr_description2/meshes/gripper/robotiq/2f85/collision/right_inner_knuckle.stl" />
+          </geometry>
+      </collision>
+      <inertial>
+          <origin xyz="-0.01926824 5.001e-05 0.02222178" rpy="0 0 0" />
+          <mass value="2.969376448e-02" />
+          <inertia ixx="9.42456e-06" iyy="8.69056e-06" izz="8.33824e-06" ixy="0.0" ixz="3.9636e-06" iyz="0.0" />
+      </inertial>
+  </link>
+  <link name="robotiq_85_left_finger_tip_link">
+      <visual>
+          <geometry>
+              <mesh filename="package://dsr_description2/meshes/gripper/robotiq/2f85/visual/left_finger_tip.dae" />
+          </geometry>
+      </visual>
+      <collision>
+          <geometry>
+              <mesh filename="package://dsr_description2/meshes/gripper/robotiq/2f85/collision/left_finger_tip.stl" />
+          </geometry>
+      </collision>
+      <inertial>
+          <origin xyz="-0.01456706 -0.0008 0.01649701" rpy="0 0 0" />
+          <mass value="4.268588744e-02" />
+          <inertia ixx="1.048152e-05" iyy="1.197888e-05" izz="4.22784e-06" ixy="0.0" ixz="3.5232e-6" iyz="0.0" />
+      </inertial>
+  </link>
+  <link name="robotiq_85_right_finger_tip_link">
+      <visual>
+          <geometry>
+              <mesh filename="package://dsr_description2/meshes/gripper/robotiq/2f85/visual/right_finger_tip.dae" />
+          </geometry>
+      </visual>
+      <collision>
+          <geometry>
+              <mesh filename="package://dsr_description2/meshes/gripper/robotiq/2f85/collision/right_finger_tip.stl" />
+          </geometry>
+      </collision>
+      <inertial>
+          <origin xyz="0.01456706 5e-05 0.01649701" rpy="0 0 0" />
+          <mass value="4.268588744e-02" />
+          <inertia ixx="1.048152e-05" iyy="1.197888e-05" izz="4.22784e-06" ixy="0.0" ixz="-3.5232e-06" iyz="0.0" />
+      </inertial>
+  </link>
+  <joint name="robotiq_85_base_joint" type="fixed">
+      <parent link="link_6" />
+      <child link="robotiq_85_base_link" />
+      <origin xyz="0 0 0.0" rpy="0 0 0"/>
+  </joint>
+  <joint name="robotiq_85_left_knuckle_joint" type="revolute">
+      <parent link="robotiq_85_base_link" />
+      <child link="robotiq_85_left_knuckle_link" />
+      <axis xyz="0 -1 0" />
+      <origin xyz="0.03060114 0.0 0.05490452" rpy="0 0 0" />
+      <limit lower="0.0" upper="0.8" velocity="0.5" effort="50" />
+  </joint>
+  <joint name="robotiq_85_right_knuckle_joint" type="revolute">
+      <parent link="robotiq_85_base_link" />
+      <child link="robotiq_85_right_knuckle_link" />
+      <axis xyz="0 -1 0" />
+      <origin xyz="-0.03060114 0.0 0.05490452" rpy="0 0 0" />
+      <limit lower="-0.8" upper="0.0" velocity="0.5" effort="50" />
+      <mimic joint="robotiq_85_left_knuckle_joint" multiplier="-1" />
+  </joint>
+  <joint name="robotiq_85_left_finger_joint" type="fixed">
+      <parent link="robotiq_85_left_knuckle_link" />
+      <child link="robotiq_85_left_finger_link" />
+      <origin xyz="0.03152616 0.0 -0.00376347" rpy="0 0 0" />
+  </joint>
+  <joint name="robotiq_85_right_finger_joint" type="fixed">
+      <parent link="robotiq_85_right_knuckle_link" />
+      <child link="robotiq_85_right_finger_link" />
+      <origin xyz="-0.03152616 0.0 -0.00376347" rpy="0 0 0" />
+  </joint>
+  <joint name="robotiq_85_left_inner_knuckle_joint" type="continuous">
+      <parent link="robotiq_85_base_link" />
+      <child link="robotiq_85_left_inner_knuckle_link" />
+      <axis xyz="0 -1 0" />
+      <origin xyz="0.0127 0.0 0.06142" rpy="0 0 0" />
+      <mimic joint="robotiq_85_left_knuckle_joint" />
+  </joint>
+  <joint name="robotiq_85_right_inner_knuckle_joint" type="continuous">
+      <parent link="robotiq_85_base_link" />
+      <child link="robotiq_85_right_inner_knuckle_link" />
+      <axis xyz="0 -1 0" />
+      <origin xyz="-0.0127 0.0 0.06142" rpy="0 0 0" />
+      <mimic joint="robotiq_85_left_knuckle_joint" multiplier="-1" />
+  </joint>
+  <joint name="robotiq_85_left_finger_tip_joint" type="continuous">
+      <parent link="robotiq_85_left_finger_link" />
+      <child link="robotiq_85_left_finger_tip_link" />
+      <axis xyz="0 -1 0" />
+      <origin xyz="0.00563134 0.0 0.04718515" rpy="0 0 0" />
+      <mimic joint="robotiq_85_left_knuckle_joint" multiplier="-1" />
+  </joint>
+  <joint name="robotiq_85_right_finger_tip_joint" type="continuous">
+      <parent link="robotiq_85_right_finger_link" />
+      <child link="robotiq_85_right_finger_tip_link" />
+      <axis xyz="0 -1 0" />
+      <origin xyz="-0.00563134 0.0 0.04718515" rpy="0 0 0" />
+      <mimic joint="robotiq_85_left_knuckle_joint" />
+  </joint>
+  <!-- End Robotiq 2F-85 Gripper -->
   <link name="world"/>
   <!-- World fixed joint-->
@@ -29,4 +242,18 @@
     <xacro:include filename="$(find dsr_description2)/ros2_control/m1013.ros2_control.xacro" />
     <xacro:m1013_ros2_control name="m1013"/>
+    <!-- Add a separate ros2_control for the gripper -->
+    <ros2_control name="RobotiqGripper" type="system">
+        <hardware>
+            <plugin>mock_components/GenericSystem</plugin>
+        </hardware>
+        <joint name="robotiq_85_left_knuckle_joint">
+            <command_interface name="position">
+                <param name="min">0.0</param>
+                <param name="max">0.8</param>
+            </command_interface>
+            <state_interface name="position"/>
+            <state_interface name="velocity"/>
+        </joint>
+    </ros2_control>
   </xacro:unless>
 </robot>

Commit message: Succeed to move gripper in rviz2 launch

File: dsr_description2/ros2_control/m1013.ros2_control.xacro (robot description, xacro)
@@ -37,6 +37,6 @@
         </command_interface>
         <command_interface name="velocity">
-          <param name="min">-3.15</param>
-          <param name="max">3.15</param>
+          <param name="min">-3.2</param>
+          <param name="max">3.2</param>
         </command_interface>
         <state_interface name="position"><param name="initial_value">0.0</param></state_interface>
@@ -47,9 +47,8 @@
           <param name="min">${neg_double_pi}</param>
           <param name="max">${double_pi}</param>
-        </command_interface
-        >
+        </command_interface>
         <command_interface name="velocity">
-          <param name="min">-3.15</param>
-          <param name="max">3.15</param>
+          <param name="min">-3.2</param>
+          <param name="max">3.2</param>
         </command_interface>
         <state_interface name="position"><param name="initial_value">0.0</param></state_interface>
@@ -58,10 +57,10 @@
       <joint name="joint_3">
         <command_interface name="position">
-          <param name="min">${neg_pi}</param>
-          <param name="max">${pi}</param>
+          <param name="min">${neg_double_pi}</param>
+          <param name="max">${double_pi}</param>
         </command_interface>
         <command_interface name="velocity">
-          <param name="min">-3.15</param>
-          <param name="max">3.15</param>
+          <param name="min">-3.2</param>
+          <param name="max">3.2</param>
         </command_interface>
         <state_interface name="position"><param name="initial_value">0.0</param></state_interface>
@@ -104,4 +103,13 @@
         <state_interface name="velocity"/>
       </joint>
+      <!-- Add gripper joint with proper interfaces -->
+      <joint name="robotiq_85_left_knuckle_joint">
+        <command_interface name="position">
+          <param name="min">0.0</param>
+          <param name="max">0.8</param>
+        </command_interface>
+        <state_interface name="position"><param name="initial_value">0.0</param></state_interface>
+        <state_interface name="velocity"/>
+      </joint>
     </ros2_control>
   </xacro:macro>

File: dsr_description2/xacro/m1013.urdf.xacro (robot description, xacro)
@@ -242,20 +242,4 @@
     <xacro:include filename="$(find dsr_description2)/ros2_control/m1013.ros2_control.xacro" />
     <xacro:m1013_ros2_control name="m1013"/>
-    <!-- Add a separate ros2_control for the gripper -->
-    <ros2_control name="RobotiqGripper" type="system">
-        <hardware>
-            <plugin>mock_components/GenericSystem</plugin>
-            <param name="mock_sensor_commands">true</param>
-            <param name="state_following_offset">0.0</param>
-        </hardware>
-        <joint name="robotiq_85_left_knuckle_joint">
-            <command_interface name="position">
-                <param name="min">0.0</param>
-                <param name="max">0.8</param>
-            </command_interface>
-            <state_interface name="position"/>
-            <state_interface name="velocity"/>
-        </joint>
-    </ros2_control>
   </xacro:unless>
 </robot>
