Commit message: hardware and xacro file modified

File: dsr_description2/ros2_control/m1013.ros2_control.xacro (robot description, xacro)
@@ -1,22 +1,21 @@
 <?xml version="1.0"?>
 <robot xmlns:xacro="http://www.ros.org/wiki/xacro">
+  <!-- Doosan M1013 ros2_control (arm-only) -->
   <xacro:macro name="m1013_ros2_control" params="
-    name
-    rate:=100
-    standby:=true
-    command:=none
-    host:=0.0.0.0
-    port:=12345
-    mode:=real
-    model:=m1013
-    gripper:=none
-    mobile:=none
-  ">
+      name
+      rate:=100
+      standby:=true
+      command:=none
+      host:=127.0.0.1
+      port:=12345
+      mode:=virtual
+      model:=m1013
+      mobile:=none">
     <xacro:property name="double_pi" value="${2.0 * pi}"/>
     <xacro:property name="neg_double_pi" value="${-2.0 * pi}"/>
-    <xacro:property name="neg_pi" value="${-1.0 * pi}"/>
     <ros2_control name="${name}" type="system">
       <hardware>
         <plugin>dsr_hardware2/DRHWInterface</plugin>
+        <!-- virtual 테스트면 true 유지 가능 (실기면 false 권장) -->
         <param name="use_mock_hardware">true</param>
         <param name="name">${name}</param>
@@ -28,7 +27,7 @@
         <param name="mode">${mode}</param>
         <param name="model">${model}</param>
-        <param name="gripper">${gripper}</param>
         <param name="mobile">${mobile}</param>
       </hardware>
+      <!-- Arm joints only -->
       <joint name="joint_1">
         <command_interface name="position">
@@ -103,13 +102,4 @@
         <state_interface name="velocity"/>
       </joint>
-      <!-- Add gripper joint with proper interfaces -->
-      <joint name="robotiq_85_left_knuckle_joint">
-        <command_interface name="position">
-          <param name="min">0.0</param>
-          <param name="max">0.8</param>
-        </command_interface>
-        <state_interface name="position"><param name="initial_value">0.0</param></state_interface>
-        <state_interface name="velocity"/>
-      </joint>
     </ros2_control>
   </xacro:macro>

File: dsr_description2/xacro/m1013.urdf.xacro (robot description, xacro)
@@ -1,4 +1,6 @@
 <?xml version="1.0"?>
-<robot xmlns:xacro="http://www.ros.org/wiki/xacro" name="m1013" >
+<robot xmlns:xacro="http://www.ros.org/wiki/xacro" name="m1013">
+  <xacro:arg name="mode" default="virtual"/>
+  <xacro:arg name="gripper_com_port" default="/dev/ttyUSB0"/>
   <xacro:arg name="color"   default="white"/>
   <xacro:arg name="gripper" default="none"/>
@@ -9,237 +11,244 @@
   <xacro:property name="gz" value="$(arg use_gazebo)"/>
   <xacro:if value="${cr == 'white'}">
-     <xacro:include filename="$(find dsr_description2)/xacro/macro.m1013.white.xacro" />
+    <xacro:include filename="$(find dsr_description2)/xacro/macro.m1013.white.xacro"/>
   </xacro:if>
   <xacro:if value="${cr == 'blue'}">
-     <xacro:include filename="$(find dsr_description2)/xacro/macro.m1013.blue.xacro" />
+    <xacro:include filename="$(find dsr_description2)/xacro/macro.m1013.blue.xacro"/>
   </xacro:if>
   <xacro:m1013 namespace="$(arg namespace)"/>
-  <!-- Robotiq 2F-85 Gripper -->
-  <link name="robotiq_85_base_link">
-      <visual>
-          <geometry>
-              <mesh filename="package://dsr_description2/meshes/gripper/robotiq/2f85/visual/robotiq_base.dae" />
-          </geometry>
-      </visual>
-      <collision>
-          <geometry>
-              <mesh filename="package://dsr_description2/meshes/gripper/robotiq/2f85/collision/robotiq_base.stl" />
-          </geometry>
-      </collision>
-      <inertial>
-          <origin xyz="0.0 2.274e-05 0.03232288" rpy="0 0 0" />
-          <mass value="6.6320197e-01" />
-          <inertia ixx="5.1617816e-04" iyy="5.8802208e-04" izz="3.9462776e-04" ixy="2.936e-8" ixz="0.0" iyz="-3.2296e-7" />
-      </inertial>
-  </link>
-  <link name="robotiq_85_left_knuckle_link">
-      <visual>
-          <geometry>
-              <mesh filename="package://dsr_description2/meshes/gripper/robotiq/2f85/visual/left_knuckle.dae" />
-          </geometry>
-      </visual>
-      <collision>
-          <geometry>
-              <mesh filename="package://dsr_description2/meshes/gripper/robotiq/2f85/collision/left_knuckle.stl" />
-          </geometry>
-      </collision>
-      <inertial>
-          <origin xyz="0.01213197 0.0002 -0.00058647" rpy="0 0 0" />
-          <mass value="1.384773208e-02" />
-          <inertia ixx="3.5232e-7" iyy="2.31944e-6" izz="2.23136e-6" ixy="0.0" ixz="1.1744e-7" iyz="0" />
-      </inertial>
-  </link>
-  <link name="robotiq_85_right_knuckle_link">
-      <visual>
-          <geometry>
-              <mesh filename="package://dsr_description2/meshes/gripper/robotiq/2f85/visual/right_knuckle.dae" />
-          </geometry>
-      </visual>
-      <collision>
-          <geometry>
-              <mesh filename="package://dsr_description2/meshes/gripper/robotiq/2f85/collision/right_knuckle.stl" />
-          </geometry>
-      </collision>
-      <inertial>
-          <origin xyz="-0.01213197 0.0002 -0.00058647" rpy="0 0 0" />
-          <mass value="1.384773208e-02" />
-          <inertia ixx="3.5232e-7" iyy="2.31944e-6" izz="2.23136e-6" ixy="0.0" ixz="-1.1744e-7" iyz="0.0" />
-      </inertial>
-  </link>
-  <link name="robotiq_85_left_finger_link">
-      <visual>
-          <geometry>
-              <mesh filename="package://dsr_description2/meshes/gripper/robotiq/2f85/visual/left_finger.dae" />
-          </geometry>
-      </visual>
-      <collision>
-          <geometry>
-              <mesh filename="package://dsr_description2/meshes/gripper/robotiq/2f85/collision/left_finger.stl" />
-          </geometry>
-      </collision>
-      <inertial>
-          <origin xyz="0.00346899 -0.00079447 0.01867121" rpy="0 0 0" />
-          <mass value="4.260376752e-02" />
-          <inertia ixx="1.385792000000000e-05" iyy="1.183208e-05" izz="5.19672e-06" ixy="0.0" ixz="-2.17264e-06" iyz="0.0" />
-      </inertial>
-  </link>
-  <link name="robotiq_85_right_finger_link">
-      <visual>
-          <geometry>
-              <mesh filename="package://dsr_description2/meshes/gripper/robotiq/2f85/visual/right_finger.dae" />
-          </geometry>
-      </visual>
-      <collision>
-          <geometry>
-              <mesh filename="package://dsr_description2/meshes/gripper/robotiq/2f85/collision/right_finger.stl" />
-          </geometry>
-      </collision>
-      <inertial>
-          <origin xyz="-0.00346899 -5.53e-06 0.01867121" rpy="0 0 0" />
-          <mass value="4.260376752000000e-02" />
-          <inertia ixx="1.385792e-05" iyy="1.183208e-05" izz="5.19672e-06" ixy="0.0" ixz="2.17264e-06" iyz="0.0" />
-      </inertial>
-  </link>
-  <link name="robotiq_85_left_inner_knuckle_link">
-      <visual>
-          <geometry>
-              <mesh filename="package://dsr_description2/meshes/gripper/robotiq/2f85/visual/left_inner_knuckle.dae" />
-          </geometry>
-      </visual>
-      <collision>
-          <geometry>
-              <mesh filename="package://dsr_description2/meshes/gripper/robotiq/2f85/collision/left_inner_knuckle.stl" />
-          </geometry>
-      </collision>
-      <inertial>
-          <origin xyz="0.01897699 0.00015001 0.02247101" rpy="0 0 0" />
-          <mass value="2.969376448e-02" />
-          <inertia ixx="9.57136e-06" iyy="8.69056e-06" izz="8.19144e-06" ixy="0.0" ixz="-3.93424e-06" iyz="0.0" />
-      </inertial>
-  </link>
-  <link name="robotiq_85_right_inner_knuckle_link">
-      <visual>
-          <geometry>
-              <mesh filename="package://dsr_description2/meshes/gripper/robotiq/2f85/visual/right_inner_knuckle.dae" />
-          </geometry>
-      </visual>
-      <collision>
-          <geometry>
-              <mesh filename="package://dsr_description2/meshes/gripper/robotiq/2f85/collision/right_inner_knuckle.stl" />
-          </geometry>
-      </collision>
-      <inertial>
-          <origin xyz="-0.01926824 5.001e-05 0.02222178" rpy="0 0 0" />
-          <mass value="2.969376448e-02" />
-          <inertia ixx="9.42456e-06" iyy="8.69056e-06" izz="8.33824e-06" ixy="0.0" ixz="3.9636e-06" iyz="0.0" />
-      </inertial>
-  </link>
-  <link name="robotiq_85_left_finger_tip_link">
-      <visual>
-          <geometry>
-              <mesh filename="package://dsr_description2/meshes/gripper/robotiq/2f85/visual/left_finger_tip.dae" />
-          </geometry>
-      </visual>
-      <collision>
-          <geometry>
-              <mesh filename="package://dsr_description2/meshes/gripper/robotiq/2f85/collision/left_finger_tip.stl" />
-          </geometry>
-      </collision>
-      <inertial>
-          <origin xyz="-0.01456706 -0.0008 0.01649701" rpy="0 0 0" />
-          <mass value="4.268588744e-02" />
-          <inertia ixx="1.048152e-05" iyy="1.197888e-05" izz="4.22784e-06" ixy="0.0" ixz="3.5232e-6" iyz="0.0" />
-      </inertial>
-  </link>
-  <link name="robotiq_85_right_finger_tip_link">
-      <visual>
-          <geometry>
-              <mesh filename="package://dsr_description2/meshes/gripper/robotiq/2f85/visual/right_finger_tip.dae" />
-          </geometry>
-      </visual>
-      <collision>
-          <geometry>
-              <mesh filename="package://dsr_description2/meshes/gripper/robotiq/2f85/collision/right_finger_tip.stl" />
-          </geometry>
-      </collision>
-      <inertial>
-          <origin xyz="0.01456706 5e-05 0.01649701" rpy="0 0 0" />
-          <mass value="4.268588744e-02" />
-          <inertia ixx="1.048152e-05" iyy="1.197888e-05" izz="4.22784e-06" ixy="0.0" ixz="-3.5232e-06" iyz="0.0" />
-      </inertial>
-  </link>
-  <joint name="robotiq_85_base_joint" type="fixed">
-      <parent link="link_6" />
-      <child link="robotiq_85_base_link" />
-      <origin xyz="0 0 0.0" rpy="0 0 0"/>
-  </joint>
-  <joint name="robotiq_85_left_knuckle_joint" type="revolute">
-      <parent link="robotiq_85_base_link" />
-      <child link="robotiq_85_left_knuckle_link" />
-      <axis xyz="0 -1 0" />
-      <origin xyz="0.03060114 0.0 0.05490452" rpy="0 0 0" />
-      <limit lower="0.0" upper="0.8" velocity="0.5" effort="50" />
-  </joint>
-  <joint name="robotiq_85_right_knuckle_joint" type="revolute">
-      <parent link="robotiq_85_base_link" />
-      <child link="robotiq_85_right_knuckle_link" />
-      <axis xyz="0 -1 0" />
-      <origin xyz="-0.03060114 0.0 0.05490452" rpy="0 0 0" />
-      <limit lower="-0.8" upper="0.0" velocity="0.5" effort="50" />
-      <mimic joint="robotiq_85_left_knuckle_joint" multiplier="-1" />
-  </joint>
-  <joint name="robotiq_85_left_finger_joint" type="fixed">
-      <parent link="robotiq_85_left_knuckle_link" />
-      <child link="robotiq_85_left_finger_link" />
-      <origin xyz="0.03152616 0.0 -0.00376347" rpy="0 0 0" />
-  </joint>
-  <joint name="robotiq_85_right_finger_joint" type="fixed">
-      <parent link="robotiq_85_right_knuckle_link" />
-      <child link="robotiq_85_right_finger_link" />
-      <origin xyz="-0.03152616 0.0 -0.00376347" rpy="0 0 0" />
-  </joint>
-  <joint name="robotiq_85_left_inner_knuckle_joint" type="continuous">
-      <parent link="robotiq_85_base_link" />
-      <child link="robotiq_85_left_inner_knuckle_link" />
-      <axis xyz="0 -1 0" />
-      <origin xyz="0.0127 0.0 0.06142" rpy="0 0 0" />
-      <mimic joint="robotiq_85_left_knuckle_joint" />
-  </joint>
-  <joint name="robotiq_85_right_inner_knuckle_joint" type="continuous">
-      <parent link="robotiq_85_base_link" />
-      <child link="robotiq_85_right_inner_knuckle_link" />
-      <axis xyz="0 -1 0" />
-      <origin xyz="-0.0127 0.0 0.06142" rpy="0 0 0" />
-      <mimic joint="robotiq_85_left_knuckle_joint" multiplier="-1" />
-  </joint>
-  <joint name="robotiq_85_left_finger_tip_joint" type="continuous">
-      <parent link="robotiq_85_left_finger_link" />
-      <child link="robotiq_85_left_finger_tip_link" />
-      <axis xyz="0 -1 0" />
-      <origin xyz="0.00563134 0.0 0.04718515" rpy="0 0 0" />
-      <mimic joint="robotiq_85_left_knuckle_joint" multiplier="-1" />
-  </joint>
-  <joint name="robotiq_85_right_finger_tip_joint" type="continuous">
-      <parent link="robotiq_85_right_finger_link" />
-      <child link="robotiq_85_right_finger_tip_link" />
-      <axis xyz="0 -1 0" />
-      <origin xyz="-0.00563134 0.0 0.04718515" rpy="0 0 0" />
-      <mimic joint="robotiq_85_left_knuckle_joint" />
-  </joint>
-  <!-- End Robotiq 2F-85 Gripper -->
+  <!-- 월드 고정 -->
   <link name="world"/>
-  <!-- World fixed joint-->
   <joint name="world_fixed" type="fixed">
     <origin xyz="0 0 0" rpy="0 0 0"/>
     <parent link="world"/>
-    <child link="base_link"/>
+    <child  link="base_link"/>
   </joint>
-  <xacro:if value="${gz}">
-    <xacro:include filename="$(find dsr_description2)/ros2_control/m1013.gz_ros2_control.xacro" />
+  <xacro:if value="${gz == 'true'}">
+    <xacro:include filename="$(find dsr_description2)/ros2_control/m1013.gz_ros2_control.xacro"/>
     <xacro:m1013_gz_ros2_control namespace="$(arg namespace)"/>
   </xacro:if>
-  <xacro:unless value="${gz}">
-    <xacro:include filename="$(find dsr_description2)/ros2_control/m1013.ros2_control.xacro" />
+  <xacro:unless value="${gz == 'true'}">
+    <xacro:include filename="$(find dsr_description2)/ros2_control/m1013.ros2_control.xacro"/>
     <xacro:m1013_ros2_control name="m1013"/>
   </xacro:unless>
+  <xacro:if value="${gr != 'none'}">
+    <link name="robotiq_85_base_link">
+    <visual>
+        <geometry>
+        <mesh filename="package://dsr_description2/meshes/gripper/robotiq/2f85/visual/robotiq_base.dae"/>
+        </geometry>
+    </visual>
+    <collision>
+        <geometry>
+        <mesh filename="package://dsr_description2/meshes/gripper/robotiq/2f85/collision/robotiq_base.stl"/>
+        </geometry>
+    </collision>
+    <inertial>
+        <origin xyz="0.0 2.274e-05 0.03232288" rpy="0 0 0"/>
+        <mass value="6.6320197e-01"/>
+        <inertia ixx="5.1617816e-04" iyy="5.8802208e-04" izz="3.9462776e-04" ixy="2.936e-8" ixz="0.0" iyz="-3.2296e-7"/>
+    </inertial>
+    </link>
+    <link name="robotiq_85_left_knuckle_link">
+    <visual>
+        <geometry>
+        <mesh filename="package://dsr_description2/meshes/gripper/robotiq/2f85/visual/left_knuckle.dae"/>
+        </geometry>
+    </visual>
+    <collision>
+        <geometry>
+        <mesh filename="package://dsr_description2/meshes/gripper/robotiq/2f85/collision/left_knuckle.stl"/>
+        </geometry>
+    </collision>
+    <inertial>
+        <origin xyz="0.01213197 0.0002 -0.00058647" rpy="0 0 0"/>
+        <mass value="1.384773208e-02"/>
+        <inertia ixx="3.5232e-7" iyy="2.31944e-6" izz="2.23136e-6" ixy="0.0" ixz="1.1744e-7" iyz="0"/>
+    </inertial>
+    </link>
+    <link name="robotiq_85_right_knuckle_link">
+    <visual>
+        <geometry>
+        <mesh filename="package://dsr_description2/meshes/gripper/robotiq/2f85/visual/right_knuckle.dae"/>
+        </geometry>
+    </visual>
+    <collision>
+        <geometry>
+        <mesh filename="package://dsr_description2/meshes/gripper/robotiq/2f85/collision/right_knuckle.stl"/>
+        </geometry>
+    </collision>
+    <inertial>
+        <origin xyz="-0.01213197 0.0002 -0.00058647" rpy="0 0 0"/>
+        <mass value="1.384773208e-02"/>
+        <inertia ixx="3.5232e-7" iyy="2.31944e-6" izz="2.23136e-6" ixy="0.0" ixz="-1.1744e-7" iyz="0.0"/>
+    </inertial>
+    </link>
+    <link name="robotiq_85_left_finger_link">
+    <visual>
+        <geometry>
+        <mesh filename="package://dsr_description2/meshes/gripper/robotiq/2f85/visual/left_finger.dae"/>
+        </geometry>
+    </visual>
+    <collision>
+        <geometry>
+        <mesh filename="package://dsr_description2/meshes/gripper/robotiq/2f85/collision/left_finger.stl"/>
+        </geometry>
+    </collision>
+    <inertial>
+        <origin xyz="0.00346899 -0.00079447 0.01867121" rpy="0 0 0"/>
+        <mass value="4.260376752e-02"/>
+        <inertia ixx="1.385792000000000e-05" iyy="1.183208e-05" izz="5.19672e-06" ixy="0.0" ixz="-2.17264e-06" iyz="0.0"/>
+    </inertial>
+    </link>
+    <link name="robotiq_85_right_finger_link">
+    <visual>
+        <geometry>
+        <mesh filename="package://dsr_description2/meshes/gripper/robotiq/2f85/visual/right_finger.dae"/>
+        </geometry>
+    </visual>
+    <collision>
+        <geometry>
+        <mesh filename="package://dsr_description2/meshes/gripper/robotiq/2f85/collision/right_finger.stl"/>
+        </geometry>
+    </collision>
+    <inertial>
+        <origin xyz="-0.00346899 -5.53e-06 0.01867121" rpy="0 0 0"/>
+        <mass value="4.260376752000000e-02"/>
+        <inertia ixx="1.385792e-05" iyy="1.183208e-05" izz="5.19672e-06" ixy="0.0" ixz="2.17264e-06" iyz="0.0"/>
+    </inertial>
+    </link>
+    <link name="robotiq_85_left_inner_knuckle_link">
+    <visual>
+        <geometry>
+        <mesh filename="package://dsr_description2/meshes/gripper/robotiq/2f85/visual/left_inner_knuckle.dae"/>
+        </geometry>
+    </visual>
+    <collision>
+        <geometry>
+        <mesh filename="package://dsr_description2/meshes/gripper/robotiq/2f85/collision/left_inner_knuckle.stl"/>
+        </geometry>
+    </collision>
+    <inertial>
+        <origin xyz="0.01897699 0.00015001 0.02247101" rpy="0 0 0"/>
+        <mass value="2.969376448e-02"/>
+        <inertia ixx="9.57136e-06" iyy="8.69056e-06" izz="8.19144e-06" ixy="0.0" ixz="-3.93424e-06" iyz="0.0"/>
+    </inertial>
+    </link>
+    <link name="robotiq_85_right_inner_knuckle_link">
+    <visual>
+        <geometry>
+        <mesh filename="package://dsr_description2/meshes/gripper/robotiq/2f85/visual/right_inner_knuckle.dae"/>
+        </geometry>
+    </visual>
+    <collision>
+        <geometry>
+        <mesh filename="package://dsr_description2/meshes/gripper/robotiq/2f85/collision/right_inner_knuckle.stl"/>
+        </geometry>
+    </collision>
+    <inertial>
+        <origin xyz="-0.01926824 5.001e-05 0.02222178" rpy="0 0 0"/>
+        <mass value="2.969376448e-02"/>
+        <inertia ixx="9.42456e-06" iyy="8.69056e-06" izz="8.33824e-06" ixy="0.0" ixz="3.9636e-06" iyz="0.0"/>
+    </inertial>
+    </link>
+    <link name="robotiq_85_left_finger_tip_link">
+    <visual>
+        <geometry>
+        <mesh filename="package://dsr_description2/meshes/gripper/robotiq/2f85/visual/left_finger_tip.dae"/>
+        </geometry>
+    </visual>
+    <collision>
+        <geometry>
+        <mesh filename="package://dsr_description2/meshes/gripper/robotiq/2f85/collision/left_finger_tip.stl"/>
+        </geometry>
+    </collision>
+    <inertial>
+        <origin xyz="-0.01456706 -0.0008 0.01649701" rpy="0 0 0"/>
+        <mass value="4.268588744e-02"/>
+        <inertia ixx="1.048152e-05" iyy="1.197888e-05" izz="4.22784e-06" ixy="0.0" ixz="3.5232e-6" iyz="0.0"/>
+    </inertial>
+    </link>
+    <link name="robotiq_85_right_finger_tip_link">
+    <visual>
+        <geometry>
+        <mesh filename="package://dsr_description2/meshes/gripper/robotiq/2f85/visual/right_finger_tip.dae"/>
+        </geometry>
+    </visual>
+    <collision>
+        <geometry>
+        <mesh filename="package://dsr_description2/meshes/gripper/robotiq/2f85/collision/right_finger_tip.stl"/>
+        </geometry>
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
File: dsr_moveit2/dsr_moveit_config_m1013/config/m1013.ros2_control.xacro (robot description, xacro)
@@ -50,6 +50,4 @@
                 <state_interface name="velocity"/>
             </joint>
-            <!-- Import Gripper Control -->
-            <!-- <xacro:insert_block name="gripper_control_xacro"/> -->
         </ros2_control>
     </xacro:macro>

File: dsr_moveit2/dsr_moveit_config_m1013/config/m1013.urdf.xacro (robot description, xacro)
@@ -6,15 +6,4 @@
     <!-- Import control_xacro -->
     <xacro:include filename="m1013.ros2_control.xacro" />
-    <!-- Import robotiq 2f85 gripper -->
-    <xacro:include filename="$(find dsr_description2)/urdf/robotiq_2f_85_macro.urdf.xacro" />
     <xacro:m1013_ros2_control name="FakeSystem" initial_positions_file="$(arg initial_positions_file)"/>
-    <!-- Attach Robotiq 2F-85 gripper -->
-    <xacro:robotiq_gripper
-        name="RobotiqGripper"
-        prefix=""
-        parent="link_6"
-        use_fake_hardware="true"
-        include_ros2_control="true">
-        <origin xyz="0 0 0" rpy="0 0 0" />
-    </xacro:robotiq_gripper>
 </robot>
