Commit message: feat(moveit): add Robotiq gripper support and planning integration (jazzy)

File: dsr_description2/ros2_control/m1013.ros2_control.xacro (robot description, xacro)
@@ -1,22 +1,22 @@
 <?xml version="1.0"?>
 <robot xmlns:xacro="http://www.ros.org/wiki/xacro">
+  <!-- Doosan M1013 ros2_control (arm-only) -->
   <xacro:macro name="m1013_ros2_control" params="
-    name
-    rate:=100
-    standby:=true
-    command:=none
-    host:=0.0.0.0
-    port:=12345
-    mode:=real
-    model:=m1013
-    gripper:=none
-    mobile:=none
-  ">
+      name
+      rate:=100
+      standby:=true
+      command:=none
+      host:=127.0.0.1
+      port:=12345
+      mode:=virtual
+      model:=m1013
+      mobile:=none">
     <xacro:property name="double_pi" value="${2.0 * pi}"/>
     <xacro:property name="neg_double_pi" value="${-2.0 * pi}"/>
-    <xacro:property name="neg_pi" value="${-1.0 * pi}"/>
     <ros2_control name="${name}" type="system">
       <hardware>
         <plugin>dsr_hardware2/DRHWInterface</plugin>
+        <!-- virtual 테스트면 true 유지 가능 (실기면 false 권장) -->
+        <param name="use_mock_hardware">true</param>
         <param name="name">${name}</param>
         <param name="rate">${rate}</param>
@@ -27,7 +27,7 @@
         <param name="mode">${mode}</param>
         <param name="model">${model}</param>
-        <param name="gripper">${gripper}</param>
         <param name="mobile">${mobile}</param>
       </hardware>
+      <!-- Arm joints only -->
       <joint name="joint_1">
         <command_interface name="position">
@@ -36,6 +36,6 @@
         </command_interface>
         <command_interface name="velocity">
-          <param name="min">-3.15</param>
-          <param name="max">3.15</param>
+          <param name="min">-3.2</param>
+          <param name="max">3.2</param>
         </command_interface>
         <state_interface name="position"><param name="initial_value">0.0</param></state_interface>
@@ -48,6 +48,6 @@
         </command_interface>
         <command_interface name="velocity">
-          <param name="min">-3.15</param>
-          <param name="max">3.15</param>
+          <param name="min">-3.2</param>
+          <param name="max">3.2</param>
         </command_interface>
         <state_interface name="position"><param name="initial_value">0.0</param></state_interface>
@@ -56,10 +56,10 @@
       <joint name="joint_3">
         <command_interface name="position">
-          <param name="min">${neg_pi}</param>
-          <param name="max">${pi}</param>
+          <param name="min">${neg_double_pi}</param>
+          <param name="max">${double_pi}</param>
         </command_interface>
         <command_interface name="velocity">
-          <param name="min">-3.15</param>
-          <param name="max">3.15</param>
+          <param name="min">-3.2</param>
+          <param name="max">3.2</param>
         </command_interface>
         <state_interface name="position"><param name="initial_value">0.0</param></state_interface>

File: dsr_description2/xacro/m1013.urdf.xacro (robot description, xacro)
@@ -1,32 +1,54 @@
 <?xml version="1.0"?>
-<robot xmlns:xacro="http://www.ros.org/wiki/xacro" name="m1013" >
-  <xacro:arg name="color"   default="white"/>
-  <xacro:arg name="gripper" default="none"/>
-  <xacro:arg name="namespace" default=""/>
+<robot xmlns:xacro="http://www.ros.org/wiki/xacro" name="m1013">
+  <xacro:arg name="mode"           default="virtual"/>
+  <xacro:arg name="color"          default="white"/>
+  <xacro:arg name="namespace"      default=""/>
+  <!-- gripper control argument -->
+  <xacro:arg name="gripper"              default="none"/>         <!-- none | robotique -->
+  <xacro:arg name="gripper_prefix"       default=""/>             <!-- ex) dsr01_ -->
+  <xacro:arg name="gripper_parent_link"  default="link_6"/>
   <xacro:arg name="use_gazebo" default="false"/>
+  <xacro:property name="gz" value="$(arg use_gazebo)"/>
   <xacro:property name="cr" value="$(arg color)"/>
   <xacro:property name="gr" value="$(arg gripper)"/>
-  <xacro:property name="gz" value="$(arg use_gazebo)"/>
   <xacro:if value="${cr == 'white'}">
-     <xacro:include filename="$(find dsr_description2)/xacro/macro.m1013.white.xacro" />
+    <xacro:include filename="$(find dsr_description2)/xacro/macro.m1013.white.xacro"/>
   </xacro:if>
   <xacro:if value="${cr == 'blue'}">
-     <xacro:include filename="$(find dsr_description2)/xacro/macro.m1013.blue.xacro" />
+    <xacro:include filename="$(find dsr_description2)/xacro/macro.m1013.blue.xacro"/>
   </xacro:if>
   <xacro:m1013 namespace="$(arg namespace)"/>
   <link name="world"/>
-  <!-- World fixed joint-->
   <joint name="world_fixed" type="fixed">
     <origin xyz="0 0 0" rpy="0 0 0"/>
     <parent link="world"/>
-    <child link="base_link"/>
+    <child  link="base_link"/>
   </joint>
-  <xacro:if value="${gz}">
-    <xacro:include filename="$(find dsr_description2)/ros2_control/m1013.gz_ros2_control.xacro" />
+  <xacro:if value="${gz == 'true'}">
+    <xacro:include filename="$(find dsr_description2)/ros2_control/m1013.gz_ros2_control.xacro"/>
     <xacro:m1013_gz_ros2_control namespace="$(arg namespace)"/>
   </xacro:if>
-  <xacro:unless value="${gz}">
-    <xacro:include filename="$(find dsr_description2)/ros2_control/m1013.ros2_control.xacro" />
+  <xacro:unless value="${gz == 'true'}">
+    <xacro:include filename="$(find dsr_description2)/ros2_control/m1013.ros2_control.xacro"/>
     <xacro:m1013_ros2_control name="m1013"/>
   </xacro:unless>
+  <xacro:if value="${gr == 'robotiq_2f85'}">
+    <xacro:include filename="$(find dsr_description2)/gripper/robotiq.xacro"/>
+    <xacro:robotiq_85
+      parent="$(arg gripper_parent_link)"
+      prefix="$(arg gripper_prefix)"/>
+    <xacro:include filename="$(find dsr_description2)/gripper/robotiq.ros2_control.xacro"/>
+      <xacro:robotiq_gripper_system
+      mode="$(arg mode)"
+      joint_name="$(arg gripper_prefix)robotiq_85_left_knuckle_joint"
+      system_name="$(arg gripper_prefix)robotiq_gripper_system"
+      pos_min="0.0"
+      pos_max="0.8"
+      init_pos="0.0"
+      speed_mult="1.0"
+      force_mult="0.5"
+      max_speed="0.150"
+      max_force="235.0"
+      mock_sensor_commands="true" />
+  </xacro:if>
 </robot>
