Commit message: update P3020 Model description

File: dsr_description2/config/macro.materials.xacro (robot description, xacro)
@@ -17,4 +17,7 @@
 			<color rgba="0.941 0.941 0.941 1.0" />
 		</material>
+		<material name="dr_blue">
+			<color rgba="0 0 0.2 1" />
+		</material>
 	</xacro:macro>
 </robot>

File: dsr_description2/xacro/macro.p3020.blue.xacro (robot description, xacro)
@@ -12,5 +12,5 @@
                     <mesh scale="0.001 0.001 0.001" filename="package://dsr_description2/meshes/p3020/1.STL"/>
                 </geometry>
-                <material name="dr_white" />
+                <material name="dr_gray" />
             </visual>
             <collision>
@@ -27,5 +27,5 @@
                     <mesh filename="package://dsr_description2/meshes/p3020/2-1.STL" scale="0.001 0.001 0.001" />
                 </geometry>
-                <material name="dr_white" />
+                <material name="dr_blue" />
             </visual>
             <visual>
@@ -34,5 +34,5 @@
                     <mesh filename="package://dsr_description2/meshes/p3020/2-2.STL" scale="0.001 0.001 0.001" />
                 </geometry>
-                <material name="dr_white" />
+                <material name="dr_blue" />
             </visual>
             <visual>
@@ -41,5 +41,5 @@
                     <mesh filename="package://dsr_description2/meshes/p3020/2-3.STL" scale="0.001 0.001 0.001" />
                 </geometry>
-                <material name="dr_white" />
+                <material name="dr_blue" />
             </visual>
             <visual>
@@ -48,5 +48,5 @@
                     <mesh filename="package://dsr_description2/meshes/p3020/2-4.STL" scale="0.001 0.001 0.001" />
                 </geometry>
-                <material name="dr_white" />
+                <material name="dr_blue" />
             </visual>
             <visual>
@@ -55,5 +55,5 @@
                     <mesh filename="package://dsr_description2/meshes/p3020/2-5.STL" scale="0.001 0.001 0.001" />
                 </geometry>
-                <material name="dr_white" />
+                <material name="dr_blue" />
             </visual>
             <collision>
@@ -95,5 +95,5 @@
                     <mesh filename="package://dsr_description2/meshes/p3020/3-1.STL" scale="0.001 0.001 0.001" color="0 0 0 1"/>
                 </geometry>
-                <material name="dr_white" />
+                <material name="dr_blue" />
             </visual>
             <visual>
@@ -102,5 +102,5 @@
                     <mesh filename="package://dsr_description2/meshes/p3020/3-2.STL" scale="0.001 0.001 0.001" />
                 </geometry>
-                <material name="dr_white" />
+                <material name="dr_blue" />
             </visual>
             <visual>
@@ -115,5 +115,5 @@
                     <mesh filename="package://dsr_description2/meshes/p3020/3-4.STL" scale="0.001 0.001 0.001" />
                 </geometry>
-                <material name="dr_white" />
+                <material name="dr_blue" />
             </visual>
             <visual>
@@ -122,5 +122,5 @@
                     <mesh filename="package://dsr_description2/meshes/p3020/3-5.STL" scale="0.001 0.001 0.001" />
                 </geometry>
-                <material name="dr_white" />
+                <material name="dr_blue" />
             </visual>
             <visual>
@@ -129,5 +129,5 @@
                     <mesh filename="package://dsr_description2/meshes/p3020/3-6.STL" scale="0.001 0.001 0.001" />
                 </geometry>
-                <material name="dr_white" />
+                <material name="dr_blue" />
             </visual>
             <visual>
@@ -136,5 +136,5 @@
                     <mesh filename="package://dsr_description2/meshes/p3020/3-7.STL" scale="0.001 0.001 0.001" />
                 </geometry>
-                <material name="dr_white" />
+                <material name="dr_blue" />
             </visual>
             <visual>
@@ -143,5 +143,7 @@
                     <mesh filename="package://dsr_description2/meshes/p3020/3-8.STL" scale="0.001 0.001 0.001" />
                 </geometry>
-                <material name="dr_white" />
+                <material name="dr_blue">
+                    <color rgba="0.490 0.490 0.486 1.0" />
+                </material>
             </visual>
             <collision>
@@ -201,5 +203,5 @@
                     <mesh filename="package://dsr_description2/meshes/p3020/4-1.STL" scale="0.001 0.001 0.001" />
                 </geometry>
-                <material name="dr_white" />
+                <material name="dr_blue" />
             </visual>
             <visual>
@@ -208,5 +210,5 @@
                     <mesh filename="package://dsr_description2/meshes/p3020/4-2.STL" scale="0.001 0.001 0.001" />
                 </geometry>
-                <material name="dr_white" />
+                <material name="dr_blue" />
             </visual>
             <visual>
@@ -215,5 +217,5 @@
                     <mesh filename="package://dsr_description2/meshes/p3020/4-3.STL" scale="0.001 0.001 0.001" />
                 </geometry>
-                <material name="dr_white" />
+                <material name="dr_blue" />
             </visual>
             <visual>
@@ -222,5 +224,5 @@
                     <mesh filename="package://dsr_description2/meshes/p3020/4-4.STL" scale="0.001 0.001 0.001" />
                 </geometry>
-                <material name="dr_white" />
+                <material name="dr_blue" />
             </visual>
             <collision>
@@ -259,5 +261,5 @@
                     <mesh filename="package://dsr_description2/meshes/p3020/6-1.STL" scale="0.001 0.001 0.001" />
                 </geometry>
-                <material name="dr_white" />
+                <material name="dr_blue" />
             </visual>
             <visual>
@@ -266,5 +268,5 @@
                     <mesh filename="package://dsr_description2/meshes/p3020/6-2.STL" scale="0.001 0.001 0.001" />
                 </geometry>
-                <material name="dr_white" />
+                <material name="dr_blue" />
             </visual>
             <visual>
@@ -273,5 +275,5 @@
                     <mesh filename="package://dsr_description2/meshes/p3020/6-3.STL" scale="0.001 0.001 0.001" />
                 </geometry>
-                <material name="dr_white" />
+                <material name="dr_blue" />
             </visual>
             <collision>
@@ -301,5 +303,5 @@
                     <mesh filename="package://dsr_description2/meshes/p3020/7.STL" scale="0.001 0.001 0.001" />
                 </geometry>
-                <material name="dr_white" />
+                <material name="dr_gray" />
             </visual>
             <collision>

File: dsr_description2/xacro/p3020.urdf.xacro (robot description, xacro)
@@ -10,4 +10,7 @@
   <xacro:if value="${cr == 'white'}">
      <xacro:include filename="$(find dsr_description2)/xacro/macro.p3020.white.xacro" />
+  </xacro:if>
+  <xacro:if value="${cr == 'blue'}">
+     <xacro:include filename="$(find dsr_description2)/xacro/macro.p3020.blue.xacro" />
   </xacro:if>
   <xacro:p3020 namespace="$(arg namespace)"/>
