Commit message: update gazebo packages for p3020

File: dsr_description2/xacro/macro.p3020.white.xacro (robot description, xacro)
@@ -1,5 +1,5 @@
 <?xml version="1.0"?>
 <robot name="p3020" xmlns:xacro="http://www.ros.org/wiki/xacro">
-    <xacro:include filename="$(find dsr_description2)/config/macro.gazebo.xacro" />
+    <xacro:include filename="$(find dsr_description2)/config/macro.gazebo.p3020.xacro" />
     <xacro:include filename="$(find dsr_description2)/config/macro.transmission.xacro" />
     <xacro:include filename="$(find dsr_description2)/config/macro.materials.xacro" />
@@ -8,347 +8,286 @@
         <!-- Base Link -->
         <link name="base_link">
-            <visual>
-                <geometry>
-                    <mesh scale="0.001 0.001 0.001" filename="package://dsr_description2/meshes/p3020/1.STL"/>
-                </geometry>
-                <material name="dr_white" />
-            </visual>
-            <collision>
-                <geometry>
-                    <mesh scale="0.001 0.001 0.001" filename="package://dsr_description2/meshes/p3020/1.STL"/>
-                </geometry>
-            </collision>
+            <inertial>
+                <mass value="9.55"/>
+                <origin xyz="6e-06   -0.007232     0.10749"/>
+                <inertia ixx="0.01" ixy="0.00001" ixz="0.00001"
+         iyy="0.01" iyz="0.00001" izz="0.01"/>
+            </inertial>
+            <visual>
+                <origin rpy="0 0 0" xyz="0 0 0"/>
+                <geometry>
+                    <mesh filename="package://dsr_description2/meshes/p3020/P3020_0_1.STL"
+                        scale="0.001 0.001 0.001"/>
+                </geometry>
+                <material name="dr_white"/>
+            </visual>
         </link>
         <!-- link_1 -->
         <link name="link_1">
-            <visual>
-                <origin xyz="0 0 -0.3943"/>
-                <geometry>
-                    <mesh filename="package://dsr_description2/meshes/p3020/2-1.STL" scale="0.001 0.001 0.001" />
-                </geometry>
-                <material name="dr_white" />
-            </visual>
-            <visual>
-                <origin xyz="0 0 -0.3943"/>
-                <geometry>
-                    <mesh filename="package://dsr_description2/meshes/p3020/2-2.STL" scale="0.001 0.001 0.001" />
-                </geometry>
-                <material name="dr_white" />
-            </visual>
-            <visual>
-                <origin xyz="0 0 -0.3943"/>
-                <geometry>
-                    <mesh filename="package://dsr_description2/meshes/p3020/2-3.STL" scale="0.001 0.001 0.001" />
-                </geometry>
-                <material name="dr_white" />
-            </visual>
-            <visual>
-                <origin xyz="0 0 -0.3943"/>
-                <geometry>
-                    <mesh filename="package://dsr_description2/meshes/p3020/2-4.STL" scale="0.001 0.001 0.001" />
-                </geometry>
-                <material name="dr_white" />
-            </visual>
-            <visual>
-                <origin xyz="0 0 -0.3943"/>
-                <geometry>
-                    <mesh filename="package://dsr_description2/meshes/p3020/2-5.STL" scale="0.001 0.001 0.001" />
-                </geometry>
-                <material name="dr_white" />
-            </visual>
-            <collision>
-                <origin xyz="0 0 -0.3943"/>
-                <geometry>
-                    <mesh filename="package://dsr_description2/meshes/p3020/2-1.STL" scale="0.001 0.001 0.001" />
-                </geometry>
-            </collision>
-            <collision>
-                <origin xyz="0 0 -0.3943"/>
-                <geometry>
-                    <mesh filename="package://dsr_description2/meshes/p3020/2-2.STL" scale="0.001 0.001 0.001" />
-                </geometry>
-            </collision>
-            <collision>
-                <origin xyz="0 0 -0.3943"/>
-                <geometry>
-                    <mesh filename="package://dsr_description2/meshes/p3020/2-3.STL" scale="0.001 0.001 0.001" />
-                </geometry>
-            </collision>
-            <collision>
-                <origin xyz="0 0 -0.3943"/>
-                <geometry>
-                    <mesh filename="package://dsr_description2/meshes/p3020/2-4.STL" scale="0.001 0.001 0.001" />
-                </geometry>
-            </collision>
-            <collision>
-                <origin xyz="0 0 -0.3943"/>
-                <geometry>
-                    <mesh filename="package://dsr_description2/meshes/p3020/2-5.STL" scale="0.001 0.001 0.001" />
-                </geometry>
-            </collision>
+            <inertial>
+                <mass value="28.624"/>
+                <origin xyz="-1.1e-05     0.11205   -0.065579"/>
+                <inertia ixx="0.69287" ixy="0.0" ixz="0.0" iyy="0.36715" iyz="0.0" izz="0.46086"/>
+            </inertial>
+            <visual>
+                <origin xyz="0 0 -0.3943"/>
+                <geometry>
+                    <mesh filename="package://dsr_description2/meshes/p3020/P3020_1_1.STL"
+                        scale="0.001 0.001 0.001"/>
+                </geometry>
+                <material name="dr_white"/>
+            </visual>
+            <visual>
+                <origin xyz="0 0 -0.3943"/>
+                <geometry>
+                    <mesh filename="package://dsr_description2/meshes/p3020/P3020_1_2.STL"
+                        scale="0.001 0.001 0.001"/>
+                </geometry>
+                <material name="dr_white"/>
+            </visual>
+            <visual>
+                <origin xyz="0 0 -0.3943"/>
+                <geometry>
+                    <mesh filename="package://dsr_description2/meshes/p3020/P3020_1_3.STL"
+                        scale="0.001 0.001 0.001"/>
+                </geometry>
+                <material name="dr_white"/>
+            </visual>
+            <visual>
+                <origin xyz="0 0 -0.3943"/>
+                <geometry>
+                    <mesh filename="package://dsr_description2/meshes/p3020/P3020_1_4.STL"
+                        scale="0.001 0.001 0.001"/>
+                </geometry>
+                <material name="dr_white"/>
+            </visual>
+            <visual>
+                <origin xyz="0 0 -0.3943"/>
+                <geometry>
+                    <mesh filename="package://dsr_description2/meshes/p3020/P3020_1_5.STL"
+                        scale="0.001 0.001 0.001"/>
+                </geometry>
+                <material name="dr_white"/>
+            </visual>
         </link>
         <!-- link_2 -->
         <link name="link_2">
-            <visual>
-                <origin xyz="0 0 -0.3943"/>
-                <geometry>
-                    <mesh filename="package://dsr_description2/meshes/p3020/3-1.STL" scale="0.001 0.001 0.001" color="0 0 0 1"/>
-                </geometry>
-                <material name="dr_white" />
-            </visual>
-            <visual>
-                <origin xyz="0 0 -0.3943"/>
-                <geometry>
-                    <mesh filename="package://dsr_description2/meshes/p3020/3-2.STL" scale="0.001 0.001 0.001" />
-                </geometry>
-                <material name="dr_white" />
-            </visual>
-            <visual>
-                <origin xyz="0 0 -0.3943"/>
-                <geometry>
-                    <mesh filename="package://dsr_description2/meshes/p3020/3-3.STL" scale="0.001 0.001 0.001" />
-                </geometry>
-            </visual>
-            <visual>
-                <origin xyz="0 0 -0.3943"/>
-                <geometry>
-                    <mesh filename="package://dsr_description2/meshes/p3020/3-4.STL" scale="0.001 0.001 0.001" />
-                </geometry>
-                <material name="dr_white" />
-            </visual>
-            <visual>
-                <origin xyz="0 0 -0.3943"/>
-                <geometry>
-                    <mesh filename="package://dsr_description2/meshes/p3020/3-5.STL" scale="0.001 0.001 0.001" />
-                </geometry>
-                <material name="dr_white" />
-            </visual>
-            <visual>
-                <origin xyz="0 0 -0.3943"/>
-                <geometry>
-                    <mesh filename="package://dsr_description2/meshes/p3020/3-6.STL" scale="0.001 0.001 0.001" />
-                </geometry>
-                <material name="dr_white" />
-            </visual>
-            <visual>
-                <origin xyz="0 0 -0.3943"/>
-                <geometry>
-                    <mesh filename="package://dsr_description2/meshes/p3020/3-7.STL" scale="0.001 0.001 0.001" />
-                </geometry>
-                <material name="dr_white" />
-            </visual>
-            <visual>
-                <origin xyz="0 0 -0.3943"/>
-                <geometry>
-                    <mesh filename="package://dsr_description2/meshes/p3020/3-8.STL" scale="0.001 0.001 0.001" />
-                </geometry>
-                <material name="dr_white" />
-            </visual>
-            <collision>
-                <origin xyz="0 0 -0.3943"/>
-                <geometry>
-                    <mesh filename="package://dsr_description2/meshes/p3020/3-1.STL" scale="0.001 0.001 0.001" />
-                </geometry>
-            </collision>
-            <collision>
-                <origin xyz="0 0 -0.3943"/>
-                <geometry>
-                    <mesh filename="package://dsr_description2/meshes/p3020/3-2.STL" scale="0.001 0.001 0.001" />
-                </geometry>
-            </collision>
-            <collision>
-                <origin xyz="0 0 -0.3943"/>
-                <geometry>
-                    <mesh filename="package://dsr_description2/meshes/p3020/3-3.STL" scale="0.001 0.001 0.001" />
-                </geometry>
-            </collision>
-            <collision>
-                <origin xyz="0 0 -0.3943"/>
-                <geometry>
-                    <mesh filename="package://dsr_description2/meshes/p3020/3-4.STL" scale="0.001 0.001 0.001" />
-                </geometry>
-            </collision>
-            <collision>
-                <origin xyz="0 0 -0.3943"/>
-                <geometry>
-                    <mesh filename="package://dsr_description2/meshes/p3020/3-5.STL" scale="0.001 0.001 0.001" />
-                </geometry>
-            </collision>
-            <collision>
-                <origin xyz="0 0 -0.3943"/>
-                <geometry>
-                    <mesh filename="package://dsr_description2/meshes/p3020/3-6.STL" scale="0.001 0.001 0.001" />
-                </geometry>
-            </collision>
-            <collision>
-                <origin xyz="0 0 -0.3943"/>
-                <geometry>
-                    <mesh filename="package://dsr_description2/meshes/p3020/3-7.STL" scale="0.001 0.001 0.001" />
-                </geometry>
-            </collision>
-            <collision>
-                <origin xyz="0 0 -0.3943"/>
-                <geometry>
-                    <mesh filename="package://dsr_description2/meshes/p3020/3-8.STL" scale="0.001 0.001 0.001" />
-                </geometry>
-            </collision>
+            <inertial>
+                <mass value="30.357"/>
+                <origin xyz="0.4005       5e-06    0.006736"/>
+                 <inertia ixx="0.17985" ixy="0.000214" ixz="0.00018611" iyy="4.5411" iyz="0.0" izz="4.4825"/>
+            </inertial>
+            <visual>
+                 <!-- <origin xyz="0 -0.2351 -0.3943" rpy="0  -1.5708 -1.-0.3943708"/> -->
+                 <origin xyz="-0.3943 0 -0.2351" rpy="1.5708 0 1.5708"/>
+                <geometry>
+                    <mesh filename="package://dsr_description2/meshes/p3020/P3020_2_1.STL"
+                        scale="0.001 0.001 0.001"/>
+                </geometry>
+                <material name="dr_white"/>
+            </visual>
+            <visual>
+                <!-- <origin xyz="0 -0.2351 -0.3943" rpy="-1.5708  -1.5708 -1.5708"/> -->
+                 <origin xyz="-0.3943 0 -0.2351" rpy="1.5708 0 1.5708"/>
+                <geometry>
+                    <mesh filename="package://dsr_description2/meshes/p3020/P3020_2_2.STL"
+                        scale="0.001 0.001 0.001"/>
+                </geometry>
+                <material name="dr_white"/>
+            </visual>
+            <visual>
+                <!-- <origin xyz="0 -0.2351 -0.3943" rpy="-1.5708  0 1.5708"/> -->
+                 <origin xyz="-0.3943 0 -0.2351" rpy="1.5708 0 1.5708"/>
+                <geometry>
+                    <mesh filename="package://dsr_description2/meshes/p3020/P3020_2_3.STL"
+                        scale="0.001 0.001 0.001"/>
+                </geometry>
+                <material name="dr_white"/>
+            </visual>
+            <visual>
+                <!-- <origin xyz="0 -0.2351 -0.3943" rpy="-1.5708  0 1.5708"/> -->
+                 <origin xyz="-0.3943 0 -0.2351" rpy="1.5708 0 1.5708"/>
+                <geometry>
+                    <mesh filename="package://dsr_description2/meshes/p3020/P3020_2_4.STL"
+                        scale="0.001 0.001 0.001"/>
+                </geometry>
+                <material name="dr_white"/>
+            </visual>
+            <visual>
+                <!-- <origin xyz="0 -0.2351 -0.3943" rpy="-1.5708  0 1.5708"/> -->
+                 <origin xyz="-0.3943 0 -0.2351" rpy="1.5708 0 1.5708"/>
+                <geometry>
+                    <mesh filename="package://dsr_description2/meshes/p3020/P3020_2_5.STL"
+                        scale="0.001 0.001 0.001"/>
+                </geometry>
+                <material name="dr_white"/>
+            </visual>
+            <visual>
+                <!-- <origin xyz="0 -0.2351 -0.3943" rpy="-1.5708  0 1.5708"/> -->
+                 <origin xyz="-0.3943 0 -0.2351" rpy="1.5708 0 1.5708"/>
+                <geometry>
+                    <mesh filename="package://dsr_description2/meshes/p3020/P3020_2_6.STL"
+                        scale="0.001 0.001 0.001"/>
+                </geometry>
+                <material name="dr_white"/>
+            </visual>
+            <visual>
+                <!-- <origin xyz="0 -0.2351 -0.3943" rpy="-1.5708  0 1.5708"/> -->
+                 <origin xyz="-0.3943 0 -0.2351" rpy="1.5708 0 1.5708"/>
+                <geometry>
+                    <mesh filename="package://dsr_description2/meshes/p3020/P3020_2_7.STL"
+                        scale="0.001 0.001 0.001"/>
+                </geometry>
+                <material name="dr_white"/>
+            </visual>
+            <visual>
+                <!-- <origin xyz="0 -0.2351 -0.3943" rpy="-1.5708  0 1.5708"/> -->
+                 <origin xyz="-0.3943 0 -0.2351" rpy="1.5708 0 1.5708"/>
+                <geometry>
+                    <mesh filename="package://dsr_description2/meshes/p3020/P3020_2_8.STL"
+                        scale="0.001 0.001 0.001"/>
+                </geometry>
+                <material name="dr_white"/>
+            </visual>
         </link>
         <!-- link_3 -->
         <link name="link_3">
-            <visual>
-                <origin xyz="0 0 -1.4043"/>
-                <geometry>
-                    <mesh filename="package://dsr_description2/meshes/p3020/4-1.STL" scale="0.001 0.001 0.001" />
-                </geometry>
-                <material name="dr_white" />
-            </visual>
-            <visual>
-                <origin xyz="0 0 -1.4043"/>
-                <geometry>
-                    <mesh filename="package://dsr_description2/meshes/p3020/4-2.STL" scale="0.001 0.001 0.001" />
-                </geometry>
-                <material name="dr_white" />
-            </visual>
-            <visual>
-                <origin xyz="0 0 -1.4043"/>
-                <geometry>
-                    <mesh filename="package://dsr_description2/meshes/p3020/4-3.STL" scale="0.001 0.001 0.001" />
-                </geometry>
-                <material name="dr_white" />
-            </visual>
-            <visual>
-                <origin xyz="0 0 -1.4043"/>
-                <geometry>
-                    <mesh filename="package://dsr_description2/meshes/p3020/4-4.STL" scale="0.001 0.001 0.001" />
-                </geometry>
-                <material name="dr_white" />
-            </visual>
-            <collision>
-                <origin xyz="0 0 -1.4043"/>
-                <geometry>
-                    <mesh filename="package://dsr_description2/meshes/p3020/4-1.STL" scale="0.001 0.001 0.001" />
-                </geometry>
-            </collision>
-            <collision>
-                <origin xyz="0 0 -1.4043"/>
-                <geometry>
-                    <mesh filename="package://dsr_description2/meshes/p3020/4-2.STL" scale="0.001 0.001 0.001" />
-                </geometry>
-            </collision>
-            <collision>
-                <origin xyz="0 0 -1.4043"/>
-                <geometry>
-                    <mesh filename="package://dsr_description2/meshes/p3020/4-3.STL" scale="0.001 0.001 0.001" />
-                </geometry>
-            </collision>
-            <collision>
-                <origin xyz="0 0 -1.4043"/>
-                <geometry>
-                    <mesh filename="package://dsr_description2/meshes/p3020/4-4.STL" scale="0.001 0.001 0.001" />
-                </geometry>
-            </collision>
+            <inertial>
+                <mass value="2.836"/>
+                <origin xyz="1.8e-05   -0.010564    -0.12656"/>
+                <inertia ixx="0.01971" ixy="0.0" ixz="0.0" iyy="0.017956" iyz="3.5784e-06" izz="0.017026"/>
+            </inertial>
+            <visual>
+                <origin rpy="1.5708 0 0" xyz="0 1.4043 -0.2351"/>
+                <geometry>
+                    <mesh filename="package://dsr_description2/meshes/p3020/P3020_3_1.STL"
+                        scale="0.001 0.001 0.001"/>
+                </geometry>
+                <material name="dr_white"/>
+            </visual>
+            <visual>
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