Commit message: Refactor controller  (#215)
* Refactor hw_interface & dsr_controller

* Fix launches as being changed workaround param to the standard way

File: dsr_description2/config/macro.transmission.xacro (robot description, xacro)
@@ -9,5 +9,4 @@
 			</joint>
 			<actuator name="motor1">
-				<hardwareInterface>hardware_interface/PositionJointInterface</hardwareInterface>
 				<mechanicalReduction>1</mechanicalReduction>
 			</actuator>
@@ -20,5 +19,4 @@
 			</joint>
 			<actuator name="motor2">
-				<hardwareInterface>hardware_interface/PositionJointInterface</hardwareInterface>
 				<mechanicalReduction>1</mechanicalReduction>
 			</actuator>
@@ -31,5 +29,4 @@
 			</joint>
 			<actuator name="motor3">
-				<hardwareInterface>hardware_interface/PositionJointInterface</hardwareInterface>
 				<mechanicalReduction>1</mechanicalReduction>
 			</actuator>
@@ -42,5 +39,4 @@
 			</joint>
 			<actuator name="motor4">
-				<hardwareInterface>hardware_interface/PositionJointInterface</hardwareInterface>
 				<mechanicalReduction>1</mechanicalReduction>
 			</actuator>
@@ -53,5 +49,4 @@
 			</joint>
 			<actuator name="motor5">
-				<hardwareInterface>hardware_interface/PositionJointInterface</hardwareInterface>
 				<mechanicalReduction>1</mechanicalReduction>
 			</actuator>
@@ -64,5 +59,4 @@
 			</joint>
 			<actuator name="motor6">
-				<hardwareInterface>hardware_interface/PositionJointInterface</hardwareInterface>
 				<mechanicalReduction>1</mechanicalReduction>
 			</actuator>

File: dsr_description2/ros2_control/a0509.ros2_control.xacro (robot description, xacro)
@@ -3,13 +3,9 @@
   <xacro:macro name="a0509_ros2_control" params="
   name
-  rate:=100
-  standby:=true
-  command:=none
   host:=0.0.0.0
+  rt_host:=0.0.0.0
   port:=12345
   mode:=real
   model:=a0509
-  gripper:=none
-  mobile:=none
   ">
     <xacro:property name="double_pi" value="${2.0 * pi}"/>
@@ -19,14 +15,9 @@
       <hardware>
         <plugin>dsr_hardware2/DRHWInterface</plugin>
-        <param name="name">${name}</param>
-        <param name="rate">${rate}</param>
-        <param name="standby">${standby}</param>
-        <param name="command">${command}</param>
         <param name="host">${host}</param>
+        <param name="rt_host">${rt_host}</param>
         <param name="port">${port}</param>
         <param name="mode">${mode}</param>
         <param name="model">${model}</param>
-        <param name="gripper">${gripper}</param>
-        <param name="mobile">${mobile}</param>
       </hardware>
       <joint name="joint_1">

File: dsr_description2/ros2_control/a0912.ros2_control.xacro (robot description, xacro)
@@ -3,13 +3,9 @@
   <xacro:macro name="a0912_ros2_control" params="
   name
-  rate:=100
-  standby:=true
-  command:=none
   host:=0.0.0.0
+  rt_host:=0.0.0.0
   port:=12345
   mode:=real
   model:=a0912
-  gripper:=none
-  mobile:=none
   ">
     <xacro:property name="double_pi" value="${2.0 * pi}"/>
@@ -19,14 +15,9 @@
       <hardware>
         <plugin>dsr_hardware2/DRHWInterface</plugin>
-        <param name="name">${name}</param>
-        <param name="rate">${rate}</param>
-        <param name="standby">${standby}</param>
-        <param name="command">${command}</param>
         <param name="host">${host}</param>
+        <param name="rt_host">${rt_host}</param>
         <param name="port">${port}</param>
         <param name="mode">${mode}</param>
         <param name="model">${model}</param>
-        <param name="gripper">${gripper}</param>
-        <param name="mobile">${mobile}</param>
       </hardware>
       <joint name="joint_1">

File: dsr_description2/ros2_control/e0509.ros2_control.xacro (robot description, xacro)
@@ -3,13 +3,9 @@
   <xacro:macro name="e0509_ros2_control" params="
   name
-  rate:=100
-  standby:=true
-  command:=none
   host:=0.0.0.0
+  rt_host:=0.0.0.0
   port:=12345
   mode:=real
   model:=e0509
-  gripper:=none
-  mobile:=none
   ">
     <xacro:property name="double_pi" value="${2.0 * pi}"/>
@@ -19,14 +15,9 @@
       <hardware>
         <plugin>dsr_hardware2/DRHWInterface</plugin>
-        <param name="name">${name}</param>
-        <param name="rate">${rate}</param>
-        <param name="standby">${standby}</param>
-        <param name="command">${command}</param>
         <param name="host">${host}</param>
+        <param name="rt_host">${rt_host}</param>
         <param name="port">${port}</param>
         <param name="mode">${mode}</param>
         <param name="model">${model}</param>
-        <param name="gripper">${gripper}</param>
-        <param name="mobile">${mobile}</param>
       </hardware>
       <joint name="joint_1">

File: dsr_description2/ros2_control/h2017.ros2_control.xacro (robot description, xacro)
@@ -3,13 +3,9 @@
   <xacro:macro name="h2017_ros2_control" params="
   name
-  rate:=100
-  standby:=true
-  command:=none
   host:=0.0.0.0
+  rt_host:=0.0.0.0
   port:=12345
   mode:=real
   model:=h2017
-  gripper:=none
-  mobile:=none
   ">
     <xacro:property name="double_pi" value="${2.0 * pi}"/>
@@ -19,14 +15,9 @@
       <hardware>
         <plugin>dsr_hardware2/DRHWInterface</plugin>
-        <param name="name">${name}</param>
-        <param name="rate">${rate}</param>
-        <param name="standby">${standby}</param>
-        <param name="command">${command}</param>
         <param name="host">${host}</param>
+        <param name="rt_host">${rt_host}</param>
         <param name="port">${port}</param>
         <param name="mode">${mode}</param>
         <param name="model">${model}</param>
-        <param name="gripper">${gripper}</param>
-        <param name="mobile">${mobile}</param>
       </hardware>
       <joint name="joint_1">

File: dsr_description2/ros2_control/h2515.ros2_control.xacro (robot description, xacro)
@@ -3,13 +3,9 @@
   <xacro:macro name="h2515_ros2_control" params="
   name
-  rate:=100
-  standby:=true
-  command:=none
   host:=0.0.0.0
+  rt_host:=0.0.0.0
   port:=12345
   mode:=real
-  model:=h2017
-  gripper:=none
-  mobile:=none
+  model:=h2515
   ">
     <xacro:property name="double_pi" value="${2.0 * pi}"/>
@@ -19,14 +15,9 @@
       <hardware>
         <plugin>dsr_hardware2/DRHWInterface</plugin>
-        <param name="name">${name}</param>
-        <param name="rate">${rate}</param>
-        <param name="standby">${standby}</param>
-        <param name="command">${command}</param>
         <param name="host">${host}</param>
+        <param name="rt_host">${rt_host}</param>
         <param name="port">${port}</param>
         <param name="mode">${mode}</param>
         <param name="model">${model}</param>
-        <param name="gripper">${gripper}</param>
-        <param name="mobile">${mobile}</param>
       </hardware>
       <joint name="joint_1">

File: dsr_description2/ros2_control/m0609.ros2_control.xacro (robot description, xacro)
@@ -3,13 +3,9 @@
   <xacro:macro name="m0609_ros2_control" params="
   name
-  rate:=100
-  standby:=true
-  command:=none
   host:=0.0.0.0
+  rt_host:=0.0.0.0
   port:=12345
   mode:=real
   model:=m0609
-  gripper:=none
-  mobile:=none
   ">
     <xacro:property name="double_pi" value="${2.0 * pi}"/>
@@ -19,14 +15,9 @@
       <hardware>
         <plugin>dsr_hardware2/DRHWInterface</plugin>
-        <param name="name">${name}</param>
-        <param name="rate">${rate}</param>
-        <param name="standby">${standby}</param>
-        <param name="command">${command}</param>
         <param name="host">${host}</param>
+        <param name="rt_host">${rt_host}</param>
         <param name="port">${port}</param>
         <param name="mode">${mode}</param>
         <param name="model">${model}</param>
-        <param name="gripper">${gripper}</param>
-        <param name="mobile">${mobile}</param>
       </hardware>
       <joint name="joint_1">

File: dsr_description2/ros2_control/m0617.ros2_control.xacro (robot description, xacro)
@@ -3,13 +3,9 @@
   <xacro:macro name="m0617_ros2_control" params="
   name
-  rate:=100
-  standby:=true
-  command:=none
   host:=0.0.0.0
+  rt_host:=0.0.0.0
   port:=12345
   mode:=real
   model:=m0617
-  gripper:=none
-  mobile:=none
   ">
     <xacro:property name="double_pi" value="${2.0 * pi}"/>
@@ -19,14 +15,9 @@
       <hardware>
         <plugin>dsr_hardware2/DRHWInterface</plugin>
-        <param name="name">${name}</param>
-        <param name="rate">${rate}</param>
-        <param name="standby">${standby}</param>
-        <param name="command">${command}</param>
         <param name="host">${host}</param>
+        <param name="rt_host">${rt_host}</param>
         <param name="port">${port}</param>
         <param name="mode">${mode}</param>
         <param name="model">${model}</param>
-        <param name="gripper">${gripper}</param>
-        <param name="mobile">${mobile}</param>
       </hardware>
       <joint name="joint_1">

File: dsr_description2/ros2_control/m1013.ros2_control.xacro (robot description, xacro)
@@ -3,13 +3,11 @@
   <!-- Doosan M1013 ros2_control (arm-only) -->
   <xacro:macro name="m1013_ros2_control" params="
-      name
-      rate:=100
-      standby:=true
-      command:=none
-      host:=127.0.0.1
-      port:=12345
-      mode:=virtual
-      model:=m1013
-      mobile:=none">
+  name
+  host:=0.0.0.0
+  rt_host:=0.0.0.0
+  port:=12345
+  mode:=real
+  model:=m1013
+  ">
     <xacro:property name="double_pi" value="${2.0 * pi}"/>
     <xacro:property name="neg_double_pi" value="${-2.0 * pi}"/>
@@ -17,15 +15,9 @@
       <hardware>
         <plugin>dsr_hardware2/DRHWInterface</plugin>
-        <!-- virtual 테스트면 true 유지 가능 (실기면 false 권장) -->
-        <param name="use_mock_hardware">true</param>
-        <param name="name">${name}</param>
-        <param name="rate">${rate}</param>
-        <param name="standby">${standby}</param>
-        <param name="command">${command}</param>
         <param name="host">${host}</param>
+        <param name="rt_host">${rt_host}</param>
         <param name="port">${port}</param>
         <param name="mode">${mode}</param>
         <param name="model">${model}</param>
-        <param name="mobile">${mobile}</param>
       </hardware>
       <!-- Arm joints only -->

File: dsr_description2/ros2_control/m1509.ros2_control.xacro (robot description, xacro)
@@ -3,13 +3,9 @@
   <xacro:macro name="m1509_ros2_control" params="
   name
-  rate:=100
-  standby:=true
-  command:=none
   host:=0.0.0.0
+  rt_host:=0.0.0.0
   port:=12345
   mode:=real
   model:=m1509
-  gripper:=none
-  mobile:=none
   ">
   <xacro:property name="double_pi" value="${2.0 * pi}"/>
@@ -19,14 +15,9 @@
       <hardware>
         <plugin>dsr_hardware2/DRHWInterface</plugin>
-        <param name="name">${name}</param>
-        <param name="rate">${rate}</param>
-        <param name="standby">${standby}</param>
-        <param name="command">${command}</param>
         <param name="host">${host}</param>
+        <param name="rt_host">${rt_host}</param>
         <param name="port">${port}</param>
         <param name="mode">${mode}</param>
         <param name="model">${model}</param>
-        <param name="gripper">${gripper}</param>
-        <param name="mobile">${mobile}</param>
       </hardware>
       <joint name="joint_1">

File: dsr_description2/ros2_control/p3020.ros2_control.xacro (robot description, xacro)
@@ -3,13 +3,9 @@
   <xacro:macro name="p3020_ros2_control" params="
   name
-  rate:=100
-  standby:=true
-  command:=none
   host:=0.0.0.0
+  rt_host:=0.0.0.0
   port:=12345
   mode:=real
   model:=p3020
-  gripper:=none
-  mobile:=none
   ">
     <xacro:property name="double_pi" value="${2.0 * pi}"/>
@@ -19,14 +15,9 @@
       <hardware>
         <plugin>dsr_hardware2/DRHWInterface</plugin>
-        <param name="name">${name}</param>
-        <param name="rate">${rate}</param>
-        <param name="standby">${standby}</param>
-        <param name="command">${command}</param>
         <param name="host">${host}</param>
+        <param name="rt_host">${rt_host}</param>
         <param name="port">${port}</param>
         <param name="mode">${mode}</param>
         <param name="model">${model}</param>
-        <param name="gripper">${gripper}</param>
-        <param name="mobile">${mobile}</param>
       </hardware>
       <joint name="joint_1">

File: dsr_description2/xacro/a0509.urdf.xacro (robot description, xacro)
@@ -9,7 +9,17 @@
   <xacro:arg name="gripper_parent_link"  default="link_6"/>
   <xacro:arg name="use_gazebo" default="false"/>
-  <xacro:property name="gz" value="$(arg use_gazebo)"/>
+  <xacro:arg name="host" default=""/>
+  <xacro:arg name="port" default=""/>
+  <xacro:arg name="rt_host" default=""/>
+  <xacro:arg name="mode" default=""/>
+  <xacro:arg name="model" default=""/>
   <xacro:property name="cr" value="$(arg color)"/>
   <xacro:property name="gr" value="$(arg gripper)"/>
+  <xacro:property name="gz" value="$(arg use_gazebo)"/>
+  <xacro:property name="host" value="$(arg host)"/>
+  <xacro:property name="rt_host" value="$(arg rt_host)"/>
+  <xacro:property name="port" value="$(arg port)"/>
+  <xacro:property name="mode" value="$(arg mode)"/>
+  <xacro:property name="model" value="$(arg model)"/>
   <xacro:if value="${cr == 'white'}">
     <xacro:include filename="$(find dsr_description2)/xacro/macro.a0509.white.xacro"/>
@@ -30,6 +40,12 @@
   </xacro:if>
   <xacro:unless value="${gz}">
-    <xacro:include filename="$(find dsr_description2)/ros2_control/a0509.ros2_control.xacro"/>
-    <xacro:a0509_ros2_control name="a0509"/>
+    <xacro:include filename="$(find dsr_description2)/ros2_control/a0509.ros2_control.xacro" />
+    <xacro:a0509_ros2_control name="a0509"
+      host="${host}"
+      rt_host="${rt_host}"
+      port="${port}"
+      mode="${mode}"
+      model="${model}"
+    />
   </xacro:unless>
   <xacro:if value="${gr == 'robotiq_2f85'}">

File: dsr_description2/xacro/a0912.urdf.xacro (robot description, xacro)
@@ -9,7 +9,17 @@
   <xacro:arg name="gripper_parent_link"  default="link_6"/>
   <xacro:arg name="use_gazebo" default="false"/>
-  <xacro:property name="gz" value="$(arg use_gazebo)"/>
+  <xacro:arg name="host" default=""/>
+  <xacro:arg name="port" default=""/>
+  <xacro:arg name="rt_host" default=""/>
+  <xacro:arg name="mode" default=""/>
+  <xacro:arg name="model" default=""/>
   <xacro:property name="cr" value="$(arg color)"/>
   <xacro:property name="gr" value="$(arg gripper)"/>
+  <xacro:property name="gz" value="$(arg use_gazebo)"/>
+  <xacro:property name="host" value="$(arg host)"/>
+  <xacro:property name="rt_host" value="$(arg rt_host)"/>
+  <xacro:property name="port" value="$(arg port)"/>
+  <xacro:property name="mode" value="$(arg mode)"/>
+  <xacro:property name="model" value="$(arg model)"/>
   <xacro:if value="${cr == 'white'}">
     <xacro:include filename="$(find dsr_description2)/xacro/macro.a0912.white.xacro"/>
@@ -30,6 +40,12 @@
   </xacro:if>
   <xacro:unless value="${gz}">
-    <xacro:include filename="$(find dsr_description2)/ros2_control/a0912.ros2_control.xacro"/>
-    <xacro:a0912_ros2_control name="a0912"/>
+    <xacro:include filename="$(find dsr_description2)/ros2_control/a0912.ros2_control.xacro" />
+    <xacro:a0912_ros2_control name="a0912"
+      host="${host}"
+      rt_host="${rt_host}"
+      port="${port}"
+      mode="${mode}"
+      model="${model}"
+    />
   </xacro:unless>
   <xacro:if value="${gr == 'robotiq_2f85'}">

File: dsr_description2/xacro/e0509.urdf.xacro (robot description, xacro)
@@ -9,7 +9,17 @@
   <xacro:arg name="gripper_parent_link"  default="link_6"/>
   <xacro:arg name="use_gazebo" default="false"/>
-  <xacro:property name="gz" value="$(arg use_gazebo)"/>
+  <xacro:arg name="host" default=""/>
+  <xacro:arg name="port" default=""/>
+  <xacro:arg name="rt_host" default=""/>
+  <xacro:arg name="mode" default=""/>
+  <xacro:arg name="model" default=""/>
   <xacro:property name="cr" value="$(arg color)"/>
   <xacro:property name="gr" value="$(arg gripper)"/>
+  <xacro:property name="gz" value="$(arg use_gazebo)"/>
+  <xacro:property name="host" value="$(arg host)"/>
+  <xacro:property name="rt_host" value="$(arg rt_host)"/>
+  <xacro:property name="port" value="$(arg port)"/>
+  <xacro:property name="mode" value="$(arg mode)"/>
+  <xacro:property name="model" value="$(arg model)"/>
   <xacro:if value="${cr == 'white'}">
     <xacro:include filename="$(find dsr_description2)/xacro/macro.e0509.white.xacro"/>
@@ -30,6 +40,13 @@
   </xacro:if>
   <xacro:unless value="${gz}">
-    <xacro:include filename="$(find dsr_description2)/ros2_control/e0509.ros2_control.xacro"/>
-    <xacro:e0509_ros2_control name="e0509"/>
+    <xacro:include filename="$(find dsr_description2)/ros2_control/e0509.ros2_control.xacro" />
+    <xacro:e0509_ros2_control
+      name="e0509"
+      host="${host}"
+      rt_host="${rt_host}"
+      port="${port}"
+      mode="${mode}"
+      model="${model}"
+    />
   </xacro:unless>
   <xacro:if value="${gr == 'robotiq_2f85'}">

File: dsr_description2/xacro/h2017.urdf.xacro (robot description, xacro)
@@ -9,7 +9,17 @@
   <xacro:arg name="gripper_parent_link"  default="link_6"/>
   <xacro:arg name="use_gazebo" default="false"/>
-  <xacro:property name="gz" value="$(arg use_gazebo)"/>
+  <xacro:arg name="host" default=""/>
+  <xacro:arg name="port" default=""/>
+  <xacro:arg name="rt_host" default=""/>
+  <xacro:arg name="mode" default=""/>
+  <xacro:arg name="model" default=""/>
   <xacro:property name="cr" value="$(arg color)"/>
   <xacro:property name="gr" value="$(arg gripper)"/>
+  <xacro:property name="gz" value="$(arg use_gazebo)"/>
+  <xacro:property name="host" value="$(arg host)"/>
+  <xacro:property name="rt_host" value="$(arg rt_host)"/>
+  <xacro:property name="port" value="$(arg port)"/>
+  <xacro:property name="mode" value="$(arg mode)"/>
+  <xacro:property name="model" value="$(arg model)"/>
   <xacro:if value="${cr == 'white'}">
     <xacro:include filename="$(find dsr_description2)/xacro/macro.h2017.white.xacro"/>
@@ -30,6 +40,13 @@
   </xacro:if>
   <xacro:unless value="${gz}">
-    <xacro:include filename="$(find dsr_description2)/ros2_control/h2017.ros2_control.xacro"/>
-    <xacro:h2017_ros2_control name="h2017"/>
+    <xacro:include filename="$(find dsr_description2)/ros2_control/h2017.ros2_control.xacro" />
+    <xacro:h2017_ros2_control
+      name="h2017"
+      host="${host}"
+      rt_host="${rt_host}"
+      port="${port}"
+      mode="${mode}"
+      model="${model}"
+    />
   </xacro:unless>
   <xacro:if value="${gr == 'robotiq_2f85'}">

File: dsr_description2/xacro/h2515.urdf.xacro (robot description, xacro)
@@ -9,7 +9,17 @@
   <xacro:arg name="gripper_parent_link"  default="link_6"/>
   <xacro:arg name="use_gazebo" default="false"/>
-  <xacro:property name="gz" value="$(arg use_gazebo)"/>
+  <xacro:arg name="host" default=""/>
+  <xacro:arg name="port" default=""/>
+  <xacro:arg name="rt_host" default=""/>
+  <xacro:arg name="mode" default=""/>
+  <xacro:arg name="model" default=""/>
   <xacro:property name="cr" value="$(arg color)"/>
   <xacro:property name="gr" value="$(arg gripper)"/>
+  <xacro:property name="gz" value="$(arg use_gazebo)"/>
+  <xacro:property name="host" value="$(arg host)"/>
+  <xacro:property name="rt_host" value="$(arg rt_host)"/>
+  <xacro:property name="port" value="$(arg port)"/>
+  <xacro:property name="mode" value="$(arg mode)"/>
+  <xacro:property name="model" value="$(arg model)"/>
   <xacro:if value="${cr == 'white'}">
     <xacro:include filename="$(find dsr_description2)/xacro/macro.h2515.white.xacro"/>
@@ -30,6 +40,13 @@
   </xacro:if>
   <xacro:unless value="${gz}">
-    <xacro:include filename="$(find dsr_description2)/ros2_control/h2515.ros2_control.xacro"/>
-    <xacro:h2515_ros2_control name="h2515"/>
+    <xacro:include filename="$(find dsr_description2)/ros2_control/h2515.ros2_control.xacro" />
+    <xacro:h2515_ros2_control
+      name="h2515"
+      host="${host}"
+      rt_host="${rt_host}"
+      port="${port}"
+      mode="${mode}"
+      model="${model}"
+    />
   </xacro:unless>
   <xacro:if value="${gr == 'robotiq_2f85'}">

File: dsr_description2/xacro/m0609.urdf.xacro (robot description, xacro)
@@ -9,7 +9,17 @@
   <xacro:arg name="gripper_parent_link"  default="link_6"/>
   <xacro:arg name="use_gazebo" default="false"/>
+  <xacro:arg name="host" default=""/>
+  <xacro:arg name="port" default=""/>
+  <xacro:arg name="rt_host" default=""/>
+  <xacro:arg name="mode" default=""/>
+  <xacro:arg name="model" default=""/>
   <xacro:property name="gz" value="$(arg use_gazebo)"/>
   <xacro:property name="cr" value="$(arg color)"/>
   <xacro:property name="gr" value="$(arg gripper)"/>
+  <xacro:property name="host" value="$(arg host)"/>
+  <xacro:property name="rt_host" value="$(arg rt_host)"/>
+  <xacro:property name="port" value="$(arg port)"/>
+  <xacro:property name="mode" value="$(arg mode)"/>
+  <xacro:property name="model" value="$(arg model)"/>
   <xacro:if value="${cr == 'white'}">
     <xacro:include filename="$(find dsr_description2)/xacro/macro.m0609.white.xacro"/>
@@ -30,6 +40,13 @@
   </xacro:if>
   <xacro:unless value="${gz}">
-    <xacro:include filename="$(find dsr_description2)/ros2_control/m0609.ros2_control.xacro"/>
-    <xacro:m0609_ros2_control name="m0609"/>
+    <xacro:include filename="$(find dsr_description2)/ros2_control/m0609.ros2_control.xacro" />
+    <xacro:m0609_ros2_control
+      name="m0609"
+      host="${host}"
+      rt_host="${rt_host}"
+      port="${port}"
+      mode="${mode}"
+      model="${model}"
+    />
   </xacro:unless>
   <xacro:if value="${gr == 'robotiq_2f85'}">

File: dsr_description2/xacro/m0617.urdf.xacro (robot description, xacro)
@@ -9,7 +9,17 @@
   <xacro:arg name="gripper_parent_link"  default="link_6"/>
   <xacro:arg name="use_gazebo" default="false"/>
-  <xacro:property name="gz" value="$(arg use_gazebo)"/>
+  <xacro:arg name="host" default=""/>
+  <xacro:arg name="port" default=""/>
+  <xacro:arg name="rt_host" default=""/>
+  <xacro:arg name="mode" default=""/>
+  <xacro:arg name="model" default=""/>
   <xacro:property name="cr" value="$(arg color)"/>
   <xacro:property name="gr" value="$(arg gripper)"/>
+  <xacro:property name="gz" value="$(arg use_gazebo)"/>
+  <xacro:property name="host" value="$(arg host)"/>
+  <xacro:property name="rt_host" value="$(arg rt_host)"/>
+  <xacro:property name="port" value="$(arg port)"/>
+  <xacro:property name="mode" value="$(arg mode)"/>
+  <xacro:property name="model" value="$(arg model)"/>
   <xacro:if value="${cr == 'white'}">
     <xacro:include filename="$(find dsr_description2)/xacro/macro.m0617.white.xacro"/>
@@ -30,6 +40,13 @@
   </xacro:if>
   <xacro:unless value="${gz}">
-    <xacro:include filename="$(find dsr_description2)/ros2_control/m0617.ros2_control.xacro"/>
-    <xacro:m0617_ros2_control name="m0617"/>
+    <xacro:include filename="$(find dsr_description2)/ros2_control/m0617.ros2_control.xacro" />
+    <xacro:m0617_ros2_control
+      name="m0617"
+      host="${host}"
+      rt_host="${rt_host}"
+      port="${port}"
+      mode="${mode}"
+      model="${model}"
+    />
   </xacro:unless>
   <xacro:if value="${gr == 'robotiq_2f85'}">
