Commit message: Refactor controller  (#215)
* Refactor hw_interface & dsr_controller

* Fix launches as being changed workaround param to the standard way

File: dsr_description2/xacro/m1013.urdf.xacro (robot description, xacro)
@@ -9,7 +9,17 @@
   <xacro:arg name="gripper_parent_link"  default="link_6"/>
   <xacro:arg name="use_gazebo" default="false"/>
-  <xacro:property name="gz" value="$(arg use_gazebo)"/>
+  <xacro:arg name="host" default=""/>
+  <xacro:arg name="port" default=""/>
+  <xacro:arg name="rt_host" default=""/>
+  <xacro:arg name="mode" default=""/>
+  <xacro:arg name="model" default=""/>
   <xacro:property name="cr" value="$(arg color)"/>
   <xacro:property name="gr" value="$(arg gripper)"/>
+  <xacro:property name="gz" value="$(arg use_gazebo)"/>
+  <xacro:property name="host" value="$(arg host)"/>
+  <xacro:property name="rt_host" value="$(arg rt_host)"/>
+  <xacro:property name="port" value="$(arg port)"/>
+  <xacro:property name="mode" value="$(arg mode)"/>
+  <xacro:property name="model" value="$(arg model)"/>
   <xacro:if value="${cr == 'white'}">
     <xacro:include filename="$(find dsr_description2)/xacro/macro.m1013.white.xacro"/>
@@ -30,6 +40,13 @@
   </xacro:if>
   <xacro:unless value="${gz}">
-    <xacro:include filename="$(find dsr_description2)/ros2_control/m1013.ros2_control.xacro"/>
-    <xacro:m1013_ros2_control name="m1013"/>
+    <xacro:include filename="$(find dsr_description2)/ros2_control/m1013.ros2_control.xacro" />
+    <xacro:m1013_ros2_control
+      name="m1013"
+      host="${host}"
+      rt_host="${rt_host}"
+      port="${port}"
+      mode="${mode}"
+      model="${model}"
+    />
   </xacro:unless>
   <xacro:if value="${gr == 'robotiq_2f85'}">

File: dsr_description2/xacro/m1509.urdf.xacro (robot description, xacro)
@@ -1,7 +1,13 @@
 <?xml version="1.0"?>
 <robot xmlns:xacro="http://www.ros.org/wiki/xacro" name="m1509" >
-  <xacro:arg name="mode"           default="virtual"/>
-  <xacro:arg name="color"          default="white"/>
-  <xacro:arg name="namespace"      default=""/>
+  <xacro:arg name="color"   default="white"/>
+  <xacro:arg name="gripper" default="none"/>
+  <xacro:arg name="namespace" default=""/>
+  <xacro:arg name="use_gazebo" default="false"/>
+  <xacro:arg name="host" default=""/>
+  <xacro:arg name="port" default=""/>
+  <xacro:arg name="rt_host" default=""/>
+  <xacro:arg name="mode" default=""/>
+  <xacro:arg name="model" default=""/>
   <!-- gripper control argument -->
   <xacro:arg name="gripper"              default="none"/>         <!-- none | robotique -->
@@ -10,4 +16,9 @@
   <xacro:arg name="use_gazebo" default="false"/>
   <xacro:property name="gz" value="$(arg use_gazebo)"/>
+  <xacro:property name="host" value="$(arg host)"/>
+  <xacro:property name="rt_host" value="$(arg rt_host)"/>
+  <xacro:property name="port" value="$(arg port)"/>
+  <xacro:property name="mode" value="$(arg mode)"/>
+  <xacro:property name="model" value="$(arg model)"/>
   <xacro:property name="cr" value="$(arg color)"/>
   <xacro:property name="gr" value="$(arg gripper)"/>
@@ -30,6 +41,13 @@
   </xacro:if>
   <xacro:unless value="${gz}">
-    <xacro:include filename="$(find dsr_description2)/ros2_control/m1509.ros2_control.xacro"/>
-    <xacro:m1509_ros2_control name="m1509"/>
+    <xacro:include filename="$(find dsr_description2)/ros2_control/m1509.ros2_control.xacro" />
+    <xacro:m1509_ros2_control
+      name="m1509"
+      host="${host}"
+      rt_host="${rt_host}"
+      port="${port}"
+      mode="${mode}"
+      model="${model}"
+    />
   </xacro:unless>
   <xacro:if value="${gr == 'robotiq_2f85'}">
