Commit message: Update hardware interface (on_init, read, write) - Added dynamic joint index mapping (hw_mapping_) in on_init. - Updated read() and write() to use hardware index mapping instead of fixed joint order. - Improved position and velocity command alignment for non-6DOF models. - Updated all model-specific ros2_control and transmission xacro files.

File: dsr_description2/config/macro.transmission.xacro (robot description, xacro)
@@ -1,71 +1,59 @@
 <?xml version="1.0"?>
 <robot xmlns:xacro="http://www.ros.org/wiki/xacro">
-	<xacro:macro name="dsr_transmission">
-		<!-- Transmission 1 -->
-		<transmission name="tran1">
-			<type>transmission_interface/SimpleTransmission</type>
-			<joint name="joint1">
-				<hardwareInterface>hardware_interface/PositionJointInterface</hardwareInterface>
-			</joint>
-			<actuator name="motor1">
-				<hardwareInterface>hardware_interface/PositionJointInterface</hardwareInterface>
-				<mechanicalReduction>1</mechanicalReduction>
-			</actuator>
-		</transmission>
-		<!-- Transmission 2 -->
-		<transmission name="tran2">
-			<type>transmission_interface/SimpleTransmission</type>
-			<joint name="joint2">
-				<hardwareInterface>hardware_interface/PositionJointInterface</hardwareInterface>
-			</joint>
-			<actuator name="motor2">
-				<hardwareInterface>hardware_interface/PositionJointInterface</hardwareInterface>
-				<mechanicalReduction>1</mechanicalReduction>
-			</actuator>
-		</transmission>
-		<!-- Transmission 3 -->
-		<transmission name="tran3">
-			<type>transmission_interface/SimpleTransmission</type>
-			<joint name="joint3">
-				<hardwareInterface>hardware_interface/PositionJointInterface</hardwareInterface>
-			</joint>
-			<actuator name="motor3">
-				<hardwareInterface>hardware_interface/PositionJointInterface</hardwareInterface>
-				<mechanicalReduction>1</mechanicalReduction>
-			</actuator>
-		</transmission>
-		<!-- Transmission 4 -->
-		<transmission name="tran4">
-			<type>transmission_interface/SimpleTransmission</type>
-			<joint name="joint4">
-				<hardwareInterface>hardware_interface/PositionJointInterface</hardwareInterface>
-			</joint>
-			<actuator name="motor4">
-				<hardwareInterface>hardware_interface/PositionJointInterface</hardwareInterface>
-				<mechanicalReduction>1</mechanicalReduction>
-			</actuator>
-		</transmission>
-		<!-- Transmission 5 -->
-		<transmission name="tran5">
-			<type>transmission_interface/SimpleTransmission</type>
-			<joint name="joint5">
-				<hardwareInterface>hardware_interface/PositionJointInterface</hardwareInterface>
-			</joint>
-			<actuator name="motor5">
-				<hardwareInterface>hardware_interface/PositionJointInterface</hardwareInterface>
-				<mechanicalReduction>1</mechanicalReduction>
-			</actuator>
-		</transmission>
-		<!-- Transmission 6 -->
-		<transmission name="tran6">
-			<type>transmission_interface/SimpleTransmission</type>
-			<joint name="joint6">
-				<hardwareInterface>hardware_interface/PositionJointInterface</hardwareInterface>
-			</joint>
-			<actuator name="motor6">
-				<hardwareInterface>hardware_interface/PositionJointInterface</hardwareInterface>
-				<mechanicalReduction>1</mechanicalReduction>
-			</actuator>
-		</transmission>
-	</xacro:macro>
+  <!--
+    DSR Transmission (ROS2 Control Style)
+    - ROS1의 transmission_interface/SimpleTransmission 제거
+    - 각 joint에 ros2_control command/state_interface 명시
+    - hardware_interface::SystemInterface(DRHWInterface)와 직접 매핑
+  -->
+  <xacro:macro name="dsr_transmission">
+    <!-- Joint1 -->
+    <joint name="joint1" type="revolute">
+      <ros2_control>
+        <command_interface name="position"/>
+        <state_interface name="position"/>
+        <state_interface name="velocity"/>
+      </ros2_control>
+    </joint>
+    <!-- Joint2 -->
+    <joint name="joint2" type="revolute">
+      <ros2_control>
+        <command_interface name="position"/>
+        <state_interface name="position"/>
+        <state_interface name="velocity"/>
+      </ros2_control>
+    </joint>
+    <!-- Joint3 -->
+    <joint name="joint3" type="revolute">
+      <ros2_control>
+        <command_interface name="position"/>
+        <state_interface name="position"/>
+        <state_interface name="velocity"/>
+      </ros2_control>
+    </joint>
+    <!-- Joint4 -->
+    <joint name="joint4" type="revolute">
+      <ros2_control>
+        <command_interface name="position"/>
+        <state_interface name="position"/>
+        <state_interface name="velocity"/>
+      </ros2_control>
+    </joint>
+    <!-- Joint5 -->
+    <joint name="joint5" type="revolute">
+      <ros2_control>
+        <command_interface name="position"/>
+        <state_interface name="position"/>
+        <state_interface name="velocity"/>
+      </ros2_control>
+    </joint>
+    <!-- Joint6 -->
+    <joint name="joint6" type="revolute">
+      <ros2_control>
+        <command_interface name="position"/>
+        <state_interface name="position"/>
+        <state_interface name="velocity"/>
+      </ros2_control>
+    </joint>
+  </xacro:macro>
 </robot>

File: dsr_description2/ros2_control/a0912.ros2_control.xacro (robot description, xacro)
@@ -4,5 +4,5 @@
   name
   rate:=100
-  standby:=ture
+  standby:=true
   command:=none
   host:=0.0.0.0
@@ -13,4 +13,7 @@
   mobile:=none
   ">
+    <xacro:property name="double_pi" value="${2.0 * pi}"/>
+    <xacro:property name="neg_double_pi" value="${-2.0 * pi}"/>
+    <xacro:property name="neg_pi" value="${-1.0 * pi}"/>
     <ros2_control name="${name}" type="system">
       <hardware>
@@ -29,6 +32,6 @@
       <joint name="joint_1">
         <command_interface name="position">
-          <param name="min">{-2*pi}</param>
-          <param name="max">{2*pi}</param>
+          <param name="min">${neg_double_pi}</param>
+          <param name="max">${double_pi}</param>
         </command_interface>
         <command_interface name="velocity">
@@ -43,6 +46,6 @@
       <joint name="joint_2">
         <command_interface name="position">
-          <param name="min">{-2*pi}</param>
-          <param name="max">{2*pi}</param>
+          <param name="min">${neg_double_pi}</param>
+          <param name="max">${double_pi}</param>
         </command_interface>
         <command_interface name="velocity">
@@ -57,6 +60,6 @@
       <joint name="joint_3">
         <command_interface name="position">
-          <param name="min">{-pi}</param>
-          <param name="max">{pi}</param>
+          <param name="min">${neg_pi}</param>
+          <param name="max">${pi}</param>
         </command_interface>
         <command_interface name="velocity">
@@ -71,6 +74,6 @@
       <joint name="joint_4">
         <command_interface name="position">
-          <param name="min">{-2*pi}</param>
-          <param name="max">{2*pi}</param>
+          <param name="min">${neg_double_pi}</param>
+          <param name="max">${double_pi}</param>
         </command_interface>
         <command_interface name="velocity">
@@ -85,6 +88,6 @@
       <joint name="joint_5">
         <command_interface name="position">
-          <param name="min">{-2*pi}</param>
-          <param name="max">{2*pi}</param>
+          <param name="min">${neg_double_pi}</param>
+          <param name="max">${double_pi}</param>
         </command_interface>
         <command_interface name="velocity">
@@ -99,6 +102,6 @@
       <joint name="joint_6">
         <command_interface name="position">
-          <param name="min">{-2*pi}</param>
-          <param name="max">{2*pi}</param>
+          <param name="min">${neg_double_pi}</param>
+          <param name="max">${double_pi}</param>
         </command_interface>
         <command_interface name="velocity">

File: dsr_description2/ros2_control/e0509.ros2_control.xacro (robot description, xacro)
@@ -4,5 +4,5 @@
   name
   rate:=100
-  standby:=ture
+  standby:=true
   command:=none
   host:=0.0.0.0
@@ -13,4 +13,7 @@
   mobile:=none
   ">
+    <xacro:property name="double_pi" value="${2.0 * pi}"/>
+    <xacro:property name="neg_double_pi" value="${-2.0 * pi}"/>
+    <xacro:property name="neg_pi" value="${-1.0 * pi}"/>
     <ros2_control name="${name}" type="system">
       <hardware>
@@ -29,6 +32,6 @@
       <joint name="joint_1">
         <command_interface name="position">
-          <param name="min">{-2*pi}</param>
-          <param name="max">{2*pi}</param>
+          <param name="min">${neg_double_pi}</param>
+          <param name="max">${double_pi}</param>
         </command_interface>
         <command_interface name="velocity">
@@ -43,6 +46,6 @@
       <joint name="joint_2">
         <command_interface name="position">
-          <param name="min">{-2*pi}</param>
-          <param name="max">{2*pi}</param>
+          <param name="min">${neg_double_pi}</param>
+          <param name="max">${double_pi}</param>
         </command_interface>
         <command_interface name="velocity">
@@ -57,6 +60,6 @@
       <joint name="joint_3">
         <command_interface name="position">
-          <param name="min">{-pi}</param>
-          <param name="max">{pi}</param>
+          <param name="min">${neg_pi}</param>
+          <param name="max">${pi}</param>
         </command_interface>
         <command_interface name="velocity">
@@ -71,6 +74,6 @@
       <joint name="joint_4">
         <command_interface name="position">
-          <param name="min">{-2*pi}</param>
-          <param name="max">{2*pi}</param>
+          <param name="min">${neg_double_pi}</param>
+          <param name="max">${double_pi}</param>
         </command_interface>
         <command_interface name="velocity">
@@ -85,6 +88,6 @@
       <joint name="joint_5">
         <command_interface name="position">
-          <param name="min">{-2*pi}</param>
-          <param name="max">{2*pi}</param>
+          <param name="min">${neg_double_pi}</param>
+          <param name="max">${double_pi}</param>
         </command_interface>
         <command_interface name="velocity">
@@ -99,6 +102,6 @@
       <joint name="joint_6">
         <command_interface name="position">
-          <param name="min">{-2*pi}</param>
-          <param name="max">{2*pi}</param>
+          <param name="min">${neg_double_pi}</param>
+          <param name="max">${double_pi}</param>
         </command_interface>
         <command_interface name="velocity">

File: dsr_description2/ros2_control/h2017.ros2_control.xacro (robot description, xacro)
@@ -4,5 +4,5 @@
   name
   rate:=100
-  standby:=ture
+  standby:=true
   command:=none
   host:=0.0.0.0
@@ -13,4 +13,7 @@
   mobile:=none
   ">
+    <xacro:property name="double_pi" value="${2.0 * pi}"/>
+    <xacro:property name="neg_double_pi" value="${-2.0 * pi}"/>
+    <xacro:property name="neg_pi" value="${-1.0 * pi}"/>
     <ros2_control name="${name}" type="system">
       <hardware>
@@ -29,6 +32,6 @@
       <joint name="joint_1">
         <command_interface name="position">
-          <param name="min">{-2*pi}</param>
-          <param name="max">{2*pi}</param>
+          <param name="min">${neg_double_pi}</param>
+          <param name="max">${double_pi}</param>
         </command_interface>
         <command_interface name="velocity">
@@ -43,6 +46,6 @@
       <joint name="joint_2">
         <command_interface name="position">
-          <param name="min">{-2*pi}</param>
-          <param name="max">{2*pi}</param>
+          <param name="min">${neg_double_pi}</param>
+          <param name="max">${double_pi}</param>
         </command_interface>
         <command_interface name="velocity">
@@ -57,6 +60,6 @@
       <joint name="joint_3">
         <command_interface name="position">
-          <param name="min">{-pi}</param>
-          <param name="max">{pi}</param>
+          <param name="min">${neg_pi}</param>
+          <param name="max">${pi}</param>
         </command_interface>
         <command_interface name="velocity">
@@ -71,6 +74,6 @@
       <joint name="joint_4">
         <command_interface name="position">
-          <param name="min">{-2*pi}</param>
-          <param name="max">{2*pi}</param>
+          <param name="min">${neg_double_pi}</param>
+          <param name="max">${double_pi}</param>
         </command_interface>
         <command_interface name="velocity">
@@ -85,6 +88,6 @@
       <joint name="joint_5">
         <command_interface name="position">
-          <param name="min">{-2*pi}</param>
-          <param name="max">{2*pi}</param>
+          <param name="min">${neg_double_pi}</param>
+          <param name="max">${double_pi}</param>
         </command_interface>
         <command_interface name="velocity">
@@ -99,6 +102,6 @@
       <joint name="joint_6">
         <command_interface name="position">
-          <param name="min">{-2*pi}</param>
-          <param name="max">{2*pi}</param>
+          <param name="min">${neg_double_pi}</param>
+          <param name="max">${double_pi}</param>
         </command_interface>
         <command_interface name="velocity">

File: dsr_description2/ros2_control/h2515.ros2_control.xacro (robot description, xacro)
@@ -4,13 +4,16 @@
   name
   rate:=100
-  standby:=ture
+  standby:=true
   command:=none
   host:=0.0.0.0
   port:=12345
   mode:=real
-  model:=h2515
+  model:=h2017
   gripper:=none
   mobile:=none
   ">
+    <xacro:property name="double_pi" value="${2.0 * pi}"/>
+    <xacro:property name="neg_double_pi" value="${-2.0 * pi}"/>
+    <xacro:property name="neg_pi" value="${-1.0 * pi}"/>
     <ros2_control name="${name}" type="system">
       <hardware>
@@ -29,6 +32,6 @@
       <joint name="joint_1">
         <command_interface name="position">
-          <param name="min">{-2*pi}</param>
-          <param name="max">{2*pi}</param>
+          <param name="min">${neg_double_pi}</param>
+          <param name="max">${double_pi}</param>
         </command_interface>
         <command_interface name="velocity">
@@ -43,6 +46,6 @@
       <joint name="joint_2">
         <command_interface name="position">
-          <param name="min">{-2*pi}</param>
-          <param name="max">{2*pi}</param>
+          <param name="min">${neg_double_pi}</param>
+          <param name="max">${double_pi}</param>
         </command_interface>
         <command_interface name="velocity">
@@ -57,6 +60,6 @@
       <joint name="joint_3">
         <command_interface name="position">
-          <param name="min">{-pi}</param>
-          <param name="max">{pi}</param>
+          <param name="min">${neg_pi}</param>
+          <param name="max">${pi}</param>
         </command_interface>
         <command_interface name="velocity">
@@ -66,11 +69,11 @@
         <state_interface name="position">
           <param name="initial_value">0.0</param>
-        </state_interface>
+        </state_interface> <!-- FIXED: missing closing tag -->
         <state_interface name="velocity"/>
       </joint>
       <joint name="joint_4">
         <command_interface name="position">
-          <param name="min">{-2*pi}</param>
-          <param name="max">{2*pi}</param>
+          <param name="min">${neg_double_pi}</param>
+          <param name="max">${double_pi}</param>
         </command_interface>
         <command_interface name="velocity">
@@ -85,6 +88,6 @@
       <joint name="joint_5">
         <command_interface name="position">
-          <param name="min">{-2*pi}</param>
-          <param name="max">{2*pi}</param>
+          <param name="min">${neg_double_pi}</param>
+          <param name="max">${double_pi}</param>
         </command_interface>
         <command_interface name="velocity">
@@ -99,6 +102,6 @@
       <joint name="joint_6">
         <command_interface name="position">
-          <param name="min">{-2*pi}</param>
-          <param name="max">{2*pi}</param>
+          <param name="min">${neg_double_pi}</param>
+          <param name="max">${double_pi}</param>
         </command_interface>
         <command_interface name="velocity">

File: dsr_description2/ros2_control/m0609.ros2_control.xacro (robot description, xacro)
@@ -4,5 +4,5 @@
   name
   rate:=100
-  standby:=ture
+  standby:=true
   command:=none
   host:=0.0.0.0
@@ -13,4 +13,7 @@
   mobile:=none
   ">
+    <xacro:property name="double_pi" value="${2.0 * pi}"/>
+    <xacro:property name="neg_double_pi" value="${-2.0 * pi}"/>
+    <xacro:property name="neg_pi" value="${-1.0 * pi}"/>
     <ros2_control name="${name}" type="system">
       <hardware>
@@ -29,6 +32,6 @@
       <joint name="joint_1">
         <command_interface name="position">
-          <param name="min">{-2*pi}</param>
-          <param name="max">{2*pi}</param>
+          <param name="min">${neg_double_pi}</param>
+          <param name="max">${double_pi}</param>
         </command_interface>
         <command_interface name="velocity">
@@ -43,6 +46,6 @@
       <joint name="joint_2">
         <command_interface name="position">
-          <param name="min">{-2*pi}</param>
-          <param name="max">{2*pi}</param>
+          <param name="min">${neg_double_pi}</param>
+          <param name="max">${double_pi}</param>
         </command_interface>
         <command_interface name="velocity">
@@ -57,6 +60,6 @@
       <joint name="joint_3">
         <command_interface name="position">
-          <param name="min">{-pi}</param>
-          <param name="max">{pi}</param>
+          <param name="min">${neg_pi}</param>
+          <param name="max">${pi}</param>
         </command_interface>
         <command_interface name="velocity">
@@ -71,6 +74,6 @@
       <joint name="joint_4">
         <command_interface name="position">
-          <param name="min">{-2*pi}</param>
-          <param name="max">{2*pi}</param>
+          <param name="min">${neg_double_pi}</param>
+          <param name="max">${double_pi}</param>
         </command_interface>
         <command_interface name="velocity">
@@ -85,6 +88,6 @@
       <joint name="joint_5">
         <command_interface name="position">
-          <param name="min">{-2*pi}</param>
-          <param name="max">{2*pi}</param>
+          <param name="min">${neg_double_pi}</param>
+          <param name="max">${double_pi}</param>
         </command_interface>
         <command_interface name="velocity">
@@ -99,6 +102,6 @@
       <joint name="joint_6">
         <command_interface name="position">
-          <param name="min">{-2*pi}</param>
-          <param name="max">{2*pi}</param>
+          <param name="min">${neg_double_pi}</param>
+          <param name="max">${double_pi}</param>
         </command_interface>
         <command_interface name="velocity">

File: dsr_description2/ros2_control/m0617.ros2_control.xacro (robot description, xacro)
@@ -4,5 +4,5 @@
   name
   rate:=100
-  standby:=ture
+  standby:=true
   command:=none
   host:=0.0.0.0
@@ -13,4 +13,7 @@
   mobile:=none
   ">
+    <xacro:property name="double_pi" value="${2.0 * pi}"/>
+    <xacro:property name="neg_double_pi" value="${-2.0 * pi}"/>
+    <xacro:property name="neg_pi" value="${-1.0 * pi}"/>
     <ros2_control name="${name}" type="system">
       <hardware>
@@ -29,6 +32,6 @@
       <joint name="joint_1">
         <command_interface name="position">
-          <param name="min">{-2*pi}</param>
-          <param name="max">{2*pi}</param>
+          <param name="min">${neg_double_pi}</param>
+          <param name="max">${double_pi}</param>
         </command_interface>
         <command_interface name="velocity">
@@ -43,6 +46,6 @@
       <joint name="joint_2">
         <command_interface name="position">
-          <param name="min">{-2*pi}</param>
-          <param name="max">{2*pi}</param>
+          <param name="min">${neg_double_pi}</param>
+          <param name="max">${double_pi}</param>
         </command_interface>
         <command_interface name="velocity">
@@ -57,6 +60,6 @@
       <joint name="joint_3">
         <command_interface name="position">
-          <param name="min">{-pi}</param>
-          <param name="max">{pi}</param>
+          <param name="min">${neg_pi}</param>
+          <param name="max">${pi}</param>
         </command_interface>
         <command_interface name="velocity">
@@ -71,6 +74,6 @@
       <joint name="joint_4">
         <command_interface name="position">
-          <param name="min">{-2*pi}</param>
-          <param name="max">{2*pi}</param>
+          <param name="min">${neg_double_pi}</param>
+          <param name="max">${double_pi}</param>
         </command_interface>
         <command_interface name="velocity">
@@ -85,6 +88,6 @@
       <joint name="joint_5">
         <command_interface name="position">
-          <param name="min">{-2*pi}</param>
-          <param name="max">{2*pi}</param>
+          <param name="min">${neg_double_pi}</param>
+          <param name="max">${double_pi}</param>
         </command_interface>
         <command_interface name="velocity">
@@ -99,6 +102,6 @@
       <joint name="joint_6">
         <command_interface name="position">
-          <param name="min">{-2*pi}</param>
-          <param name="max">{2*pi}</param>
+          <param name="min">${neg_double_pi}</param>
+          <param name="max">${double_pi}</param>
         </command_interface>
         <command_interface name="velocity">
