Commit message: Model connected

File: dsr_moveit2/dsr_moveit_config_m1013/config/m1013.ros2_control.xacro (robot description, xacro)
@@ -50,4 +50,6 @@
                 <state_interface name="velocity"/>
             </joint>
+            <!-- Import Gripper Control -->
+            <!-- <xacro:insert_block name="gripper_control_xacro"/> -->
         </ros2_control>
     </xacro:macro>

File: dsr_moveit2/dsr_moveit_config_m1013/config/m1013.urdf.xacro (robot description, xacro)
@@ -6,4 +6,15 @@
     <!-- Import control_xacro -->
     <xacro:include filename="m1013.ros2_control.xacro" />
+    <!-- Import robotiq 2f85 gripper -->
+    <xacro:include filename="$(find dsr_description2)/urdf/robotiq_2f_85_macro.urdf.xacro" />
     <xacro:m1013_ros2_control name="FakeSystem" initial_positions_file="$(arg initial_positions_file)"/>
+    <!-- Attach Robotiq 2F-85 gripper -->
+    <xacro:robotiq_gripper
+        name="RobotiqGripper"
+        prefix=""
+        parent="link_6"
+        use_fake_hardware="false"
+        include_ros2_control="false">
+        <origin xyz="0 0 0" rpy="0 0 0" />
+    </xacro:robotiq_gripper>
 </robot>
