Commit message: Refactoring: Moveit2 gripper code

File: dsr_description2/gripper/robotiq.ros2_control.xacro (robot description, xacro)
@@ -1,9 +1,6 @@
 <?xml version="1.0"?>
 <robot xmlns:xacro="http://www.ros.org/wiki/xacro">
-  <!-- Robotiq Gripper ros2_control system (mode-aware) -->
   <xacro:arg name="mode" default="virtual"/>
   <xacro:arg name="mock_sensor_commands" default="true"/>
-  <xacro:arg name="com_port" default="/dev/ttyUSB0"/>
-  <!-- 조인트/시스템 이름을 파라미터화 (프리픽스 대응) -->
   <xacro:arg name="joint_name"  default="robotiq_85_left_knuckle_joint"/>
   <xacro:arg name="system_name" default="robotiq_gripper_system"/>
@@ -15,24 +12,20 @@
   <xacro:arg name="max_speed" default="0.150"/>
   <xacro:arg name="max_force" default="235.0"/>
-  <xacro:macro name="robotiq_gripper_system" params="
-      mode:=${mode}
-      com_port:=${com_port}
-      joint_name:=${joint_name}
-      system_name:=${system_name}
-      pos_min:=${pos_min}
-      pos_max:=${pos_max}
-      init_pos:=${init_pos}
-      speed_mult:=${speed_mult}
-      force_mult:=${force_mult}
-      max_speed:=${max_speed}
-      max_force:=${max_force}
-      mock_sensor_commands:=${mock_sensor_commands}">
-    <!-- REAL: 실제 하드웨어 드라이버 -->
+<xacro:macro name="robotiq_gripper_system" params="
+      mode
+      joint_name
+      system_name
+      pos_min
+      pos_max
+      init_pos
+      speed_mult
+      force_mult
+      max_speed
+      max_force
+      mock_sensor_commands">
     <xacro:if value="${mode == 'real'}">
       <ros2_control name="${system_name}" type="system">
         <hardware>
-          <!-- 실제 사용 드라이버 플러그인명 확인/수정 필요 -->
           <plugin>robotiq_driver/RobotiqGripperHardwareInterface</plugin>
-          <param name="COM_port">${com_port}</param>
           <param name="gripper_speed_multiplier">${speed_mult}</param>
           <param name="gripper_force_multiplier">${force_mult}</param>
@@ -52,5 +45,4 @@
       </ros2_control>
     </xacro:if>
-    <!-- VIRTUAL: 모의 하드웨어 -->
     <xacro:unless value="${mode == 'real'}">
       <ros2_control name="${system_name}" type="system">

File: dsr_description2/gripper/robotiq.xacro (robot description, xacro)
@@ -1,13 +1,5 @@
 <?xml version="1.0"?>
 <robot xmlns:xacro="http://www.ros.org/wiki/xacro">
-  <!--
-    Robotiq 2F-85 module
-    Params:
-      parent  : 부착 부모 링크명 (예: tool0, link_6 등)
-      prefix  : 멀티로봇 충돌 방지용 접두사 (예: dsr01_)
-      base_xyz/base_rpy : 베이스 조인트 오프셋 (필요시 조정)
-  -->
   <xacro:macro name="robotiq_85" params="parent prefix base_xyz:='0 0 0' base_rpy:='0 0 0'">
-    <!-- ===== Links ===== -->
     <link name="${prefix}robotiq_85_base_link">
       <visual>
@@ -99,5 +91,4 @@
       </inertial>
     </link>
-    <!-- 닫힘 고정 TCP 링크 -->
     <link name="${prefix}gripper_tcp_closed">
       <inertial>
@@ -114,5 +105,4 @@
       </visual>
     </link>
-        <!-- 닫힘 고정 TCP 링크 -->
     <link name="${prefix}gripper_tcp_opened">
       <inertial>
@@ -129,5 +119,4 @@
       </visual>
     </link>
-    <!-- ===== Joints ===== -->
     <joint name="${prefix}robotiq_85_base_joint" type="fixed">
       <parent link="${parent}"/>
@@ -135,5 +124,4 @@
       <origin xyz="${base_xyz}" rpy="${base_rpy}"/>
     </joint>
-    <!-- Actuated joint (controller 대상) -->
     <joint name="${prefix}robotiq_85_left_knuckle_joint" type="revolute">
       <parent link="${prefix}robotiq_85_base_link"/>

Commit message: Refactoring:robotiq_ros2.control.xacro

File: dsr_description2/gripper/robotiq.ros2_control.xacro (robot description, xacro)
@@ -24,25 +24,4 @@
       max_force
       mock_sensor_commands">
-    <xacro:if value="${mode == 'real'}">
-      <ros2_control name="${system_name}" type="system">
-        <hardware>
-          <plugin>robotiq_driver/RobotiqGripperHardwareInterface</plugin>
-          <param name="gripper_speed_multiplier">${speed_mult}</param>
-          <param name="gripper_force_multiplier">${force_mult}</param>
-          <param name="gripper_max_speed">${max_speed}</param>
-          <param name="gripper_max_force">${max_force}</param>
-        </hardware>
-        <joint name="${joint_name}">
-          <command_interface name="position">
-            <param name="min">${pos_min}</param>
-            <param name="max">${pos_max}</param>
-          </command_interface>
-          <state_interface name="position">
-            <param name="initial_value">${init_pos}</param>
-          </state_interface>
-          <state_interface name="velocity"/>
-        </joint>
-      </ros2_control>
-    </xacro:if>
     <xacro:unless value="${mode == 'real'}">
       <ros2_control name="${system_name}" type="system">
